File: ssla.kicad_pcb (KiCad board)
At the start: 4 copper layers, 81 x 49 mm, 217 parts, among them J1 USB_C_Receptacle_USB2.0_14P, J2 Conn_02x10_Odd_Even, J3 Conn_02x10_Odd_Even, J4 Conn_02x10_Odd_Even, J5 Conn_02x10_Odd_Even, J6 TC2050, U1 TLV75533PDRV, U2 AP2127K-2.5, U3 BL24C256A, U4 USBLC6-2P6, U5 CY7C68013A-56LTX, U6 ECP5U_25_CABGA256, U7 W25Q16JVUXIQ, U8 TPS62A01ADRLR, Y1 24 MHz

Commit message: Ordered
Parts:
- added C48: 4.7u, Capacitor_SMD:C_0402_1005Metric, B.Cu at (153.0, 80.4)
- added C49: 4.7u, Capacitor_SMD:C_0402_1005Metric, B.Cu at (156.2, 76.4)
- added D66: LED_Small, LED_SMD:LED_0603_1608Metric, F.Cu at (146.0, 85.2)
- added R83: 1k, Resistor_SMD:R_0402_1005Metric, F.Cu at (148.5, 85.2)
- moved C23 26.8 mm to (123.6, 71.8), turned to -90 degrees
- moved C28 23.9 mm to (129.0, 72.3), turned to -90 degrees
- moved U2 23.0 mm to (126.2, 72.3)
- moved FB1 14.9 mm to (130.5, 83.6)
Connections:
- U6 pad A10: /PB7/FD7 -> /PB2/FD2
- U6 pad A11: /PB1/FD1 -> /PB3/FD3
- U6 pad A12: /PA2/SLOE -> /PB4/FD4
- U6 pad A13: /PB3/FD3 -> /PB5/FD5
- U6 pad A14: /PA0/~{INT0} -> /PB6/FD6
- U6 pad A15: /CTL0/FLAGA -> /PB7/FD7
- U6 pad A2: unconnected-(U6B-PT4A/+-PadA2) -> /LED
- U6 pad A9: /RDY0/SLRD -> /PB0/FD0
- U6 pad B1: /IO16 -> /IO22
- U6 pad B10: /PA6/PKTEND -> /PB1/FD1
- U6 pad B11: /PA4/FIOADDR0 -> /RDY0/SLRD
- U6 pad B12: /PB2/FD2 -> /CTL0/FLAGA
- U6 pad B13: /PB5/FD5 -> /CTL1/FLAGB
- U6 pad B14: /PB4/FD4 -> /PA0/~{INT0}
- U6 pad B15: /IO33 -> /IO46
- U6 pad B16: /IO32 -> /IO47
- U6 pad B2: /IO17 -> /IO23
- U6 pad C1: /IO18 -> /IO20
- U6 pad C10: /PB6/FD6 -> /RDY1/SLWR
- U6 pad C12: /PB0/FD0 -> /PA5/FIOADDR1
- U6 pad C13: /PA5/FIOADDR1 -> /PA2/SLOE
- U6 pad C15: /IO35 -> /IO44
- U6 pad C16: /IO34 -> /IO45
- U6 pad C2: /IO19 -> /IO21
- U6 pad D1: /IO20 -> /IO19
- U6 pad D12: /CTL1/FLAGB -> /PA4/FIOADDR0
- U6 pad D13: /RDY1/SLWR -> /PA6/PKTEND
- U6 pad D16: /IO36 -> /IO42
- U6 pad E1: /IO23 -> /IO17
- U6 pad E15: /IO37 -> /IO41
- U6 pad E16: /IO39 -> /IO43
- U6 pad E2: /IO21 -> /IO18
- U6 pad F1: /IO24 -> /IO31
- U6 pad F15: /IO38 -> /IO39
- U6 pad F2: /IO22 -> /IO16
- U6 pad G1: /IO26 -> /IO29
- U6 pad G15: /IO41 -> /IO37
- U6 pad G16: /IO43 -> /IO38
- U6 pad G2: /IO25 -> /IO30
- U6 pad H15: /IO44 -> /IO36
- U6 pad H2: /IO27 -> /IO28
- U6 pad J1: /IO28 -> /IO27
- U6 pad J15: /IO46 -> /IO34
- U6 pad J16: /IO45 -> /IO35
- U6 pad J2: /IO29 -> /IO26
- U6 pad K1: /IO30 -> /IO25
- U6 pad K15: /IO42 -> /IO32
- U6 pad K16: /IO47 -> /IO33
- U6 pad K2: /IO31 -> /IO24
- U6 pad L1: /IO00 -> /IO15
- U6 pad L15: /IO49 -> /IO54
- U6 pad L16: /IO48 -> /IO55
- U6 pad L2: /IO01 -> /IO14
- U6 pad M1: /IO02 -> /IO13
- U6 pad M15: /IO51 -> /IO52
- U6 pad M16: /IO50 -> /IO53
- U6 pad M2: /IO03 -> /IO12
- U6 pad N1: /IO04 -> /IO11
- U6 pad N16: /IO52 -> /IO51
- U6 pad N3: /IO13 -> /IO08
- U6 pad P1: /IO06 -> /IO09
- U6 pad P14: /IO56 -> /IO63
- U6 pad P15: /IO53 -> /IO49
- U6 pad P16: /IO54 -> /IO50
- U6 pad P2: /IO05 -> /IO10
- U6 pad P3: /IO15 -> /IO05
- U6 pad R12: /IO62 -> /IO56
- U6 pad R13: /IO60 -> /IO58
- U6 pad R14: /IO59 -> /IO60
- U6 pad R15: /IO57 -> /IO62
- U6 pad R16: /IO55 -> /IO48
- U6 pad R2: /IO08 -> /IO06
- U6 pad R3: /IO10 -> /IO03
- U6 pad R4: /IO11 -> /IO01
- U6 pad T13: /IO63 -> /IO57
- U6 pad T14: /IO61 -> /IO59
- U6 pad T15: /IO58 -> /IO61
- U6 pad T2: /IO09 -> /IO04
- U6 pad T3: /IO12 -> /IO02
- U6 pad T4: /IO14 -> /IO00
Routing:
- net +3V3: track 102.3 -> 180.7 mm, vias 22 -> 25
- net +2V5: track 18.8 -> 50.2 mm, vias 2 -> 3
- net +5V: track 3.21 -> 34.5 mm
- net GND: track 95.0 -> 114.4 mm, vias 139 -> 160
- net +1V1: track 46.2 -> 63.9 mm, vias 5 -> 7
- net /PA6/PKTEND: track 16.0 -> 20.1 mm, vias 1 -> 2
- net /PA4/FIOADDR0: track 15.7 -> 19.6 mm
- net /PA2/SLOE: track 14.5 -> 17.7 mm, vias 1 -> 2
- net /CTL1/FLAGB: track 15.5 -> 12.4 mm
- net /PB0/FD0: track 10.8 -> 7.83 mm, vias 1 -> 0
- net /IO63: track 7.16 -> 9.67 mm
- net /LED: track 0.00 -> 2.49 mm
- net /SW: track 0.00 -> 2.42 mm
- net /CDONE: track 45.4 -> 43.3 mm
- net /PROGRAMN: track 45.6 -> 43.6 mm
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Other:
- board text added: "ACQ"
- board text added: "By Emil Fresk"
- board text added: "DONE"
- board text added: "RECOVERY"
