File: ssla.kicad_pcb (KiCad board)
At the start: 4 copper layers, 81 x 49 mm, 221 parts, among them J1 USB_C_Receptacle_USB2.0_14P, J2 Conn_02x10_Odd_Even, J3 Conn_02x10_Odd_Even, J4 Conn_02x10_Odd_Even, J5 Conn_02x10_Odd_Even, J6 TC2050, U1 TLV75533PDRV, U2 AP2127K-2.5, U3 BL24C256A, U4 USBLC6-2P6, U5 CY7C68013A-56LTX, U6 ECP5U_25_CABGA256, U7 W25Q16JVUXIQ, U8 TPS62A01ADRLR, Y1 24 MHz

Commit message: wip
Parts:
- removed C11, C12, C15, C18, C21, C22, C25, C26, C27, C29, C30: 0.1u, Capacitor_SMD:C_0402_1005Metric
- removed C19, C20: 12p, Capacitor_SMD:C_0402_1005Metric
- removed TP11, TP12: TestPoint_Small, TestPoint:TestPoint_Pad_D1.0mm
- removed U3: BL24C256A, Package_SO:TSSOP-8_4.4x3mm_P0.65mm
- removed U4: USBLC6-2P6, Package_TO_SOT_SMD:SOT-666
- removed U5: CY7C68013A-56LTX, Package_DFN_QFN:QFN-56-1EP_8x8mm_P0.5mm_EP4.5x5.2mm
- added C50: 22u, Capacitor_SMD:C_0603_1608Metric, F.Cu at (94.8, 100.9)
- added C51: 2.2u, Capacitor_SMD:C_0402_1005Metric, F.Cu at (109.0, 103.2)
- added C52: 0.1u, Capacitor_SMD:C_0402_1005Metric, F.Cu at (107.1, 103.2)
- added C53: 0.1u, Capacitor_SMD:C_0402_1005Metric, F.Cu at (105.1, 103.2)
- added C54: 22u, Capacitor_SMD:C_0603_1608Metric, F.Cu at (92.3, 100.9)
- added C55: 0.1u, Capacitor_SMD:C_0402_1005Metric, F.Cu at (103.1, 103.2)
- added C56: 0.1u, Capacitor_SMD:C_0402_1005Metric, F.Cu at (127.6, 87.5)
- added C57: 0.1u, Capacitor_SMD:C_0402_1005Metric, F.Cu at (127.6, 88.5)
- added C58: 10u, Capacitor_SMD:C_0603_1608Metric, F.Cu at (89.8, 100.9)
- added FB2: 120 ohm, Inductor_SMD:L_0402_1005Metric, F.Cu at (134.4, 76.7)
- added J7: RJ45_Hanrun_HR911105A_Horizontal, Connector_RJ:RJ45_Hanrun_HR911105A_Horizontal, F.Cu at (122.0, 80.4)
- added R84: 6.49k, Resistor_SMD:R_0402_1005Metric, F.Cu at (139.5, 82.6)
- added R85: 1k, Resistor_SMD:R_0402_1005Metric, F.Cu at (99.1, 100.3)
- added R86: 10k, Resistor_SMD:R_0402_1005Metric, F.Cu at (97.1, 100.3)
- added U9: KSZ8081RNA, Package_DFN_QFN:QFN-24-1EP_4x4mm_P0.5mm_EP2.6x2.6mm, F.Cu at (139.8, 78.6)
- C8: value 4.7u -> 0.1u; moved to F.Cu
- R4: value 0 -> 22; footprint Resistor_SMD:R_0805_2012Metric -> Resistor_SMD:R_0402_1005Metric
- R5: value 2.2k -> 22
- R6: value 100k -> 5.1k; moved to F.Cu
- R7: value 2.2k -> 5.1k
- R8: value 100k -> 10k; moved to F.Cu
- Y1: value 24 MHz -> 25 MHz; footprint Crystal:Crystal_SMD_2016-4Pin_2.0x1.6mm -> Oscillator:Oscillator_SMD_SiT_PQFN-4Pin_2.0x1.6mm
- moved R8 43.7 mm to (103.0, 100.3)
- moved FB1 24.0 mm to (113.8, 66.4), turned to 180 degrees
- moved J1 23.3 mm to (108.0, 64.0)
- moved C24 19.1 mm to (117.9, 69.1)
- moved C32 19.1 mm to (115.5, 70.4)
- moved C33 19.1 mm to (117.8, 74.1)
- moved C34 19.1 mm to (117.8, 72.6)
- moved R81 19.1 mm to (115.5, 71.4)
- moved R82 19.1 mm to (115.5, 69.4)
- moved U8 19.1 mm to (117.9, 70.8)
- moved L1 19.1 mm to (120.6, 70.7)
- moved R2 18.7 mm to (116.1, 66.7)
- moved R1 18.7 mm to (117.2, 66.7)
- moved U1 16.6 mm to (125.3, 70.5)
- moved C3 16.6 mm to (123.5, 70.5)
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Connections:
- net /PA0/~{INT0} renamed /~{ETH.RST}
- C8 pad 1: +3V3 -> GND
- C8 pad 2: GND -> +3V3
- J1 pad A6: /D_P -> unconnected-(J1-D+-PadA6)
- J1 pad A7: /D_N -> unconnected-(J1-D--PadA7)
- J1 pad B6: /D_P -> unconnected-(J1-D+-PadB6)
- J1 pad B7: /D_N -> unconnected-(J1-D--PadB7)
- R4 pad 1: +3V3 -> Net-(Y1-OUT)
- R4 pad 2: Net-(U3-A1) -> /FPGA_XI
- R5 pad 1: +3V3 -> Net-(Y1-OUT)
- R5 pad 2: /SCL -> /PHY_XI
- R6 pad 2: /~{RESET} -> /ETH.MDIO
- R7 pad 2: /SDA -> /ETH.MDC
- R8 pad 2: +3V3 -> GND
- U6 pad A10: /PB2/FD2 -> /ETH.TXD0
- U6 pad A11: /PB3/FD3 -> /ETH.TXD1
- U6 pad A12: /PB4/FD4 -> /ETH.RXD0
- U6 pad A13: /PB5/FD5 -> /ETH.RXD1
- U6 pad A14: /PB6/FD6 -> /ETH.CRS_DV
- U6 pad A15: /PB7/FD7 -> /ETH.RXER
- U6 pad A9: /PB0/FD0 -> /ETH.TXEN
- U6 pad B10: /PB1/FD1 -> unconnected-(U6C-PT44A/+-PadB10)
- U6 pad B11: /RDY0/SLRD -> unconnected-(U6C-PT49A/+-PadB11)
- U6 pad B12: /CTL0/FLAGA -> /ETH.MDIO
- U6 pad B13: /CTL1/FLAGB -> /ETH.MDC
- U6 pad B9: /CLKOUT -> /FPGA_XI
- U6 pad C10: /RDY1/SLWR -> unconnected-(U6C-PT44B/--PadC10)
- U6 pad C12: /PA5/FIOADDR1 -> unconnected-(U6C-PT56B/--PadC12)
- U6 pad C13: /PA2/SLOE -> unconnected-(U6C-PT60B/--PadC13)
- U6 pad C8: /IFCLK -> /ETH.REF_CLK
- U6 pad D12: /PA4/FIOADDR0 -> unconnected-(U6C-PT58A/+-PadD12)
- U6 pad D13: /PA6/PKTEND -> unconnected-(U6C-PT62A/+-PadD13)
- Y1 pad 1: /XTALIN -> +3V3
- Y1 pad 3: /XTALOUT -> Net-(Y1-OUT)
- Y1 pad 4: GND -> +3V3
Routing:
- net +3V3: track 180.7 -> 120.7 mm, vias 25 -> 15
- net /PROGRAMN: track 43.6 -> 3.38 mm, vias 2 -> 1
- net /CDONE: track 43.3 -> 7.62 mm, vias 4 -> 2
- net GND: track 114.4 -> 87.9 mm, vias 160 -> 125
- net /RDY1/SLWR: track 23.1 -> 0.00 mm, vias 2 -> 0
- net /RDY0/SLRD: track 22.5 -> 0.00 mm, vias 2 -> 0
- net /PA6/PKTEND: track 20.1 -> 0.00 mm, vias 2 -> 0
- net /PA4/FIOADDR0: track 19.6 -> 0.00 mm, vias 2 -> 0
- net /PA5/FIOADDR1: track 19.0 -> 0.00 mm, vias 2 -> 0
- net /CLKOUT: track 19.0 -> 0.00 mm, vias 2 -> 0
- net /D-: track 18.6 -> 0.00 mm
- net /PA2/SLOE: track 17.7 -> 0.00 mm, vias 2 -> 0
- net /TX+: track 0.00 -> 17.4 mm
- net /TX-: track 0.00 -> 17.3 mm
- net /D+: track 17.1 -> 0.00 mm
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Other:
- board size 81 x 49 mm -> 97 x 49 mm

Commit message: save
Parts:
- removed C1, C10, C14, C17, C37, C39, C41, C43, C45, C5, C9: 10n, Capacitor_SMD:C_0402_1005Metric
- removed C13, C16, C2, C35, C36, C38, C4, C40, C42, C44, C52, C53, C55, C56, C57, C6, C7, C8: 0.1u, Capacitor_SMD:C_0402_1005Metric
- removed C23, C24, C3, C46, C47, C48, C49: 4.7u, Capacitor_SMD:C_0402_1005Metric
- removed C28, C31, C33, C34, C58: 10u, Capacitor_SMD:C_0603_1608Metric
- removed C32: 27p, Capacitor_SMD:C_0402_1005Metric
- removed C50, C54: 22u, Capacitor_SMD:C_0603_1608Metric
- removed C51: 2.2u, Capacitor_SMD:C_0402_1005Metric
- removed D1, D10, D11, D12, D13, D14, D15, D16, D17, D18, D19, D2, D20, D21, D22, D23, D24, D25, D26, D27, D28, D29, D3, D30, D31, D32, D33, D34, D35, D36, D37, D38, D39, D4, D40, D41, D42, D43, D44, D45, D46, D47, D48, D49, D5, D50, D51, D52, D53, D54, D55, D56, D57, D58, D59, D6, D60, D61, D62, D63, D64, D7, D8, D9: D_TVS_Small, Diode_SMD:D_SOD-923
- removed D65, D66: LED_Small, LED_SMD:LED_0603_1608Metric
- removed FB1: FerriteBead_Small, Resistor_SMD:R_0402_1005Metric
- removed FB2: 120 ohm, Inductor_SMD:L_0402_1005Metric
- removed H1, H2, H3, H4: MountingHole_Pad, MountingHole:MountingHole_2.2mm_M2_Pad_Via
- removed J1: USB_C_Receptacle_USB2.0_14P, Connector_USB:USB_C_Receptacle_GCT_USB4105-xx-A_16P_TopMnt_Horizontal
- removed J2, J3, J4, J5: Conn_02x10_Odd_Even, Connector_IDC:IDC-Header_2x10_P2.54mm_Vertical
- removed J7: RJ45_Hanrun_HR911105A_Horizontal, Connector_RJ:RJ45_Hanrun_HR911105A_Horizontal
- removed L1: 1.5u, Inductor_SMD:L_1008_2520Metric
- removed R1, R2, R6, R7: 5.1k, Resistor_SMD:R_0402_1005Metric
- removed R10, R3, R43, R44, R83, R85, R9: 1k, Resistor_SMD:R_0402_1005Metric
- removed R11, R12, R13, R14, R15, R16, R17, R18, R19, R20, R21, R22, R23, R24, R25, R26, R27, R28, R29, R30, R31, R32, R33, R34, R35, R36, R37, R38, R39, R40, R41, R42, R46, R47, R48, R49, R50, R51, R52, R53, R54, R55, R56, R57, R58, R59, R60, R61, R62, R63, R64, R65, R66, R67, R68, R69, R70, R71, R72, R73, R74, R75, R76, R77: 100, Resistor_SMD:R_0402_1005Metric
- removed R4, R5: 22, Resistor_SMD:R_0402_1005Metric
- removed R45, R78, R79, R8, R80, R86: 10k, Resistor_SMD:R_0402_1005Metric
- removed R81: 82k, Resistor_SMD:R_0402_1005Metric
- removed R82: 100k, Resistor_SMD:R_0402_1005Metric
- removed R84: 6.49k, Resistor_SMD:R_0402_1005Metric
- removed U1: TLV75533PDRV, Package_SON:WSON-6-1EP_2x2mm_P0.65mm_EP1x1.6mm
- removed U2: AP2127K-2.5, Package_TO_SOT_SMD:SOT-23-5
- removed U8: TPS62A01ADRLR, Package_TO_SOT_SMD:SOT-563
- removed Y1: 25 MHz, Oscillator:Oscillator_SMD_SiT_PQFN-4Pin_2.0x1.6mm
- added C101: 0.1u, Capacitor_SMD:C_0402_1005Metric, F.Cu at (144.0, 85.3)
- added C102: 10n, Capacitor_SMD:C_0402_1005Metric, F.Cu at (62.5, 65.1)
- added C103: 0.1u, Capacitor_SMD:C_0402_1005Metric, F.Cu at (62.5, 67.1)
- added C104: 4.7u, Capacitor_SMD:C_0402_1005Metric, F.Cu at (62.5, 69.0)
- added C201: 0.1u, Capacitor_SMD:C_0402_1005Metric, B.Cu at (157.9, 93.5)
- added C202: 0.1u, Capacitor_SMD:C_0402_1005Metric, B.Cu at (169.4, 93.5)
- added C203: 0.1u, Capacitor_SMD:C_0402_1005Metric, B.Cu at (180.9, 93.5)
- added C301: 0.1u, Capacitor_SMD:C_0402_1005Metric, B.Cu at (169.4, 68.5)
- added C302: 0.1u, Capacitor_SMD:C_0402_1005Metric, B.Cu at (157.9, 68.5)
- added C303: 0.1u, Capacitor_SMD:C_0402_1005Metric, B.Cu at (180.9, 68.5)
- added C401: 4.7u, Capacitor_SMD:C_0402_1005Metric, F.Cu at (132.5, 61.0)
- added C402: 4.7u, Capacitor_SMD:C_0402_1005Metric, F.Cu at (139.0, 61.0)
- added C403: 4.7u, Capacitor_SMD:C_0402_1005Metric, F.Cu at (132.5, 63.5)
- added C404: 4.7u, Capacitor_SMD:C_0402_1005Metric, F.Cu at (139.0, 63.4)
- added C405: 4.7u, Capacitor_SMD:C_0402_1005Metric, F.Cu at (138.6, 68.6)
- added C406: 27p, Capacitor_SMD:C_0402_1005Metric, F.Cu at (134.7, 59.9)
- added C407: 27p, Capacitor_SMD:C_0402_1005Metric, F.Cu at (141.2, 59.9)
- added C408: 27p, Capacitor_SMD:C_0402_1005Metric, F.Cu at (130.3, 64.6)
- added C409: 22u, Capacitor_SMD:C_0603_1608Metric, F.Cu at (132.8, 56.2)
- added C410: 22u, Capacitor_SMD:C_0603_1608Metric, F.Cu at (139.3, 57.7)
- added C411: 22u, Capacitor_SMD:C_0603_1608Metric, F.Cu at (132.2, 66.8)
- added C412: 22u, Capacitor_SMD:C_0603_1608Metric, F.Cu at (132.8, 57.7)
- added C413: 22u, Capacitor_SMD:C_0603_1608Metric, F.Cu at (139.3, 56.2)
- added C414: 4.7u, Capacitor_SMD:C_0402_1005Metric, F.Cu at (138.6, 69.6)
- added C501: 0.1u, Capacitor_SMD:C_0402_1005Metric, F.Cu at (42.5, 77.1)
- added C502: 0.1u, Capacitor_SMD:C_0402_1005Metric, F.Cu at (42.5, 79.0)
- added C503: 0.1u, Capacitor_SMD:C_0402_1005Metric, F.Cu at (42.5, 81.0)
- added C504: 22u, Capacitor_SMD:C_0603_1608Metric, F.Cu at (40.2, 93.3)
- added C505: 0.1u, Capacitor_SMD:C_0402_1005Metric, F.Cu at (42.5, 83.0)
- added C506: 22u, Capacitor_SMD:C_0603_1608Metric, F.Cu at (40.2, 95.8)
- added C507: 0.1u, Capacitor_SMD:C_0402_1005Metric, F.Cu at (42.5, 85.0)
- added C508: 2.2u, Capacitor_SMD:C_0402_1005Metric, F.Cu at (42.5, 86.9)
- added C509: 0.1u, Capacitor_SMD:C_0402_1005Metric, F.Cu at (42.5, 88.9)
- added C510: 10n, Capacitor_SMD:C_0402_1005Metric, F.Cu at (42.5, 90.9)
- added C601: 10n, Capacitor_SMD:C_0402_1005Metric, F.Cu at (79.9, 48.5)
- added C602: 0.1u, Capacitor_SMD:C_0402_1005Metric, F.Cu at (79.9, 50.5)
- added C603: 0.1u, Capacitor_SMD:C_0402_1005Metric, B.Cu at (167.2, 82.6)
- added C604: 0.1u, Capacitor_SMD:C_0402_1005Metric, F.Cu at (79.9, 54.4)
- added C605: 10n, Capacitor_SMD:C_0402_1005Metric, F.Cu at (79.9, 56.4)
- added C606: 10n, Capacitor_SMD:C_0402_1005Metric, F.Cu at (82.7, 48.5)
- added C607: 10n, Capacitor_SMD:C_0402_1005Metric, F.Cu at (82.7, 50.5)
- added C608: 0.1u, Capacitor_SMD:C_0402_1005Metric, F.Cu at (82.7, 52.4)
- added C609: 0.1u, Capacitor_SMD:C_0402_1005Metric, F.Cu at (82.7, 54.4)
- added C610: 0.1u, Capacitor_SMD:C_0402_1005Metric, F.Cu at (82.7, 56.4)
- added C611: 4.7u, Capacitor_SMD:C_0402_1005Metric, F.Cu at (85.6, 48.5)
- added C612: 10n, Capacitor_SMD:C_0402_1005Metric, F.Cu at (85.6, 50.5)
- added C613: 4.7u, Capacitor_SMD:C_0402_1005Metric, F.Cu at (85.6, 52.4)
- added C701: 0.1u, Capacitor_SMD:C_0402_1005Metric, F.Cu at (94.5, 90.9)
- added C702: 10n, Capacitor_SMD:C_0402_1005Metric, F.Cu at (94.5, 92.9)
- added C703: 0.1u, Capacitor_SMD:C_0402_1005Metric, F.Cu at (94.5, 94.8)
- added C704: 10n, Capacitor_SMD:C_0402_1005Metric, F.Cu at (94.5, 96.8)
- added C801: 4.7u, Capacitor_SMD:C_0402_1005Metric, F.Cu at (94.5, 77.1)
- added C802: 0.1u, Capacitor_SMD:C_0402_1005Metric, F.Cu at (94.5, 79.0)
- added C803: 10n, Capacitor_SMD:C_0402_1005Metric, F.Cu at (94.5, 81.0)
- added C804: 4.7u, Capacitor_SMD:C_0402_1005Metric, F.Cu at (94.5, 83.0)
- added C805: 0.1u, Capacitor_SMD:C_0402_1005Metric, F.Cu at (94.5, 85.0)
- added C806: 10n, Capacitor_SMD:C_0402_1005Metric, F.Cu at (94.5, 86.9)
- added C901: 0.1u, Capacitor_SMD:C_0402_1005Metric, F.Cu at (148.4, 62.5)
- added D101: RED, LED_SMD:LED_0603_1608Metric, F.Cu at (121.0, 70.5)
- added D601: RED, LED_SMD:LED_0603_1608Metric, F.Cu at (167.5, 77.0)
- added D901: CDSOD323-T03SC, Diode_SMD:D_SOD-323, F.Cu at (149.0, 57.0)
- added FB101: 120 ohm, Inductor_SMD:L_0402_1005Metric, F.Cu at (48.0, 63.1)
- added FB501: 120 ohm, Inductor_SMD:L_0402_1005Metric, F.Cu at (39.7, 77.1)
- added H101: MountingHole_Pad, MountingHole:MountingHole_2.2mm_M2_Pad_Via, F.Cu at (192.5, 54.0)
- added H102: MountingHole_Pad, MountingHole:MountingHole_2.2mm_M2_Pad_Via, F.Cu at (192.5, 106.0)
- added H103: MountingHole_Pad, MountingHole:MountingHole_2.2mm_M2_Pad_Via, F.Cu at (121.5, 54.0)
- added H104: MountingHole_Pad, MountingHole:MountingHole_2.2mm_M2_Pad_Via, F.Cu at (121.5, 106.0)
- added J101: Sync In, Connector_JST:JST_PH_B2B-PH-K_1x02_P2.00mm_Vertical, F.Cu at (152.0, 58.0)
- added J102: USB_C_Receptacle_USB2.0_14P, Connector_USB:USB_C_Receptacle_GCT_USB4105-xx-A_16P_TopMnt_Horizontal, F.Cu at (121.5, 62.0)
- added J103: Channel 1, Connector_IDC:IDC-Header_2x10_P2.54mm_Vertical, F.Cu at (166.6, 99.8)
- added J104: Channel 2, Connector_IDC:IDC-Header_2x10_P2.54mm_Vertical, F.Cu at (189.4, 60.2)
- added J105: Sync Out, Connector_JST:JST_PH_B2B-PH-K_1x02_P2.00mm_Vertical, F.Cu at (139.5, 104.0)
- added J106: Sync Out, Connector_JST:JST_PH_B2B-PH-K_1x02_P2.00mm_Vertical, F.Cu at (121.5, 97.0)
- added J107: Sync Out, Connector_JST:JST_PH_B2B-PH-K_1x02_P2.00mm_Vertical, F.Cu at (127.5, 97.0)
- added J108: Sync Out, Connector_JST:JST_PH_B2B-PH-K_1x02_P2.00mm_Vertical, F.Cu at (133.5, 97.0)
- added J109: Sync Out, Connector_JST:JST_PH_B2B-PH-K_1x02_P2.00mm_Vertical, F.Cu at (127.5, 104.0)
- added J110: Sync Out, Connector_JST:JST_PH_B2B-PH-K_1x02_P2.00mm_Vertical, F.Cu at (133.5, 104.0)
- added J111: Sync Out, Connector_JST:JST_PH_B2B-PH-K_1x02_P2.00mm_Vertical, F.Cu at (139.5, 97.0)
- added J112: Sync Out, Connector_JST:JST_PH_B2B-PH-K_1x02_P2.00mm_Vertical, F.Cu at (145.5, 97.0)
- added J113: Sync Out, Connector_JST:JST_PH_B2B-PH-K_1x02_P2.00mm_Vertical, F.Cu at (151.5, 97.0)
- added J114: Sync Out, Connector_JST:JST_PH_B2B-PH-K_1x02_P2.00mm_Vertical, F.Cu at (145.5, 104.0)
- added J115: Sync Out, Connector_JST:JST_PH_B2B-PH-K_1x02_P2.00mm_Vertical, F.Cu at (151.5, 104.0)
- added J116: Sync Out, Connector_JST:JST_PH_B2B-PH-K_1x02_P2.00mm_Vertical, F.Cu at (157.5, 104.0)
- added J501: RJ45_Hanrun_HR911105A_Horizontal, Connector_RJ:RJ45_Hanrun_HR911105A_Horizontal, F.Cu at (135.1, 75.6)
- added L401: 1u, Inductor_SMD:L_0805_2012Metric, F.Cu at (130.4, 58.7)
- added L402: 1u, Inductor_SMD:L_0805_2012Metric, F.Cu at (136.9, 58.7)
- added L403: 1u, Inductor_SMD:L_0805_2012Metric, F.Cu at (134.6, 65.8)
- added R101: 5.1k, Resistor_SMD:R_0402_1005Metric, F.Cu at (48.0, 65.1)
- added R102: 33, Resistor_SMD:R_0402_1005Metric, F.Cu at (145.5, 81.5)
- added R103: 33, Resistor_SMD:R_0402_1005Metric, F.Cu at (143.5, 81.5)
- added R104: 5.1k, Resistor_SMD:R_0402_1005Metric, F.Cu at (48.0, 71.1)
- added R105: 1k, Resistor_SMD:R_0402_1005Metric, F.Cu at (123.5, 70.5)
- added R201: 100k, Resistor_SMD:R_0402_1005Metric, B.Cu at (187.3, 109.6)
- added R202: 100k, Resistor_SMD:R_0402_1005Metric, B.Cu at (185.3, 109.6)
- added R203: 100k, Resistor_SMD:R_0402_1005Metric, B.Cu at (183.3, 109.6)
- added R204: 100k, Resistor_SMD:R_0402_1005Metric, B.Cu at (181.3, 109.6)
- added R205: 100k, Resistor_SMD:R_0402_1005Metric, B.Cu at (179.3, 109.6)
- added R206: 100k, Resistor_SMD:R_0402_1005Metric, B.Cu at (177.3, 109.6)
- added R207: 100k, Resistor_SMD:R_0402_1005Metric, B.Cu at (175.3, 109.6)
- added R208: 100k, Resistor_SMD:R_0402_1005Metric, B.Cu at (173.3, 109.6)
- added R209: 100k, Resistor_SMD:R_0402_1005Metric, B.Cu at (187.3, 106.7)
- added R210: 100k, Resistor_SMD:R_0402_1005Metric, B.Cu at (185.3, 106.7)
- added R211: 100k, Resistor_SMD:R_0402_1005Metric, B.Cu at (183.3, 106.7)
- added R212: 100k, Resistor_SMD:R_0402_1005Metric, B.Cu at (181.3, 106.7)
- added R213: 100k, Resistor_SMD:R_0402_1005Metric, B.Cu at (179.3, 106.7)
- added R214: 100k, Resistor_SMD:R_0402_1005Metric, B.Cu at (177.3, 106.7)
- added R215: 100k, Resistor_SMD:R_0402_1005Metric, B.Cu at (175.3, 106.7)
- added R216: 100k, Resistor_SMD:R_0402_1005Metric, B.Cu at (173.3, 106.7)
- added R217: 33, Resistor_SMD:R_0402_1005Metric, F.Cu at (170.5, 89.5)
- added R218: 33, Resistor_SMD:R_0402_1005Metric, F.Cu at (171.5, 89.5)
- added R219: 33, Resistor_SMD:R_0402_1005Metric, F.Cu at (173.5, 89.5)
- added R220: 33, Resistor_SMD:R_0402_1005Metric, F.Cu at (175.5, 89.5)
- added R221: 33, Resistor_SMD:R_0402_1005Metric, F.Cu at (174.5, 89.5)
- added R222: 33, Resistor_SMD:R_0402_1005Metric, F.Cu at (172.5, 89.5)
- added R223: 33, Resistor_SMD:R_0402_1005Metric, F.Cu at (182.0, 89.5)
- added R224: 33, Resistor_SMD:R_0402_1005Metric, F.Cu at (183.0, 89.5)
- added R225: 33, Resistor_SMD:R_0402_1005Metric, F.Cu at (185.0, 89.5)
- added R226: 33, Resistor_SMD:R_0402_1005Metric, F.Cu at (187.0, 89.5)
- added R227: 33, Resistor_SMD:R_0402_1005Metric, F.Cu at (186.0, 89.5)
- added R228: 33, Resistor_SMD:R_0402_1005Metric, F.Cu at (184.0, 89.5)
- added R229: 33, Resistor_SMD:R_0402_1005Metric, F.Cu at (159.0, 89.5)
- added R230: 33, Resistor_SMD:R_0402_1005Metric, F.Cu at (160.0, 89.5)
- added R231: 33, Resistor_SMD:R_0402_1005Metric, F.Cu at (162.0, 89.5)
- added R232: 33, Resistor_SMD:R_0402_1005Metric, F.Cu at (161.0, 89.5)
- added R301: 100k, Resistor_SMD:R_0402_1005Metric, B.Cu at (185.5, 53.5)
- added R302: 100k, Resistor_SMD:R_0402_1005Metric, B.Cu at (183.5, 53.5)
- added R303: 100k, Resistor_SMD:R_0402_1005Metric, B.Cu at (181.5, 53.5)
- added R304: 100k, Resistor_SMD:R_0402_1005Metric, B.Cu at (179.5, 53.5)
- added R305: 100k, Resistor_SMD:R_0402_1005Metric, B.Cu at (177.5, 53.5)
- added R306: 100k, Resistor_SMD:R_0402_1005Metric, B.Cu at (175.5, 53.5)
- added R307: 100k, Resistor_SMD:R_0402_1005Metric, B.Cu at (173.5, 53.5)
- added R308: 100k, Resistor_SMD:R_0402_1005Metric, B.Cu at (171.6, 53.5)
- added R309: 100k, Resistor_SMD:R_0402_1005Metric, B.Cu at (185.5, 50.6)
- added R310: 100k, Resistor_SMD:R_0402_1005Metric, B.Cu at (183.5, 50.6)
- added R311: 100k, Resistor_SMD:R_0402_1005Metric, B.Cu at (181.5, 50.6)
- added R312: 100k, Resistor_SMD:R_0402_1005Metric, B.Cu at (179.5, 50.6)
- added R313: 100k, Resistor_SMD:R_0402_1005Metric, B.Cu at (177.5, 50.6)
- added R314: 100k, Resistor_SMD:R_0402_1005Metric, B.Cu at (175.5, 50.6)
- added R315: 100k, Resistor_SMD:R_0402_1005Metric, B.Cu at (173.5, 50.6)
- added R316: 100k, Resistor_SMD:R_0402_1005Metric, B.Cu at (171.6, 50.6)
- added R317: 33, Resistor_SMD:R_0402_1005Metric, F.Cu at (168.5, 70.5)
- added R318: 33, Resistor_SMD:R_0402_1005Metric, F.Cu at (169.5, 70.5)
- added R319: 33, Resistor_SMD:R_0402_1005Metric, F.Cu at (170.5, 70.5)
- added R320: 33, Resistor_SMD:R_0402_1005Metric, F.Cu at (173.5, 70.5)
- added R321: 33, Resistor_SMD:R_0402_1005Metric, F.Cu at (172.5, 70.5)
- added R322: 33, Resistor_SMD:R_0402_1005Metric, F.Cu at (171.5, 70.5)
- added R323: 33, Resistor_SMD:R_0402_1005Metric, F.Cu at (157.0, 70.5)
- added R324: 33, Resistor_SMD:R_0402_1005Metric, F.Cu at (158.0, 70.5)
- added R325: 33, Resistor_SMD:R_0402_1005Metric, F.Cu at (159.0, 70.5)
- added R326: 33, Resistor_SMD:R_0402_1005Metric, F.Cu at (162.0, 70.5)
- added R327: 33, Resistor_SMD:R_0402_1005Metric, F.Cu at (161.0, 70.5)
- added R328: 33, Resistor_SMD:R_0402_1005Metric, F.Cu at (160.0, 70.5)
- added R329: 33, Resistor_SMD:R_0402_1005Metric, F.Cu at (182.0, 70.5)
- added R330: 33, Resistor_SMD:R_0402_1005Metric, F.Cu at (183.0, 70.5)
- added R331: 33, Resistor_SMD:R_0402_1005Metric, F.Cu at (184.0, 70.5)
- added R332: 33, Resistor_SMD:R_0402_1005Metric, F.Cu at (185.0, 70.5)
- added R401: 82k, Resistor_SMD:R_0402_1005Metric, F.Cu at (134.7, 58.9)
- added R402: 100k, Resistor_SMD:R_0402_1005Metric, F.Cu at (134.7, 60.9)
- added R403: 200k, Resistor_SMD:R_0402_1005Metric, F.Cu at (141.2, 58.9)
- added R404: 100k, Resistor_SMD:R_0402_1005Metric, F.Cu at (141.2, 60.9)
- added R405: 450k, Resistor_SMD:R_0402_1005Metric, F.Cu at (130.3, 65.6)
- added R406: 100k, Resistor_SMD:R_0402_1005Metric, F.Cu at (130.3, 63.6)
- added R501: 1k, Resistor_SMD:R_0402_1005Metric, F.Cu at (39.7, 79.1)
- added R502: 10k, Resistor_SMD:R_0402_1005Metric, F.Cu at (39.7, 81.1)
- added R503: 10k, Resistor_SMD:R_0402_1005Metric, F.Cu at (39.7, 83.0)
- added R504: 10k, Resistor_SMD:R_0402_1005Metric, F.Cu at (39.7, 85.0)
- added R505: 5.1k, Resistor_SMD:R_0402_1005Metric, F.Cu at (39.7, 87.0)
- added R506: 5.1k, Resistor_SMD:R_0402_1005Metric, F.Cu at (39.7, 89.0)
- added R507: 6.49k, Resistor_SMD:R_0402_1005Metric, F.Cu at (39.7, 91.0)
- added R508: 33, Resistor_SMD:R_0402_1005Metric, F.Cu at (148.5, 75.5)
- added R509: 33, Resistor_SMD:R_0402_1005Metric, F.Cu at (148.5, 74.5)
- added R510: 33, Resistor_SMD:R_0402_1005Metric, F.Cu at (148.5, 73.5)
- added R511: 33, Resistor_SMD:R_0402_1005Metric, F.Cu at (147.1, 79.2)
- added R512: 33, Resistor_SMD:R_0402_1005Metric, F.Cu at (147.1, 80.2)
- added R513: 33, Resistor_SMD:R_0402_1005Metric, F.Cu at (147.2, 78.3)
- added R514: 33, Resistor_SMD:R_0402_1005Metric, F.Cu at (147.2, 77.3)
- added R515: 33, Resistor_SMD:R_0402_1005Metric, F.Cu at (147.1, 76.4)
- added R601: 10k, Resistor_SMD:R_0402_1005Metric, B.Cu at (167.5, 77.9)
- added R602: 10k, Resistor_SMD:R_0402_1005Metric, F.Cu at (88.5, 50.5)
- added R603: 10k, Resistor_SMD:R_0402_1005Metric, F.Cu at (88.5, 52.5)
- added R604: 33, Resistor_SMD:R_0402_1005Metric, F.Cu at (88.5, 54.5)
- added R605: 1k, Resistor_SMD:R_0402_1005Metric, B.Cu at (165.7, 84.2)
- added R606: 1k, Resistor_SMD:R_0402_1005Metric, B.Cu at (161.0, 80.1)
- added R607: 1k, Resistor_SMD:R_0402_1005Metric, B.Cu at (164.1, 80.4)
- added R608: 10k, Resistor_SMD:R_0402_1005Metric, F.Cu at (170.1, 77.0)
- added R609: 10k, Resistor_SMD:R_0402_1005Metric, B.Cu at (163.1, 80.4)
- added R610: 10k, Resistor_SMD:R_0402_1005Metric, B.Cu at (161.2, 83.4)
- added R611: 10k, Resistor_SMD:R_0402_1005Metric, B.Cu at (164.7, 84.2)
- added R612: 10k, Resistor_SMD:R_0402_1005Metric, B.Cu at (167.5, 78.9)
- added R901: 33, Resistor_SMD:R_0402_1005Metric, F.Cu at (147.0, 54.0)
- added R902: 33, Resistor_SMD:R_0402_1005Metric, F.Cu at (145.0, 54.0)
- added R903: 1k, Resistor_SMD:R_0402_1005Metric, F.Cu at (146.6, 63.5)
- added U101: NUF6401MNT1, footprints:DFN-12-1EP_1.35x3mm_P0.5mm, F.Cu at (138.0, 91.0)
- added U102: NUF6401MNT1, footprints:DFN-12-1EP_1.35x3mm_P0.5mm, F.Cu at (151.0, 91.0)
- added U201: SN74LV6T17, Package_DFN_QFN:DHVQFN-14-1EP_2.5x3mm_P0.5mm_EP1x1.5mm, B.Cu at (172.0, 92.5)
- added U202: SN74LV6T17, Package_DFN_QFN:DHVQFN-14-1EP_2.5x3mm_P0.5mm_EP1x1.5mm, B.Cu at (183.5, 92.5)
- added U203: SN74LV6T17, Package_DFN_QFN:DHVQFN-14-1EP_2.5x3mm_P0.5mm_EP1x1.5mm, B.Cu at (160.5, 92.5)
- added U204: NUF6401MNT1, footprints:DFN-12-1EP_1.35x3mm_P0.5mm, B.Cu at (176.0, 92.5)
- added U205: NUF6401MNT1, footprints:DFN-12-1EP_1.35x3mm_P0.5mm, B.Cu at (187.5, 92.5)
- added U206: NUF6401MNT1, footprints:DFN-12-1EP_1.35x3mm_P0.5mm, B.Cu at (164.5, 92.5)
- added U301: SN74LV6T17, Package_DFN_QFN:DHVQFN-14-1EP_2.5x3mm_P0.5mm_EP1x1.5mm, B.Cu at (172.0, 67.5)
- added U302: SN74LV6T17, Package_DFN_QFN:DHVQFN-14-1EP_2.5x3mm_P0.5mm_EP1x1.5mm, B.Cu at (160.5, 67.5)
- added U303: SN74LV6T17, Package_DFN_QFN:DHVQFN-14-1EP_2.5x3mm_P0.5mm_EP1x1.5mm, B.Cu at (183.5, 67.5)
- added U304: NUF6401MNT1, footprints:DFN-12-1EP_1.35x3mm_P0.5mm, B.Cu at (176.0, 67.5)
- added U305: NUF6401MNT1, footprints:DFN-12-1EP_1.35x3mm_P0.5mm, B.Cu at (164.5, 67.5)
- added U306: NUF6401MNT1, footprints:DFN-12-1EP_1.35x3mm_P0.5mm, B.Cu at (187.5, 67.5)
- added U401: TPS62A01ADRLR, Package_TO_SOT_SMD:SOT-563, F.Cu at (132.5, 59.5)
- added U402: TPS62A01ADRLR, Package_TO_SOT_SMD:SOT-563, F.Cu at (139.0, 59.5)
- added U403: TPS62A01ADRLR, Package_TO_SOT_SMD:SOT-563, F.Cu at (132.5, 65.0)
- added U404: AP2127K-2.5, Package_TO_SOT_SMD:SOT-23-5, F.Cu at (138.5, 66.0)
- added U901: TLP2362, Package_SO:SO-5-6_4.55x3.7mm_P1.27mm, F.Cu at (146.0, 59.0)
- added Y101: 25 MHz, Oscillator:Oscillator_SMD_SiT_PQFN-4Pin_2.0x1.6mm, F.Cu at (144.0, 83.5)
- U100: renamed from U6; value ECP5U_25_CABGA256 -> ECP5U_25
- moved U501 3.90 mm to (143.5, 77.5)
- renumbered J6 to J601, U9 to U501, U7 to U601
Connections:
- net /ETH.MDC renamed /Ethernet/ETH.MDC
- net /ETH.MDIO renamed /Ethernet/ETH.MDIO
- net /SPI_CLK renamed /FPGA settings & programming/SPI_CLK
- net /SPI_CS renamed /FPGA settings & programming/SPI_CS
- net /SPI_D2 renamed /FPGA settings & programming/SPI_D2
- net /SPI_D3 renamed /FPGA settings & programming/SPI_D3
- net /SPI_MISO renamed /FPGA settings & programming/SPI_MISO
- net /SPI_MOSI renamed /FPGA settings & programming/SPI_MOSI
- net /TCK renamed /FPGA settings & programming/TCK
- net /TDI renamed /FPGA settings & programming/TDI
- net /TDO renamed /FPGA settings & programming/TDO
- net /TMS renamed /FPGA settings & programming/TMS
- net /~{ETH.RST} renamed /Ethernet/ETH.~{RST}
- J601 pad 1: +3V3 -> Net-(J601-Pad1)
- J601 pad 5: unconnected-(J6-Pin_5-Pad5) -> GND
- J601 pad 9: unconnected-(J6-Pin_9-Pad9) -> GND
- U100 pad A10: /ETH.TXD0 -> /Ethernet/ETH.TXD0_{F}
- U100 pad A11: /ETH.TXD1 -> /Ethernet/ETH.TXD1_{F}
- U100 pad A12: /ETH.RXD0 -> /Ethernet/ETH.RXD0_{F}
- U100 pad A13: /ETH.RXD1 -> /Ethernet/ETH.RXD1_{F}
- U100 pad A14: /ETH.CRS_DV -> /Ethernet/ETH.CRS_DV_{F}
- U100 pad A15: /ETH.RXER -> /Ethernet/ETH.RXER_{F}
- U100 pad A3: unconnected-(U6B-PT6A/+-PadA3) -> /SYNC_IN
- U100 pad A9: /ETH.TXEN -> /Ethernet/ETH.TXEN_{F}
- U100 pad B1: /IO22 -> unconnected-(U100G-PL2A/+/HS/LDQ8-PadB1)
- U100 pad B15: /IO46 -> unconnected-(U100D-PR2B/-/S0_IN/HS/RDQ8-PadB15)
- U100 pad B16: /IO47 -> unconnected-(U100D-PR2A/+/HS/RDQ8-PadB16)
- U100 pad B2: /IO23 -> unconnected-(U100G-PL2B/-/HS/LDQ8-PadB2)
- U100 pad B4: unconnected-(U6B-PT11B/--PadB4) -> /SYNC_OUT4
- U100 pad B6: unconnected-(U6B-PT22B/--PadB6) -> /SYNC_OUT8
- U100 pad B7: unconnected-(U6B-PT27B/-/PCLKC0_1-PadB7) -> /SYNC_OUT12
- U100 pad B9: /FPGA_XI -> /Ethernet/FPGA.25MHz_CLOCK_IN
- U100 pad C1: /IO20 -> unconnected-(U100G-PL5A/+/HS/LDQ8-PadC1)
- U100 pad C15: /IO44 -> unconnected-(U100D-PR5B/-/HS/RDQ8-PadC15)
- U100 pad C16: /IO45 -> unconnected-(U100D-PR5A/+/HS/RDQ8-PadC16)
- U100 pad C2: /IO21 -> unconnected-(U100G-PL5B/-/HS/LDQ8-PadC2)
- U100 pad C4: unconnected-(U6B-PT11A/+-PadC4) -> /SYNC_OUT3
- U100 pad C6: unconnected-(U6B-PT22A/+-PadC6) -> /SYNC_OUT7
- U100 pad C7: unconnected-(U6B-PT27A/+/PCLKT0_1-PadC7) -> /SYNC_OUT11
- U100 pad C8: /ETH.REF_CLK -> /Ethernet/ETH.REF_CLK_{F}
- U100 pad D1: /IO19 -> unconnected-(U100G-PL8A/+/HS/LDQS8-PadD1)
- U100 pad D16: /IO42 -> unconnected-(U100D-PR8A/+/HS/RDQS8-PadD16)
- U100 pad D4: unconnected-(U6B-PT9B/--PadD4) -> /SYNC_OUT2
- U100 pad D5: unconnected-(U6B-PT13B/--PadD5) -> /SYNC_OUT6
- U100 pad D7: unconnected-(U6B-PT24B/-/GR_PCLK0_0-PadD7) -> /SYNC_OUT10
- U100 pad E1: /IO17 -> unconnected-(U100G-PL11D/-/LDQ8-PadE1)
- U100 pad E15: /IO41 -> unconnected-(U100D-PR8B/-/HS/RDQSN8-PadE15)
- U100 pad E16: /IO43 -> unconnected-(U100D-PR11D/-/RDQ8-PadE16)
- U100 pad E2: /IO18 -> unconnected-(U100G-PL8B/-/HS/LDQSN8-PadE2)
- U100 pad E4: unconnected-(U6B-PT9A/+-PadE4) -> /SYNC_OUT1
- U100 pad E5: unconnected-(U6B-PT13A/+-PadE5) -> /SYNC_OUT5
- U100 pad E7: unconnected-(U6B-PT24A/+/GR_PCLK0_1-PadE7) -> /SYNC_OUT9
- U100 pad F1: /IO31 -> unconnected-(U100G-PL14A/+/HS/LDQ20-PadF1)
- U100 pad F15: /IO39 -> unconnected-(U100D-PR11C/+/RDQ8-PadF15)
- U100 pad F16: /IO40 -> unconnected-(U100D-PR14A/+/HS/RDQ20-PadF16)
- U100 pad F2: /IO16 -> unconnected-(U100G-PL11C/+/LDQ8-PadF2)
- U100 pad G1: /IO29 -> unconnected-(U100G-PL20A/+/GR_PCLK7_1/HS/LDQS20-PadG1)
- U100 pad G15: /IO37 -> unconnected-(U100D-PR14B/-/HS/RDQ20-PadG15)
- U100 pad G16: /IO38 -> unconnected-(U100D-PR20A/+/GR_PCLK2_1/HS/RDQS20-PadG16)
- U100 pad G2: /IO30 -> unconnected-(U100G-PL14B/-/HS/LDQ20-PadG2)
- U100 pad H15: /IO36 -> unconnected-(U100D-PR20B/-/HS/RDQSN20-PadH15)
- U100 pad H2: /IO28 -> unconnected-(U100G-PL20B/-/HS/LDQSN20-PadH2)
- U100 pad J1: /IO27 -> unconnected-(U100G-PL23A/+/PCLKT7_1/HS/LDQ20-PadJ1)
- U100 pad J15: /IO34 -> unconnected-(U100D-PR23B/-/PCLKC2_1/HS/RDQ20-PadJ15)
- U100 pad J16: /IO35 -> unconnected-(U100D-PR23A/+/PCLKT2_1/HS/RDQ20-PadJ16)
- U100 pad J2: /IO26 -> unconnected-(U100G-PL23B/-/PCLKC7_1/HS/LDQ20-PadJ2)
- U100 pad J6: +3V3 -> +1V8
- U100 pad J7: +3V3 -> +1V8
- U100 pad K1: /IO25 -> unconnected-(U100G-PL23C/+/PCLKT7_0/LDQ20-PadK1)
- U100 pad K11: +3V3 -> +1V8
- U100 pad K15: /IO32 -> unconnected-(U100D-PR23D/-/PCLKC2_0/RDQ20-PadK15)
- U100 pad K16: /IO33 -> unconnected-(U100D-PR23C/+/PCLKT2_0/RDQ20-PadK16)
- U100 pad K2: /IO24 -> unconnected-(U100G-PL23D/-/PCLKC7_0/LDQ20-PadK2)
- U100 pad L1: /IO15 -> /Logic Channels/PORT1_I0
- U100 pad L11: +3V3 -> +1V8
- U100 pad L15: /IO54 -> /Logic Channels/PORT2_I1
- U100 pad L16: /IO55 -> /Logic Channels/PORT2_I0
- U100 pad L2: /IO14 -> /Logic Channels/PORT1_I1
- U100 pad M1: /IO13 -> /Logic Channels/PORT1_I2
- U100 pad M15: /IO52 -> /Logic Channels/PORT2_I3
- U100 pad M16: /IO53 -> /Logic Channels/PORT2_I2
- U100 pad M2: /IO12 -> /Logic Channels/PORT1_I3
- U100 pad N1: /IO11 -> /Logic Channels/PORT1_I4
- U100 pad N16: /IO51 -> /Logic Channels/PORT2_I4
- U100 pad N3: /IO08 -> /Logic Channels/PORT1_I8
- U100 pad P1: /IO09 -> /Logic Channels/PORT1_I6
- U100 pad P10: /CFG_1 -> /FPGA settings & programming/CFG_1
- U100 pad P14: /IO63 -> /Logic Channels/PORT2_I8
- U100 pad P15: /IO49 -> /Logic Channels/PORT2_I5
- U100 pad P16: /IO50 -> /Logic Channels/PORT2_I6
- U100 pad P2: /IO10 -> /Logic Channels/PORT1_I5
- U100 pad P3: /IO05 -> /Logic Channels/PORT1_I9
- U100 pad P9: /CDONE -> /FPGA settings & programming/CDONE
- U100 pad R1: /IO07 -> /Logic Channels/PORT1_I7
- U100 pad R12: /IO56 -> /Logic Channels/PORT2_I14
- U100 pad R13: /IO58 -> /Logic Channels/PORT2_I12
- U100 pad R14: /IO60 -> /Logic Channels/PORT2_I11
- U100 pad R15: /IO62 -> /Logic Channels/PORT2_I9
- U100 pad R16: /IO48 -> /Logic Channels/PORT2_I7
- U100 pad R2: /IO06 -> /Logic Channels/PORT1_I10
- U100 pad R3: /IO03 -> /Logic Channels/PORT1_I12
- U100 pad R4: /IO01 -> /Logic Channels/PORT1_I13
- U100 pad R9: /PROGRAMN -> /FPGA settings & programming/PROGRAMN
- U100 pad T13: /IO57 -> /Logic Channels/PORT2_I15
- U100 pad T14: /IO59 -> /Logic Channels/PORT2_I13
- U100 pad T15: /IO61 -> /Logic Channels/PORT2_I10
- U100 pad T2: /IO04 -> /Logic Channels/PORT1_I11
- U100 pad T3: /IO02 -> /Logic Channels/PORT1_I14
- U100 pad T4: /IO00 -> /Logic Channels/PORT1_I15
- U100 pad T9: /INITN -> /FPGA settings & programming/INITN
- U501 pad 1: /VDD_1.2 -> /Ethernet/VDD_1.2
- U501 pad 12: /ETH.RXD1 -> /Ethernet/ETH.RXD1
- U501 pad 13: /ETH.RXD0 -> /Ethernet/ETH.RXD0
- U501 pad 15: /ETH.CRS_DV -> /Ethernet/ETH.CRS_DV
- U501 pad 16: /ETH.REF_CLK -> /Ethernet/ETH.REF_CLK
- U501 pad 17: /ETH.RXER -> /Ethernet/ETH.RXER
- U501 pad 19: /ETH.TXEN -> /Ethernet/ETH.TXEN
- U501 pad 2: /VDDA_3.3 -> /Ethernet/VDDA_3.3
- U501 pad 20: /ETH.TXD0 -> /Ethernet/ETH.TXD0
- U501 pad 21: /ETH.TXD1 -> /Ethernet/ETH.TXD1
- U501 pad 23: Net-(U9-LED0/ANEN_SPEED) -> /Ethernet/LED0/ANEN_SPEED
- U501 pad 3: /RX- -> /Ethernet/RX-
- U501 pad 4: /RX+ -> /Ethernet/RX+
- U501 pad 5: /TX- -> /Ethernet/TX-
- U501 pad 6: /TX+ -> /Ethernet/TX+
- U501 pad 8: /PHY_XI -> /Ethernet/ETH.25MHz_CLOCK_IN
- U501 pad 9: Net-(U9-REXT) -> /Ethernet/REXT
Routing:
- net +3V3: track 120.7 -> 54.0 mm, vias 15 -> 12
- net +1V1: track 75.6 -> 16.9 mm
- net +2V5: track 59.9 -> 14.3 mm, vias 3 -> 4
- net /IO08: track 45.1 -> 0.00 mm, vias 1 -> 0
- net /IO09: track 40.5 -> 0.00 mm, vias 1 -> 0
- net /IO48: track 39.7 -> 0.00 mm, vias 1 -> 0
- net GND: track 87.9 -> 48.7 mm, vias 125 -> 97
- net /IO49: track 39.3 -> 0.00 mm, vias 1 -> 0
- net /IO39: track 37.4 -> 0.00 mm, vias 1 -> 0
- net /IO31: track 36.9 -> 0.00 mm, vias 1 -> 0
- net /IO10: track 36.8 -> 0.00 mm, vias 1 -> 0
- net /IO30: track 35.9 -> 0.00 mm, vias 1 -> 0
- net /IO38: track 34.4 -> 0.00 mm, vias 1 -> 0
- net /IO50: track 33.4 -> 0.00 mm, vias 1 -> 0
- net /IO37: track 31.9 -> 0.00 mm, vias 1 -> 0
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Other:
- board size 97 x 49 mm -> 76 x 57 mm
- board text removed: "Ch 0"
- board text removed: "Ch 3"
- board text removed: "RECOVERY"

Commit message: Save
Parts:
- moved R201 22.0 mm to (166.4, 102.9)
- moved R209 20.0 mm to (167.6, 102.9)
- moved R202 17.7 mm to (168.9, 102.9)
- moved R206 11.5 mm to (186.7, 102.9)
- moved R205 11.0 mm to (188.0, 102.9)
- moved R208 10.7 mm to (181.6, 102.9)
- moved R204 10.4 mm to (189.2, 102.9)
- moved R207 10.1 mm to (182.9, 102.9)
- moved R203 9.86 mm to (190.5, 102.9)
- moved R210 6.24 mm to (180.3, 102.9)
- moved R211 5.69 mm to (179.1, 102.9)
- moved R212 5.18 mm to (177.8, 102.9)
- moved R216 4.96 mm to (170.2, 102.9)
- moved R213 4.72 mm to (176.5, 102.9)
- moved R214 4.34 mm to (175.3, 102.9)
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Routing:
- net /Logic Channels/P1.6: track 0.00 -> 8.30 mm
- net /Logic Channels/P1.0: track 0.00 -> 8.30 mm
- net /Logic Channels/P2.5: track 0.00 -> 8.27 mm
- net /Logic Channels/P2.4: track 0.00 -> 7.55 mm
- net /Logic Channels/P1.7: track 0.00 -> 7.55 mm
- net /Logic Channels/P1.1: track 0.00 -> 7.55 mm
- net /Logic Channels/P2.3: track 0.00 -> 6.82 mm
- net /Logic Channels/P1.2: track 0.00 -> 6.82 mm
- net /Logic Channels/P2.2: track 0.00 -> 6.10 mm
- net /Logic Channels/P1.3: track 0.00 -> 6.10 mm
- net /Logic Channels/P2.7: track 0.00 -> 5.37 mm
- net /Logic Channels/P2.1: track 0.00 -> 5.37 mm
- net /Logic Channels/P1.4: track 0.00 -> 5.37 mm
- net /Logic Channels/P2.11: track 0.00 -> 5.28 mm
- net /Logic Channels/P1.12: track 0.00 -> 5.18 mm
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
Commit message: Save
Parts:
- C102, C103, C104, C501, C502, C503, C504, C505, C506, C507, C508, C509, C510, C601, C602, C604, C605, C606, C607, C608, C609, C610, C611, C612, C613, C701, C702, C703, C704, C801, C802, C803, C804, C805, C806, FB501, R501, R502, R505, R506, R507, R602, R603, R604: moved to B.Cu
- moved C509 112.4 mm to (154.5, 78.5), turned to 90 degrees
- moved C510 111.6 mm to (153.5, 78.5), turned to 90 degrees
- moved R502 107.3 mm to (146.9, 79.2), turned to -90 degrees
- moved C504 107.0 mm to (146.0, 77.2), turned to 180 degrees
- moved R506 106.2 mm to (145.5, 79.8), turned to 180 degrees
- moved R505 106.0 mm to (145.5, 80.9), turned to 180 degrees
- moved R507 104.5 mm to (143.5, 79.2), turned to 180 degrees
- moved R503 104.0 mm to (143.2, 73.7), turned to 90 degrees
- moved C501 103.0 mm to (145.5, 78.8)
- moved C506 102.3 mm to (141.0, 78.5)
- moved R504 102.2 mm to (141.3, 74.2), turned to 180 degrees
- moved FB501 100.3 mm to (140.0, 76.7), turned to 90 degrees
- moved C508 100.2 mm to (142.0, 74.9)
- moved C507 99.9 mm to (142.0, 75.9), turned to 180 degrees
- moved C505 99.1 mm to (141.5, 77.3), turned to 180 degrees
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Connections:
- R105 pad 1: /LED -> /Logic Channels/ACQ_LED
- U100 pad A2: /LED -> unconnected-(U100B-PT4A/+-PadA2)
- U100 pad A3: /SYNC_IN -> unconnected-(U100B-PT6A/+-PadA3)
- U100 pad B1: unconnected-(U100G-PL2A/+/HS/LDQ8-PadB1) -> /SYNC_OUT1
- U100 pad B10: unconnected-(U100C-PT44A/+-PadB10) -> /Ethernet/ETH.MDC
- U100 pad B12: /Ethernet/ETH.MDIO -> unconnected-(U100C-PT56A/+-PadB12)
- U100 pad B13: /Ethernet/ETH.MDC -> unconnected-(U100C-PT60A/+-PadB13)
- U100 pad B2: unconnected-(U100G-PL2B/-/HS/LDQ8-PadB2) -> /SYNC_OUT2
- U100 pad B4: /SYNC_OUT4 -> unconnected-(U100B-PT11B/--PadB4)
- U100 pad B6: /SYNC_OUT8 -> unconnected-(U100B-PT22B/--PadB6)
- U100 pad B7: /SYNC_OUT12 -> unconnected-(U100B-PT27B/-/PCLKC0_1-PadB7)
- U100 pad B8: unconnected-(U100C-PT35B/-/PCLKC1_0-PadB8) -> /Ethernet/ETH.MDIO
- U100 pad C1: unconnected-(U100G-PL5A/+/HS/LDQ8-PadC1) -> /SYNC_OUT5
- U100 pad C2: unconnected-(U100G-PL5B/-/HS/LDQ8-PadC2) -> /SYNC_OUT6
- U100 pad C3: unconnected-(U100G-PL2C/+/LDQ8-PadC3) -> /SYNC_OUT3
- U100 pad C4: /SYNC_OUT3 -> unconnected-(U100B-PT11A/+-PadC4)
- U100 pad C6: /SYNC_OUT7 -> unconnected-(U100B-PT22A/+-PadC6)
- U100 pad C7: /SYNC_OUT11 -> unconnected-(U100B-PT27A/+/PCLKT0_1-PadC7)
- U100 pad D3: unconnected-(U100G-PL2D/-/LDQ8-PadD3) -> /SYNC_OUT4
- U100 pad D4: /SYNC_OUT2 -> unconnected-(U100B-PT9B/--PadD4)
- U100 pad D5: /SYNC_OUT6 -> unconnected-(U100B-PT13B/--PadD5)
- U100 pad D7: /SYNC_OUT10 -> unconnected-(U100B-PT24B/-/GR_PCLK0_0-PadD7)
- U100 pad E1: unconnected-(U100G-PL11D/-/LDQ8-PadE1) -> /SYNC_OUT8
- U100 pad E4: /SYNC_OUT1 -> unconnected-(U100B-PT9A/+-PadE4)
- U100 pad E5: /SYNC_OUT5 -> unconnected-(U100B-PT13A/+-PadE5)
- U100 pad E7: /SYNC_OUT9 -> unconnected-(U100B-PT24A/+/GR_PCLK0_1-PadE7)
- U100 pad F1: unconnected-(U100G-PL14A/+/HS/LDQ20-PadF1) -> /SYNC_OUT9
- U100 pad F2: unconnected-(U100G-PL11C/+/LDQ8-PadF2) -> /SYNC_OUT7
- U100 pad G1: unconnected-(U100G-PL20A/+/GR_PCLK7_1/HS/LDQS20-PadG1) -> /SYNC_OUT11
- U100 pad G2: unconnected-(U100G-PL14B/-/HS/LDQ20-PadG2) -> /SYNC_OUT10
- U100 pad H2: unconnected-(U100G-PL20B/-/HS/LDQSN20-PadH2) -> /SYNC_OUT12
- U100 pad L13: unconnected-(U100E-PR29C/+/GR_PCLK3_1/RDQ32-PadL13) -> /Logic Channels/ACQ_LED
- U100 pad L14: unconnected-(U100E-PR32C/+/RDQ32-PadL14) -> /SYNC_IN
Routing:
- net +1V8: track 18.0 -> 185.8 mm
- net +1V1: track 16.9 -> 64.7 mm
- net +3V3: track 54.0 -> 98.9 mm, vias 12 -> 19
- net /Ethernet/LED0/ANEN_SPEED: track 0.00 -> 26.1 mm, vias 0 -> 1
- net +2V5: track 14.3 -> 40.0 mm
- net GND: track 52.2 -> 76.7 mm, vias 99 -> 127
- net /Power/5V: track 3.29 -> 27.1 mm
- net /Logic Channels/PORT1_I9: track 2.87 -> 26.2 mm
- net /Logic Channels/PORT1_I10: track 2.66 -> 24.8 mm
- net /Logic Channels/PORT2_I15: track 1.90 -> 23.2 mm
- net /SYNC_OUT1: track 0.00 -> 21.1 mm
- net /Logic Channels/PORT1_I8: track 5.37 -> 26.3 mm
- net /Logic Channels/PORT2_I14: track 3.15 -> 23.6 mm
- net /SYNC_OUT2: track 0.00 -> 20.0 mm
- net /SYNC_OUT3: track 0.00 -> 19.9 mm
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- added copper zone on In2.Cu, net +1V1
- added copper zone on In2.Cu, net +3V3
- added copper zone on F.Cu, net GND
Other:
- board text added: "SYNC IN"
- board text added: "SYNC OUT"
