File: ssla.kicad_sch (KiCad schematic)
At the start: 52 parts

Commit message: Save
Parts:
- added H101, H102, H103, H104: MountingHole_Pad, MountingHole:MountingHole_2.2mm_M2_Pad_Via, symbol Mechanical:MountingHole_Pad
- added J102, J103, J104, J105: Conn_02x10_Odd_Even, Connector_PinHeader_2.54mm:PinHeader_2x10_P2.54mm_Vertical_SMD, symbol Connector_Generic:Conn_02x10_Odd_Even
- FB101: renamed from FB?; footprint (none) -> Resistor_SMD:R_0402_1005Metric
- U104: renamed from U?; footprint Package_DFN_QFN:QFN-56-1EP_8x8mm_P0.5mm_EP4.5x5.2mm_ThermalVias_TopTented -> Package_DFN_QFN:QFN-56-1EP_8x8mm_P0.5mm_EP4.5x5.2mm
- gave numbers to parts that had none: 46
Connections:
- net D+: now also U103.3 (I/O2); no longer U103.4 (I/O2)
- net D-: now also U103.1 (I/O1); no longer U103.6 (I/O1)
- net D_N: now also U103.6 (I/O1); no longer U103.1 (I/O1)
- net D_P: now also U103.4 (I/O2); no longer U103.3 (I/O2)
- net GND: now also H101.1, H102.1, H103.1, H104.1, J102.15 (Pin_15), J102.16 (Pin_16), J102.5 (Pin_5), J102.6 (Pin_6), J103.15 (Pin_15), J103.16 (Pin_16), J103.5 (Pin_5), J103.6 (Pin_6), J104.15 (Pin_15), J104.16 (Pin_16), J104.5 (Pin_5), J104.6 (Pin_6), J105.15 (Pin_15), J105.16 (Pin_16), J105.5 (Pin_5), J105.6 (Pin_6)
- net IO00: now also U105.A11 (IOT_168), J102.1 (Pin_1)
- net IO01: now also U105.A10 (IOT_170), J102.3 (Pin_3)
- net IO02: now also U105.C9 (IOT_172), J102.7 (Pin_7)
- net IO03: now also U105.B9 (IOT_174), J102.9 (Pin_9)
- net IO04: now also U105.B8 (IOT_177), J102.11 (Pin_11)
- net IO05: now also U105.A9 (IOT_178), J102.13 (Pin_13)
- net IO06: now also U105.C8 (IOT_179), J102.17 (Pin_17)
- net IO07: now also U105.D7 (IOT_181), J102.19 (Pin_19)
- net IO08: now also U105.A8 (IOT_190), J102.2 (Pin_2)
- net IO09: now also U105.C7 (IOT_191), J102.4 (Pin_4)
- net IO10: now also U105.A7 (IOT_192), J102.8 (Pin_8)
- net IO11: now also U105.B7 (IOT_197_GBIN1), J102.10 (Pin_10)
- net IO12: now also U105.B6 (IOT_198_GBIN0), J102.12 (Pin_12)
- net IO13: now also U105.A6 (IOT_206), J102.14 (Pin_14)
- net IO14: now also U105.A5 (IOT_207), J102.18 (Pin_18)
- net IO15: now also U105.B5 (IOT_208), J102.20 (Pin_20)
- net IO16: now also U105.A4 (IOT_211), J103.1 (Pin_1)
- net IO17: now also U105.D5 (IOT_212), J103.3 (Pin_3)
- net IO18: now also U105.B4 (IOT_219), J103.7 (Pin_7)
- net IO19: now also U105.B3 (IOT_221), J103.9 (Pin_9)
- net IO20: now also U105.A2 (IOT_222), J103.11 (Pin_11)
- net IO21: now also U105.A3 (IOT_223), J103.13 (Pin_13)
- net IO22: now also U105.A1 (IOT_225), J103.17 (Pin_17)
- net IO23: now also U105.J11 (IOR_114), J103.19 (Pin_19)
- net IO24: now also U105.K11 (IOR_115), J103.2 (Pin_2)
- net IO25: now also U105.H10 (IOR_116), J103.4 (Pin_4)
- net IO26: now also U105.J10 (IOR_117), J103.8 (Pin_8)
- net IO27: now also U105.G8 (IOR_118), J103.10 (Pin_10)
- net IO28: now also U105.H11 (IOR_119), J103.12 (Pin_12)
- net IO29: now also U105.G10 (IOR_120), J103.14 (Pin_14)
- net IO30: now also U105.G9 (IOR_128), J103.18 (Pin_18)
- net IO31: now also U105.G11 (IOR_129), J103.20 (Pin_20)
- net IO32: now also U105.F10 (IOR_136), J104.1 (Pin_1)
- net IO33: now also U105.F9 (IOR_137), J104.3 (Pin_3)
- net IO34: now also U105.F11 (IOR_140_GBIN3), J104.7 (Pin_7)
- net IO35: now also U105.E10 (IOR_141_GBIN2), J104.9 (Pin_9)
- net IO36: now also U105.E9 (IOR_144), J104.11 (Pin_11)
- net IO37: now also U105.E8 (IOR_146), J104.13 (Pin_13)
- net IO38: now also U105.D9 (IOR_147), J104.17 (Pin_17)
- net IO39: now also U105.E11 (IOR_148), J104.19 (Pin_19)
- net IO40: now also U105.D11 (IOR_152), J104.2 (Pin_2)
- net IO41: now also U105.D10 (IOR_154), J104.4 (Pin_4)
- net IO42: now also U105.C11 (IOR_160), J104.8 (Pin_8)
- net IO43: now also U105.B11 (IOR_161), J104.10 (Pin_10)
- net IO44: now also U105.B1 (IOL_2A), J104.12 (Pin_12)
- net IO45: now also U105.B2 (IOL_2B), J104.14 (Pin_14)
- net IO46: now also U105.C4 (IOL_4A), J104.18 (Pin_18)
- net IO47: now also U105.C3 (IOL_4B), J104.20 (Pin_20)
- net IO48: now also U105.C2 (IOL_5A), J105.1 (Pin_1)
- net IO49: now also U105.C1 (IOL_5B), J105.3 (Pin_3)
- net IO50: now also U105.E1 (IOL_8A), J105.7 (Pin_7)
- net IO51: now also U105.D1 (IOL_8B), J105.9 (Pin_9)
- net IO52: now also U105.D2 (IOL_9A), J105.11 (Pin_11)
- net IO53: now also U105.D3 (IOL_9B), J105.13 (Pin_13)
- net IO54: now also U105.E2 (IOL_10A), J105.17 (Pin_17)
- net IO55: now also U105.E3 (IOL_10B), J105.19 (Pin_19)
- net IO56: now also U105.F1 (IOL_12A), J105.2 (Pin_2)
- net IO57: now also U105.F2 (IOL_12B), J105.4 (Pin_4)
- net IO58: now also U105.F4 (IOL_13A), J105.8 (Pin_8)
- net IO59: now also U105.F3 (IOL_13B_GBIN7), J105.10 (Pin_10)
- net IO60: now also U105.G1 (IOL_14A_GBIN6), J105.12 (Pin_12)
- net IO61: now also U105.G2 (IOL_14B), J105.14 (Pin_14)
- net IO62: now also U105.G3 (IOL_17A), J105.18 (Pin_18)
- net IO63: now also U105.H3 (IOL_17B), J105.20 (Pin_20)
- net PB1/FD1: now reaches U105.J9 (IOB_106_SDI)
- net PB1/FD1: now also U104.19 (PB1/FD1)
- net PB3/FD3: now reaches U105.K10 (IOB_108_SS)
- net PB3/FD3: now also U104.21 (PB3/FD3)
- net PB0/FD0: now reaches U105.K9 (IOB_105_SDO)
- net PB0/FD0: now also U104.18 (PB0/FD0)
- net PB2/FD2: now reaches U105.L10 (IOB_107_SCK)
- net PB2/FD2: now also U104.20 (PB2/FD2)
- net RDY0/SLRD: now reaches U104.1 (RDY0/SLRD)
- net RDY0/SLRD: now also U105.H7 (IOB_87)
- net IFCLK: now reaches U104.13 (IFCLK)
- net IFCLK: now also U105.L5 (IOB_81_GBIN5)
- net RDY1/SLWR: now reaches U104.2 (RDY1/SLWR)
- net RDY1/SLWR: now also U105.K7 (IOB_89)
- net PB4/FD4: now reaches U104.22 (PB4/FD4)
- net PB4/FD4: now also U105.J8 (IOB_91)
- net PB5/FD5: now reaches U104.23 (PB5/FD5)
- net PB5/FD5: now also U105.L7 (IOB_94)
- net PB6/FD6: now reaches U104.24 (PB6/FD6)
- net PB6/FD6: now also U105.L8 (IOB_103_CBSEL0)
- net PB7/FD7: now reaches U104.25 (PB7/FD7)
- net PB7/FD7: now also U105.H9 (IOB_104_CBSEL1)
- net CTL0/FLAGA: now reaches U104.29 (CTL0/FLAGA)
- net CTL1/FLAGB: now reaches U104.30 (CTL1/FLAGB)
- net CTL2/FLAGC: now reaches U104.31 (CTL2/FLAGC)
- net PA0/~{INT0}: now reaches U104.33 (PA0/~{INT0})
- net PA1/~{INT1}: now reaches U104.34 (PA1/~{INT1})
- net PA2/SLOE: now reaches U104.35 (PA2/SLOE)
- net PA3/WU2: now reaches U104.36 (PA3/WU2)
- net PA4/FIOADDR0: now reaches U104.37 (PA4/FIOADDR0)
- net PA5/FIOADDR1: now reaches U104.38 (PA5/FIOADDR1)
- net PA6/PKTEND: now reaches U104.39 (PA6/PKTEND)
- net PA7/FLAGD/~{SLCS}: now reaches U104.40 (PA7/FLAGD/~{SLCS})
- net PD0/FD8: now reaches U104.45 (PD0/FD8)
- net PD1/FD9: now reaches U104.46 (PD1/FD9)
- net PD2/FD10: now reaches U104.47 (PD2/FD10)
- net PD3/FD11: now reaches U104.48 (PD3/FD11)
- net PD4/FD12: now reaches U104.49 (PD4/FD12)
- net PD5/FD13: now reaches U104.50 (PD5/FD13)
- net PD6/FD14: now reaches U104.51 (PD6/FD14)
- net PD7/FD15: now reaches U104.52 (PD7/FD15)
- net CLKOUT: now reaches U104.54 (CLKOUT)
- net CLKOUT: now also U105.K6 (IOB_82_GBIN4)

Commit message: 0 unrouted
Parts:
- added C15, C28, C31, C36: 0.1u, Capacitor_SMD:C_0402_1005Metric, symbol Device:C_Small
- added D1, D10, D11, D12, D13, D14, D15, D16, D17, D18, D19, D2, D20, D21, D22, D23, D24, D25, D26, D27, D28, D29, D3, D30, D31, D32, D33, D34, D35, D36, D37, D38, D39, D4, D40, D41, D42, D43, D44, D45, D46, D47, D48, D49, D5, D50, D51, D52, D53, D54, D55, D56, D57, D58, D59, D6, D60, D61, D62, D63, D64, D7, D8, D9: D_TVS_Small, Diode_SMD:D_SOD-923, symbol Device:D_TVS_Small
- added J6: Conn_ARM_JTAG_SWD_10, Connector_PinHeader_1.27mm:PinHeader_2x05_P1.27mm_Vertical_SMD, symbol Connector:Conn_ARM_JTAG_SWD_10
- added R10, R45, R78, R79, R9: 10k, Resistor_SMD:R_0402_1005Metric, symbol Device:R_Small
- added R11, R12, R13, R14, R15, R16, R17, R18, R19, R20, R21, R22, R23, R24, R25, R26, R27, R28, R29, R30, R31, R32, R33, R34, R35, R36, R37, R38, R39, R40, R41, R42, R46, R47, R48, R49, R50, R51, R52, R53, R54, R55, R56, R57, R58, R59, R60, R61, R62, R63, R64, R65, R66, R67, R68, R69, R70, R71, R72, R73, R74, R75, R76, R77: 100, Resistor_SMD:R_0402_1005Metric, symbol Device:R_Small
- added R4: 0, Resistor_SMD:R_0402_1005Metric, symbol Device:R_Small
- added R8: 100k, Resistor_SMD:R_0402_1005Metric, symbol Device:R_Small
- added TP11, TP12: TestPoint_Small, TestPoint:TestPoint_Pad_D1.0mm, symbol Connector:TestPoint_Small
- added U3: BL24C256A, Package_SO:TSSOP-8_4.4x3mm_P0.65mm, symbol Memory_EEPROM:CAT24C256
- added U7: W25Q16JVUXIQ, Package_SON:Winbond_USON-8-1EP_3x2mm_P0.5mm_EP0.2x1.6mm, symbol flash:W25Q16JVSS
- J2: renamed from J102; footprint Connector_PinHeader_2.54mm:PinHeader_2x10_P2.54mm_Vertical_SMD -> Connector_IDC:IDC-Header_2x10_P2.54mm_Vertical_SMD
- J3: renamed from J103; footprint Connector_PinHeader_2.54mm:PinHeader_2x10_P2.54mm_Vertical_SMD -> Connector_IDC:IDC-Header_2x10_P2.54mm_Vertical_SMD
- J4: renamed from J104; footprint Connector_PinHeader_2.54mm:PinHeader_2x10_P2.54mm_Vertical_SMD -> Connector_IDC:IDC-Header_2x10_P2.54mm_Vertical_SMD
- J5: renamed from J105; footprint Connector_PinHeader_2.54mm:PinHeader_2x10_P2.54mm_Vertical_SMD -> Connector_IDC:IDC-Header_2x10_P2.54mm_Vertical_SMD
- R6: renamed from R105; value 2.2k -> 100k
- renumbered C101 to C1, C110 to C10, C111 to C11, C112 to C12, C113 to C13, C114 to C14, C115 to C16, C116 to C17, C117 to C18, C118 to C19, C102 to C2, C119 to C20, C120 to C21, C121 to C22, C122 to C23, C123 to C24, C124 to C25, C125 to C26, C126 to C27, C127 to C29, C103 to C3, C128 to C30, C129 to C32, C130 to C33, C131 to C34, C132 to C35, C104 to C4, C105 to C5, C106 to C6, C107 to C7, C108 to C8, C109 to C9, FB101 to FB1, H101 to H1, H102 to H2, H103 to H3, H104 to H4, J101 to J1, R101 to R1, R102 to R2, R103 to R3, R107 to R43, R108 to R44, R104 to R5, R106 to R7, U101 to U1, U102 to U2, U103 to U4, U104 to U5, U105 to U6, Y101 to Y1
Connections:
- net PA1/~{INT1} is gone; now on net ~{CRESET}: U5.34 (PA1/~{INT1})
- net PA3/WU2 is gone; now on net CDONE: U5.36 (PA3/WU2)
- net +3V3: now also C15.1, C28.1, C31.1, C36.1, J6.1 (VTref), R10.2, R4.1, R45.2, R78.2, R79.2, R8.2, R9.2, U3.1 (A0), U3.8 (VCC), U7.8 (VCC)
- net CLKOUT: now also U6.L5 (IOB_81_GBIN5), TP12.1; no longer U6.K6 (IOB_82_GBIN4)
- net CTL0/FLAGA: now also U6.H7 (IOB_87)
- net CTL1/FLAGB: now also U6.H9 (IOB_104_CBSEL1)
- net GND: now also C15.2, C28.2, C31.2, C36.2, D1.1 (A1), D10.1 (A1), D11.1 (A1), D12.1 (A1), D13.1 (A1), D14.1 (A1), D15.1 (A1), D16.1 (A1), D17.1 (A1), D18.1 (A1), D19.1 (A1), D2.1 (A1), D20.1 (A1), D21.1 (A1), D22.1 (A1), D23.1 (A1), D24.1 (A1), D25.1 (A1), D26.1 (A1), D27.1 (A1), D28.1 (A1), D29.1 (A1), D3.1 (A1), D30.1 (A1), D31.1 (A1), D32.1 (A1), D33.1 (A1), D34.1 (A1), D35.1 (A1), D36.1 (A1), D37.1 (A1), D38.1 (A1), D39.1 (A1), D4.1 (A1), D40.1 (A1), D41.1 (A1), D42.1 (A1), D43.1 (A1), D44.1 (A1), D45.1 (A1), D46.1 (A1), D47.1 (A1), D48.1 (A1), D49.1 (A1), D5.1 (A1), D50.1 (A1), D51.1 (A1), D52.1 (A1), D53.1 (A1), D54.1 (A1), D55.1 (A1), D56.1 (A1), D57.1 (A1), D58.1 (A1), D59.1 (A1), D6.1 (A1), D60.1 (A1), D61.1 (A1), D62.1 (A1), D63.1 (A1), D64.1 (A1), D7.1 (A1), D8.1 (A1), D9.1 (A1), J6.3 (GND), J6.5 (GND), J6.9 (GNDDetect), U3.4 (GND), U7.4 (GND), U7.9 (GND)
- net IFCLK: now also U6.K6 (IOB_82_GBIN4), TP11.1; no longer U6.L5 (IOB_81_GBIN5)
- net IO00: now also U6.A5 (IOT_207), D1.2 (A2), R11.2; no longer J2.1 (Pin_1), U6.A11 (IOT_168)
- net IO01: now also U6.A6 (IOT_206), D2.2 (A2), R12.2; no longer J2.3 (Pin_3), U6.A10 (IOT_170)
- net IO02: now also U6.A7 (IOT_192), D3.2 (A2), R13.2; no longer J2.7 (Pin_7), U6.C9 (IOT_172)
- net IO03: now also U6.A8 (IOT_190), D4.2 (A2), R14.2; no longer J2.9 (Pin_9), U6.B9 (IOT_174)
- net IO04: now also D5.2 (A2), R15.2; no longer J2.11 (Pin_11)
- net IO05: now also D6.2 (A2), R16.2; no longer J2.13 (Pin_13)
- net IO06: now also U6.B9 (IOT_174), D7.2 (A2), R17.2; no longer J2.17 (Pin_17), U6.C8 (IOT_179)
- net IO07: now also U6.A10 (IOT_170), D8.2 (A2), R18.2; no longer J2.19 (Pin_19), U6.D7 (IOT_181)
- net IO08: now also U6.B5 (IOT_208), D9.2 (A2), R46.2; no longer J2.2 (Pin_2), U6.A8 (IOT_190)
- net IO09: now also U6.D7 (IOT_181), D10.2 (A2), R47.2; no longer J2.4 (Pin_4), U6.C7 (IOT_191)
- net IO10: now also U6.C7 (IOT_191), D11.2 (A2), R48.2; no longer J2.8 (Pin_8), U6.A7 (IOT_192)
- net IO11: now also U6.C9 (IOT_172), D12.2 (A2), R49.2; no longer J2.10 (Pin_10), U6.B7 (IOT_197_GBIN1)
- net IO12: now also U6.A11 (IOT_168), D13.2 (A2), R50.2; no longer J2.12 (Pin_12), U6.B6 (IOT_198_GBIN0)
- net IO13: now also U6.B11 (IOR_161), D14.2 (A2), R51.2; no longer J2.14 (Pin_14), U6.A6 (IOT_206)
- net IO14: now also U6.C11 (IOR_160), D15.2 (A2), R52.2; no longer J2.18 (Pin_18), U6.A5 (IOT_207)
- net IO15: now also U6.D9 (IOR_147), D16.2 (A2), R53.2; no longer J2.20 (Pin_20), U6.B5 (IOT_208)
- net IO16: now also U6.E9 (IOR_144), D17.2 (A2), R19.2; no longer J3.1 (Pin_1), U6.A4 (IOT_211)
- net IO17: now also U6.E8 (IOR_146), D18.2 (A2), R20.2; no longer J3.3 (Pin_3), U6.D5 (IOT_212)
- net IO18: now also U6.G8 (IOR_118), D19.2 (A2), R21.2; no longer J3.7 (Pin_7), U6.B4 (IOT_219)
- net IO19: now also U6.G9 (IOR_128), D20.2 (A2), R22.2; no longer J3.9 (Pin_9), U6.B3 (IOT_221)
- net IO20: now also U6.J10 (IOR_117), D21.2 (A2), R23.2; no longer J3.11 (Pin_11), U6.A2 (IOT_222)
- net IO21: now also U6.K11 (IOR_115), D22.2 (A2), R24.2; no longer J3.13 (Pin_13), U6.A3 (IOT_223)
- net IO22: now also U6.F10 (IOR_136), D23.2 (A2), R25.2; no longer J3.17 (Pin_17), U6.A1 (IOT_225)
- net IO23: now also U6.F9 (IOR_137), D24.2 (A2), R26.2; no longer J3.19 (Pin_19), U6.J11 (IOR_114)
- net IO24: now also U6.G11 (IOR_129), D25.2 (A2), R54.2; no longer J3.2 (Pin_2), U6.K11 (IOR_115)
- net IO25: now also U6.G10 (IOR_120), D26.2 (A2), R55.2; no longer J3.4 (Pin_4), U6.H10 (IOR_116)
- net IO26: now also U6.H11 (IOR_119), D27.2 (A2), R56.2; no longer J3.8 (Pin_8), U6.J10 (IOR_117)
- net IO27: now also U6.H10 (IOR_116), D28.2 (A2), R57.2; no longer J3.10 (Pin_10), U6.G8 (IOR_118)
- net IO28: now also U6.J11 (IOR_114), D29.2 (A2), R58.2; no longer J3.12 (Pin_12), U6.H11 (IOR_119)
- net IO29: now also U6.D11 (IOR_152), D30.2 (A2), R59.2; no longer J3.14 (Pin_14), U6.G10 (IOR_120)
- net IO30: now also U6.D10 (IOR_154), D31.2 (A2), R60.2; no longer J3.18 (Pin_18), U6.G9 (IOR_128)
- net IO31: now also U6.E11 (IOR_148), D32.2 (A2), R61.2; no longer J3.20 (Pin_20), U6.G11 (IOR_129)
- net IO32: now also U6.E1 (IOL_8A), D33.2 (A2), R27.2; no longer J4.1 (Pin_1), U6.F10 (IOR_136)
- net IO33: now also U6.F2 (IOL_12B), D34.2 (A2), R28.2; no longer J4.3 (Pin_3), U6.F9 (IOR_137)
- net IO34: now also U6.F1 (IOL_12A), D35.2 (A2), R29.2; no longer J4.7 (Pin_7), U6.F11 (IOR_140_GBIN3)
- net IO35: now also U6.G2 (IOL_14B), D36.2 (A2), R30.2; no longer J4.9 (Pin_9), U6.E10 (IOR_141_GBIN2)
- net IO36: now also U6.H2 (IOL_18B), D37.2 (A2), R31.2; no longer J4.11 (Pin_11), U6.E9 (IOR_144)
- net IO37: now also U6.J1 (IOL_23A), D38.2 (A2), R32.2; no longer J4.13 (Pin_13), U6.E8 (IOR_146)
- net IO38: now also U6.K2 (IOL_25A), D39.2 (A2), R33.2; no longer J4.17 (Pin_17), U6.D9 (IOR_147)
- net IO39: now also U6.K1 (IOL_23B), D40.2 (A2), R34.2; no longer J4.19 (Pin_19), U6.E11 (IOR_148)
- net IO40: now also U6.H1 (IOL_18A), D41.2 (A2), R62.2; no longer J4.2 (Pin_2), U6.D11 (IOR_152)
- net IO41: now also U6.J2 (IOL_25B), D42.2 (A2), R63.2; no longer J4.4 (Pin_4), U6.D10 (IOR_154)
- net IO42: now also U6.C4 (IOL_4A), D43.2 (A2), R64.2; no longer J4.8 (Pin_8), U6.C11 (IOR_160)
- net IO43: now also U6.D3 (IOL_9B), D44.2 (A2), R65.2; no longer J4.10 (Pin_10), U6.B11 (IOR_161)
- net IO44: now also U6.E3 (IOL_10B), D45.2 (A2), R66.2; no longer J4.12 (Pin_12), U6.B1 (IOL_2A)
- net IO45: now also U6.F4 (IOL_13A), D46.2 (A2), R67.2; no longer J4.14 (Pin_14), U6.B2 (IOL_2B)
- net IO46: now also U6.G3 (IOL_17A), D47.2 (A2), R68.2; no longer J4.18 (Pin_18), U6.C4 (IOL_4A)
- net IO47: now also U6.H3 (IOL_17B), D48.2 (A2), R69.2; no longer J4.20 (Pin_20), U6.C3 (IOL_4B)
- net IO48: now also U6.A4 (IOT_211), D49.2 (A2), R35.2; no longer J5.1 (Pin_1), U6.C2 (IOL_5A)
- net IO49: now also U6.A3 (IOT_223), D50.2 (A2), R36.2; no longer J5.3 (Pin_3), U6.C1 (IOL_5B)
- net IO50: now also U6.A2 (IOT_222), D51.2 (A2), R37.2; no longer J5.7 (Pin_7), U6.E1 (IOL_8A)
- net IO51: now also U6.B2 (IOL_2B), D52.2 (A2), R38.2; no longer J5.9 (Pin_9), U6.D1 (IOL_8B)
- net IO52: now also U6.C2 (IOL_5A), D53.2 (A2), R39.2; no longer J5.11 (Pin_11), U6.D2 (IOL_9A)
- net IO53: now also U6.D2 (IOL_9A), D54.2 (A2), R40.2; no longer J5.13 (Pin_13), U6.D3 (IOL_9B)
- net IO54: now also U6.D1 (IOL_8B), D55.2 (A2), R41.2; no longer J5.17 (Pin_17), U6.E2 (IOL_10A)
- net IO55: now also U6.E2 (IOL_10A), D56.2 (A2), R42.2; no longer J5.19 (Pin_19), U6.E3 (IOL_10B)
- net IO56: now also U6.B4 (IOT_219), D57.2 (A2), R70.2; no longer J5.2 (Pin_2), U6.F1 (IOL_12A)
- net IO57: now also U6.B3 (IOT_221), D58.2 (A2), R71.2; no longer J5.4 (Pin_4), U6.F2 (IOL_12B)
- net IO58: now also U6.C3 (IOL_4B), D59.2 (A2), R72.2; no longer J5.8 (Pin_8), U6.F4 (IOL_13A)
- net IO59: now also U6.A1 (IOT_225), D60.2 (A2), R73.2; no longer J5.10 (Pin_10), U6.F3 (IOL_13B_GBIN7)
- net IO60: now also U6.B1 (IOL_2A), D61.2 (A2), R74.2; no longer J5.12 (Pin_12), U6.G1 (IOL_14A_GBIN6)
- net IO61: now also U6.C1 (IOL_5B), D62.2 (A2), R75.2; no longer J5.14 (Pin_14), U6.G2 (IOL_14B)
- net IO62: now also U6.C8 (IOT_179), D63.2 (A2), R76.2; no longer J5.18 (Pin_18), U6.G3 (IOL_17A)
- net IO63: now also U6.D5 (IOT_212), D64.2 (A2), R77.2; no longer J5.20 (Pin_20), U6.H3 (IOL_17B)
- net PA0/~{INT0}: now also U6.J7 (IOB_86), R8.1
- net PA2/SLOE: now also U6.J8 (IOB_91)
- net PA4/FIOADDR0: now also U6.J5 (IOB_78)
- net PA5/FIOADDR1: now also U6.J3 (IOB_57)
- net PA6/PKTEND: now also U6.J4 (IOB_64)
- net PB0/FD0: now also U6.L8 (IOB_103_CBSEL0); no longer U6.K9 (IOB_105_SDO)
- net PB1/FD1: now also U6.K7 (IOB_89); no longer U6.J9 (IOB_106_SDI)
- net PB2/FD2: now also U6.L7 (IOB_94); no longer U6.L10 (IOB_107_SCK)
- net PB3/FD3: now also U6.K5 (IOB_79); no longer U6.K10 (IOB_108_SS)
- net PB4/FD4: now also U6.L4 (IOB_72); no longer U6.J8 (IOB_91)
- net PB5/FD5: now also U6.K4 (IOB_73); no longer U6.L7 (IOB_94)
- net PB6/FD6: now also U6.L3 (IOB_71); no longer U6.L8 (IOB_103_CBSEL0)
- net PB7/FD7: now also U6.K3 (IOB_63); no longer U6.H9 (IOB_104_CBSEL1)
- net RDY0/SLRD: now also U6.L2 (IOB_61); no longer U6.H7 (IOB_87)
- net RDY1/SLWR: now also U6.L1 (IOB_56); no longer U6.K7 (IOB_89)
- net SCL: now also U3.6 (SCL)
- net SDA: now also U3.5 (SDA)
- net CDONE: now reaches U6.K8 (CDONE)
- net CDONE: now also R10.1
- net ~{CRESET}: now reaches U6.L9 (~{CRESET})
- net ~{CRESET}: now also J6.10 (~{RESET}), R9.1
- net CTL2/FLAGC: no longer names the net of U5.31 (CTL2/FLAGC)
- net PA7/FLAGD/~{SLCS}: no longer names the net of U5.40 (PA7/FLAGD/~{SLCS})
- net PD0/FD8: no longer names the net of U5.45 (PD0/FD8)
- net PD1/FD9: no longer names the net of U5.46 (PD1/FD9)
- net PD2/FD10: no longer names the net of U5.47 (PD2/FD10)
- net PD3/FD11: no longer names the net of U5.48 (PD3/FD11)
- net PD4/FD12: no longer names the net of U5.49 (PD4/FD12)
- net PD5/FD13: no longer names the net of U5.50 (PD5/FD13)
- net PD6/FD14: no longer names the net of U5.51 (PD6/FD14)
- net PD7/FD15: no longer names the net of U5.52 (PD7/FD15)
- new net: J5.4 (Pin_4), R71.1
- new net: J4.8 (Pin_8), R64.1
- new net: J4.12 (Pin_12), R66.1
- new net: J3.12 (Pin_12), R58.1
- new net: J3.18 (Pin_18), R60.1
- new net: J5.14 (Pin_14), R75.1
- new net: J2.17 (Pin_17), R17.1
- new net: J2.10 (Pin_10), R49.1
- new net: J4.19 (Pin_19), R34.1
- new net: J2.7 (Pin_7), R13.1
- new net: J3.3 (Pin_3), R20.1
- new net: J5.20 (Pin_20), R77.1
- new net: J5.13 (Pin_13), R40.1
- new net: J2.4 (Pin_4), R47.1
- new net: J2.9 (Pin_9), R14.1
- new net: J2.2 (Pin_2), R46.1
- new net: J5.7 (Pin_7), R37.1
- new net: J5.1 (Pin_1), R35.1
- new net: R4.2, U3.2 (A1)
- new net: J5.11 (Pin_11), R39.1
- new net: J5.10 (Pin_10), R73.1
- new net: J2.20 (Pin_20), R53.1
- new net: J3.8 (Pin_8), R56.1
- new net: J3.1 (Pin_1), R19.1
- new net: J4.11 (Pin_11), R31.1
- new net: J5.12 (Pin_12), R74.1
- new net: J5.17 (Pin_17), R41.1
- new net: J5.18 (Pin_18), R76.1
- new net: J5.19 (Pin_19), R42.1
- new net: J5.2 (Pin_2), R70.1
- new net: J5.3 (Pin_3), R36.1
- new net: J5.8 (Pin_8), R72.1
- new net: J5.9 (Pin_9), R38.1
- new net: R78.1, U7.7 (IO3)
- new net: J2.11 (Pin_11), R15.1
- new net: J4.10 (Pin_10), R65.1
- new net: J3.11 (Pin_11), R23.1
- new net: J3.10 (Pin_10), R57.1
- new net: J3.13 (Pin_13), R24.1
- new net: J3.14 (Pin_14), R59.1
- new net: J3.17 (Pin_17), R25.1
- new net: J3.19 (Pin_19), R26.1
- new net: J3.2 (Pin_2), R54.1
- new net: J3.20 (Pin_20), R61.1
- new net: J3.4 (Pin_4), R55.1
- new net: J3.7 (Pin_7), R21.1
- new net: J3.9 (Pin_9), R22.1
- new net: J2.18 (Pin_18), R52.1
- new net: J4.4 (Pin_4), R63.1
- new net: J4.3 (Pin_3), R28.1
- new net: J2.1 (Pin_1), R11.1
- new net: R79.1, U7.3 (IO2)
- new net: J2.3 (Pin_3), R12.1
- new net: J4.20 (Pin_20), R69.1
- new net: J4.14 (Pin_14), R67.1
- new net: J2.14 (Pin_14), R51.1
- new net: J4.13 (Pin_13), R32.1
- new net: J4.17 (Pin_17), R33.1
- new net: J4.7 (Pin_7), R29.1
- new net: J2.12 (Pin_12), R50.1
- new net: J2.19 (Pin_19), R18.1
- new net: J2.13 (Pin_13), R16.1
- new net: J4.9 (Pin_9), R30.1
- new net: J2.8 (Pin_8), R48.1
- new net: J4.18 (Pin_18), R68.1
- new net: J4.2 (Pin_2), R62.1
- new net: J4.1 (Pin_1), R27.1
- new net IOB_105_SDO: J6.6 (SWO/TDO), U6.K9 (IOB_105_SDO), U7.5 (DI(IO0))
- new net IOB_106_SDI: J6.8 (NC/TDI), U6.J9 (IOB_106_SDI), U7.2 (DO(IO1))
- new net IOB_107_SCK: J6.4 (SWCLK/TCK), U6.L10 (IOB_107_SCK), U7.6 (CLK)
- new net IOB_108_SS: J6.2 (SWDIO/TMS), R45.1, U6.K10 (IOB_108_SS), U7.1 (~{CS})
- no-connect marks 3 -> 22
Other:
- moved on the sheet: C18

Commit message: LCSC part numbers, started moving to through-hole IDC connector
Parts:
- C1, C16, C17, C2, C3, C34, C35, C4, C8: LCSC (none) -> C23733
- C10, C11, C12, C13, C14, C15, C18, C21, C22, C23, C24, C25, C26, C27, C28, C29, C30, C31, C32, C33, C36, C5, C6, C7, C9: LCSC (none) -> C307331
- C19, C20: value 10p -> 12p; LCSC (none) -> C1547
- FB1: LCSC (none) -> C491490
- J2: footprint Connector_IDC:IDC-Header_2x10_P2.54mm_Vertical_SMD -> Connector_IDC:IDC-Header_2x10_P2.54mm_Vertical; LCSC (none) -> C221051
- R1, R2: LCSC (none) -> C25905
- R10, R45, R78, R79, R9: LCSC (none) -> C25744
- R11, R12, R13, R14, R15, R16, R17, R18, R19, R20, R21, R22, R23, R24, R25, R26, R27, R28, R29, R30, R31, R32, R33, R34, R35, R36, R37, R38, R39, R40, R41, R42, R43, R44, R46, R47, R48, R49, R50, R51, R52, R53, R54, R55, R56, R57, R58, R59, R60, R61, R62, R63, R64, R65, R66, R67, R68, R69, R70, R71, R72, R73, R74, R75, R76, R77: LCSC (none) -> C25076
- R3, R6, R8: LCSC (none) -> C258090
- R5, R7: LCSC (none) -> C25933
- U1: LCSC (none) -> C2861750; MFPN (none) -> TLV75533PDRV
- U2: LCSC (none) -> C2866903; MFPN (none) -> TLV75512PDRV
- U4: MFPN (none) -> USBLC6-2P6
- U5: LCSC (none) -> C14912; MFPN (none) -> CY7C68013A-56LTXC
- U6: LCSC (none) -> C1521843
- Y1: LCSC (none) -> C2689430; MFPN (none) -> E1SB24E000007E

Commit message: Save
Parts:
- J3, J4, J5: footprint Connector_IDC:IDC-Header_2x10_P2.54mm_Vertical_SMD -> Connector_IDC:IDC-Header_2x10_P2.54mm_Vertical; LCSC (none) -> C221051
Changed lines of the file:
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@@
 			)
 		)
-		(property "Footprint" "Connector_IDC:IDC-Header_2x10_P2.54mm_Vertical_SMD"
+		(property "Footprint" "Connector_IDC:IDC-Header_2x10_P2.54mm_Vertical"
 			(at 273.05 133.35 0)
 			(effects
@@
 			)
 		)
-		(property "LCSC" ""
+		(property "LCSC" "C221051"
 			(at 273.05 133.35 0)
 			(effects
@@
 			)
 		)
-		(property "Footprint" "Connector_IDC:IDC-Header_2x10_P2.54mm_Vertical_SMD"
+		(property "Footprint" "Connector_IDC:IDC-Header_2x10_P2.54mm_Vertical"
 			(at 273.05 72.39 0)
 			(effects
@@
 			)
 		)
-		(property "LCSC" ""
+		(property "LCSC" "C221051"
 			(at 273.05 72.39 0)
 			(effects
@@
 			)
 		)
-		(property "Footprint" "Connector_IDC:IDC-Header_2x10_P2.54mm_Vertical_SMD"
+		(property "Footprint" "Connector_IDC:IDC-Header_2x10_P2.54mm_Vertical"
 			(at 273.05 102.87 0)
 			(effects
@@
 			)
 		)
-		(property "LCSC" ""
+		(property "LCSC" "C221051"
 			(at 273.05 102.87 0)
 			(effects

Commit message: Save
Parts:
- U7: symbol flash:W25Q16JVSS -> Memory_Flash:W25Q32JVZP
Connections:
- net IO24: now also U6.J11 (IOR_114); no longer U6.G11 (IOR_129)
- net IO25: now also U6.H10 (IOR_116); no longer U6.G10 (IOR_120)
- net IO27: now also U6.G10 (IOR_120); no longer U6.H10 (IOR_116)
- net IO28: now also U6.G11 (IOR_129); no longer U6.J11 (IOR_114)
- no-connect marks 22 -> 21
Other:
- moved on the sheet: C36, D1, D10, D11, D12, D13, D14, D15, D16, D17, D18, D19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

Commit message: Started move to ECP5
Parts:
- removed J6: Conn_ARM_JTAG_SWD_10, Connector_PinHeader_1.27mm:PinHeader_2x05_P1.27mm_Vertical_SMD, symbol Connector:Conn_ARM_JTAG_SWD_10
- removed U2: TLV75512PDRV, Package_SON:WSON-6-1EP_2x2mm_P0.65mm_EP1x1.6mm, symbol Regulator_Linear:TLV75512PDRV
- removed U6: ICE40HX8K-BG121, Package_BGA:BGA-121_9.0x9.0mm_Layout11x11_P0.8mm_Ball0.4mm_Pad0.35mm_NSMD, symbol FPGA_Lattice:ICE40HX8K-BG121
- added C37, C39, C41, C43, C45: 10n, Capacitor_SMD:C_0402_1005Metric, symbol Device:C_Small
- added C38, C40, C42, C44: 0.1u, Capacitor_SMD:C_0402_1005Metric, symbol Device:C_Small
- added D65: LED_Small, LED_SMD:LED_0603_1608Metric, symbol Device:LED_Small
- added J6: TC2050, Connector:Tag-Connect_TC2050-IDC-NL_2x05_P1.27mm_Vertical, symbol Connector_Generic:Conn_01x10
- added L1: 1.5u, Inductor_SMD:L_1008_2520Metric, symbol Device:L
- added R80: 10k, Resistor_SMD:R_0402_1005Metric, symbol Device:R_Small
- added R81: 82k, Resistor_SMD:R_0402_1005Metric, symbol Device:R_Small
- added R82: 100k, Resistor_SMD:R_0402_1005Metric, symbol Device:R_Small
- added U2: AP2127K-2.5, Package_TO_SOT_SMD:SOT-23-5, symbol Regulator_Linear:AP2127K-2.5
- added U6: ECP5U_25_CABGA256, Package_BGA:BGA-256_14.0x14.0mm_Layout16x16_P0.8mm_Ball0.45mm_Pad0.32mm_NSMD, symbol Lattice_ECP5_FPGA:ECP5U_25_CABGA256
- added U8: TPS62A01ADRLR, Package_TO_SOT_SMD:SOT-563, symbol dc_dc_regulators:TPS62A01
- C1, C17: value 4.7u -> 10n; LCSC C23733 -> C307331
- C10, C14, C5, C9: value 0.1u -> 10n
- C16, C2, C35, C4: value 4.7u -> 0.1u; LCSC C23733 -> C307331
- C23, C24: value 0.1u -> 4.7u; LCSC C307331 -> C23733
- C28, C31, C33: value 0.1u -> 10u; footprint Capacitor_SMD:C_0402_1005Metric -> Capacitor_SMD:C_0603_1608Metric; LCSC C307331 -> C182375; Specification (none) -> 16V,X5R
- C32: value 0.1u -> 27p; LCSC C307331 -> (none)
- C34: value 4.7u -> 10u; footprint Capacitor_SMD:C_0402_1005Metric -> Capacitor_SMD:C_0603_1608Metric; LCSC C23733 -> C182375; Specification (none) -> 16V,X5R
- R10, R9: value 10k -> 1k; LCSC C25744 -> C258090
- R3: value 100k -> 1k
- R4: footprint Resistor_SMD:R_0402_1005Metric -> Resistor_SMD:R_0805_2012Metric
- R43, R44: value 100 -> 1k; LCSC C25076 -> C258090
Connections:
- net +3V3: now also C1.2, C2.2, C35.2, C4.2, C5.2, R43.2, R44.2, C37.2, C38.2, C39.2, C40.2, C41.2, C42.2, C43.2, C44.2, C45.2, J6.1 (Pin_1), R80.2, U6.F10 (VCCIO1[2]), U6.F11 (VCCIO1[2]), U6.F6 (VCCIO0[2]), U6.F7 (VCCIO0[2]), U6.H11 (VCCIO2[2]), U6.H6 (VCCIO7[2]), U6.H7 (VCCIO7[2]), U6.J11 (VCCIO2[2]), U6.J6 (VCCIO6[2]), U6.J7 (VCCIO6[2]), U6.K11 (VCCIO3[2]), U6.L11 (VCCIO3[2]), U6.L6 (VCCIO8); no longer C1.1, C13.1, C16.1, C23.1, C28.1, C5.1, C9.1
- net +5V: now also C23.1, C24.1, U1.4 (EN), U2.1 (VIN), U2.3 (EN), U8.3 (VIN), U8.4 (EN); no longer C4.1
- net CDONE: now also D65.1 (K), U6.P9 (DONE); no longer R10.1
- net CLKOUT: now also U6.B9 (PT38A/+/GR_PCLK1_0)
- net CTL0/FLAGA: now also U6.A15 (PT67B/-)
- net CTL1/FLAGB: now also U6.D12 (PT58A/+)
- net GND: now also C1.1, C10.1, C13.1, C14.1, C16.1, C17.1, C2.1, C33.2, C34.2, C35.1, C4.1, C5.1, C6.1, C7.1, C9.1, R3.1, C37.1, C38.1, C39.1, C40.1, C41.1, C42.1, C43.1, C44.1, C45.1, J6.3 (Pin_3), R82.1, U2.2 (GND), U6.A1 (GND[27]), U6.A16 (GND[27]), U6.D15 (GND[27]), U6.D2 (GND[27]), U6.F8 (GND[27]), U6.F9 (GND[27]), U6.G10 (GND[27]), U6.G8 (GND[27]), U6.H1 (GND[27]), U6.H10 (GND[27]), U6.H16 (GND[27]), U6.H8 (GND[27]), U6.H9 (GND[27]), U6.J10 (GND[27]), U6.J8 (GND[27]), U6.J9 (GND[27]), U6.K10 (GND[27]), U6.K6 (GND[27]), U6.K7 (GND[27]), U6.K8 (GND[27]), U6.K9 (GND[27]), U6.N10 (CFG_0), U6.N15 (GND[27]), U6.N2 (GND[27]), U6.R10 (CFG_2), U6.T1 (GND[27]), U6.T12 (GND[27]), U6.T16 (GND[27]), U6.T5 (GND[27]), U8.1 (GND); no longer C1.2, C10.2, C13.2, C14.2, C16.2, C17.2, C2.2, C4.2, C5.2, C6.2, C7.2, C9.2
- net IFCLK: now also U6.C8 (PT35A/+/PCLKT1_0)
- net IO00: now also U6.L1 (PL26A/+/PCLKT6_1/HS/LDQ32)
- net IO01: now also U6.L2 (PL26B/-/PCLKC6_1/HS/LDQ32)
- net IO02: now also U6.M1 (PL26C/+/PCLKT6_0/LDQ32)
- net IO03: now also U6.M2 (PL26D/-/PCLKC6_0/LDQ32)
- net IO04: now also U6.N1 (PL32A/+/HS/LDQS32)
- net IO05: now also U6.P2 (PL32B/-/HS/LDQSN32)
- net IO06: now also U6.P1 (PL35A/+/HS/LDQ32)
- net IO07: now also U6.R1 (PL35B/-/VREF1_6/HS/LDQ32)
- net IO08: now also U6.R2 (PL38C/+/LDQ44)
- net IO09: now also U6.T2 (PL38D/-/LDQ44)
- net IO10: now also U6.R3 (PL41B/-/HS/LDQ44)
- net IO11: now also U6.R4 (PL41C/+/LDQ44)
- net IO12: now also U6.T3 (PL41D/-/LDQ44)
- net IO13: now also U6.N3 (PL35D/-/LDQ32)
- net IO14: now also U6.T4 (PL44B/-/HS/LDQSN44)
- net IO15: now also U6.P3 (PL38B/-/HS/LDQ44)
- net IO16: now also U6.B1 (PL2A/+/HS/LDQ8)
- net IO17: now also U6.B2 (PL2B/-/HS/LDQ8)
- net IO18: now also U6.C1 (PL5A/+/HS/LDQ8)
- net IO19: now also U6.C2 (PL5B/-/HS/LDQ8)
- net IO20: now also U6.D1 (PL8A/+/HS/LDQS8)
- net IO21: now also U6.E2 (PL8B/-/HS/LDQSN8)
- net IO22: now also U6.F2 (PL11C/+/LDQ8)
- net IO23: now also U6.E1 (PL11D/-/LDQ8)
- net IO24: now also U6.F1 (PL14A/+/HS/LDQ20)
- net IO25: now also U6.G2 (PL14B/-/HS/LDQ20)
- net IO26: now also U6.G1 (PL20A/+/GR_PCLK7_1/HS/LDQS20)
- net IO27: now also U6.H2 (PL20B/-/HS/LDQSN20)
- net IO28: now also U6.J1 (PL23A/+/PCLKT7_1/HS/LDQ20)
- net IO29: now also U6.J2 (PL23B/-/PCLKC7_1/HS/LDQ20)
- net IO30: now also U6.K1 (PL23C/+/PCLKT7_0/LDQ20)
- net IO31: now also U6.K2 (PL23D/-/PCLKC7_0/LDQ20)
- net IO32: now also U6.B16 (PR2A/+/HS/RDQ8)
- net IO33: now also U6.B15 (PR2B/-/S0_IN/HS/RDQ8)
- net IO34: now also U6.C16 (PR5A/+/HS/RDQ8)
- net IO35: now also U6.C15 (PR5B/-/HS/RDQ8)
- net IO36: now also U6.D16 (PR8A/+/HS/RDQS8)
- net IO37: now also U6.E15 (PR8B/-/HS/RDQSN8)
- net IO38: now also U6.F15 (PR11C/+/RDQ8)
- net IO39: now also U6.E16 (PR11D/-/RDQ8)
- net IO40: now also U6.F16 (PR14A/+/HS/RDQ20)
- net IO41: now also U6.G15 (PR14B/-/HS/RDQ20)
- net IO42: now also U6.K15 (PR23D/-/PCLKC2_0/RDQ20)
- net IO43: now also U6.G16 (PR20A/+/GR_PCLK2_1/HS/RDQS20)
- net IO44: now also U6.H15 (PR20B/-/HS/RDQSN20)
- net IO45: now also U6.J16 (PR23A/+/PCLKT2_1/HS/RDQ20)
- net IO46: now also U6.J15 (PR23B/-/PCLKC2_1/HS/RDQ20)
- net IO47: now also U6.K16 (PR23C/+/PCLKT2_0/RDQ20)
- net IO48: now also U6.L16 (PR26A/+/PCLKT3_1/HS/RDQ32)
- net IO49: now also U6.L15 (PR26B/-/PCLKC3_1/HS/RDQ32)
- net IO50: now also U6.M16 (PR26C/+/PCLKT3_0/RDQ32)
- net IO51: now also U6.M15 (PR26D/-/PCLKC3_0/RDQ32)
- net IO52: now also U6.N16 (PR32A/+/HS/RDQS32)
- net IO53: now also U6.P15 (PR32B/-/HS/RDQSN32)
- net IO54: now also U6.P16 (PR35A/+/HS/RDQ32)
- net IO55: now also U6.R16 (PR35B/-/VREF1_3/HS/RDQ32)
- net IO56: now also U6.P14 (PR38B/-/HS/RDQ44)
- net IO57: now also U6.R15 (PR38C/+/RDQ44)
- net IO58: now also U6.T15 (PR38D/-/RDQ44)
- net IO59: now also U6.R14 (PR41B/-/HS/RDQ44)
- net IO60: now also U6.R13 (PR41C/+/RDQ44)
- net IO61: now also U6.T14 (PR41D/-/RDQ44)
- net IO62: now also U6.R12 (PR44A/+/HS/RDQS44)
- net IO63: now also U6.T13 (PR44B/-/HS/RDQSN44)
- net PA0/~{INT0}: now also U6.A14 (PT65B/-)
- net PA2/SLOE: now also U6.A12 (PT53B/-)
- net PA4/FIOADDR0: now also U6.B11 (PT49A/+)
- net PA5/FIOADDR1: now also U6.C13 (PT60B/-)
- net PA6/PKTEND: now also U6.B10 (PT44A/+)
- net PB0/FD0: now also U6.C12 (PT56B/-)
- net PB1/FD1: now also U6.A11 (PT53A/+)
- net PB2/FD2: now also U6.B12 (PT56A/+)
- net PB3/FD3: now also U6.A13 (PT65A/+)
- net PB4/FD4: now also U6.B14 (PT67A/+)
- net PB5/FD5: now also U6.B13 (PT60A/+)
- net PB6/FD6: now also U6.C10 (PT44B/-)
- net PB7/FD7: now also U6.A10 (PT42B/-)
- net RDY0/SLRD: now also U6.A9 (PT42A/+)
- net RDY1/SLWR: now also U6.D13 (PT62A/+)
- net ~{CRESET}: no longer R9.1
- net +1V1: now reaches C32.2
- net +1V1: now also C13.2, C14.2, C16.2, C17.2, C33.1, C34.1, C6.2, C9.2, L1.2, R81.2, U6.G6 (VCC[6]), U6.G7 (VCC[6]), U6.G9 (VCC[6]), U6.L10 (VCC[6]), U6.L8 (VCC[6]), U6.L9 (VCC[6]); no longer C34.2
- net SPI_D3: now reaches R78.1, U7.7 (IO3)
- net SPI_D3: now also U6.N7 (PB9A/+/D3/IO3)
- net SPI_D2: now reaches R79.1, U7.3 (IO2)
- net SPI_D2: now also U6.M7 (PB9B/-/D2/IO2)
- removed net +1V2: C10.1, C14.1, C17.1, C2.1, C24.1, C6.1, R3.1, R43.1, R44.1
- removed net 3V3_EN: C7.1, R3.2, U1.4 (EN)
- net IOB_105_SDO renamed SPI_MOSI
- net SPI_MOSI: now also U6.T8 (PB11B/-/D0/MOSI/IO0)
- net IOB_106_SDI renamed SPI_MISO
- net SPI_MISO: now also U6.T7 (PB11A/+/D1/MISO/IO1)
- net IOB_107_SCK renamed SPI_CLK
- net SPI_CLK: now also R9.1, U6.N9 (CCLK/MCLK/SCK)
- net IOB_108_SS renamed SPI_CS
- net SPI_CS: now also U6.N8 (PB15A/+/HOLDN/DI/BUSY/CSSPIN/CEN)
- new net: D65.2 (A), R43.1
- new net +2V5: C10.2, C28.1, C7.2, U2.5 (VOUT), U6.G11 (VCCAUX[2]), U6.L7 (VCCAUX[2])
- new net CFG_1: R10.1, U6.P10 (CFG_1)
- new net FB: C32.1, R81.1, R82.2, U8.5 (FB)
- new net INITN: R80.1, U6.T9 (INITN)
- new net PROGRAMN: R44.1, U6.R9 (PROGRAMN)
- new net SW: L1.1, U8.2 (SW)
- new net TCK: J6.4 (Pin_4), R3.2, U6.T10 (TCK)
- new net TDI: J6.8 (Pin_8), U6.R11 (TDI)
- new net TDO: J6.6 (Pin_6), U6.M10 (TDO)
- new net TMS: J6.2 (Pin_2), U6.T11 (TMS)
- no-connect marks 21 -> 27
Other:
- note added: "DESIGN NOTE: Master SPI config."
- moved on the sheet: C3, C36, D1, D10, D11, D12, D13, D14, D15, D16, D17, D18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

Commit message: Save
Parts:
- added C46, C47: 4.7u, Capacitor_SMD:C_0402_1005Metric, symbol Device:C_Small
Connections:
- net ~{CRESET} is gone; now on net PROGRAMN: U5.34 (PA1/~{INT1})
- net +3V3: now also C46.1, C47.1
- net GND: now also C46.2, C47.2
- no-connect marks 27 -> 128
