File: ssla.kicad_sch (KiCad schematic)
At the start: 217 parts, among them J1 USB_C_Receptacle_USB2.0_14P, J2 Conn_02x10_Odd_Even, J3 Conn_02x10_Odd_Even, J4 Conn_02x10_Odd_Even, J5 Conn_02x10_Odd_Even, J6 TC2050, U1 TLV75533PDRV, U2 AP2127K-2.5, U3 BL24C256A, U4 USBLC6-2P6, U5 CY7C68013A-56LTX, U6 ECP5U_25_CABGA256, U7 W25Q16JVUXIQ, U8 TPS62A01ADRLR, Y1 24 MHz

Commit message: Ordered
Parts:
- added C48, C49: 4.7u, Capacitor_SMD:C_0402_1005Metric, symbol Device:C_Small
- added D66: LED_Small, LED_SMD:LED_0603_1608Metric, symbol Device:LED_Small
- added R83: 1k, Resistor_SMD:R_0402_1005Metric, symbol Device:R_Small
- C1, C10, C14, C17, C37, C39, C41, C43, C45, C5, C9: LCSC C307331 -> C15195
- C32: LCSC (none) -> C126504
- R10, R3, R43, R44, R9: LCSC C258090 -> C11702
- R80: LCSC C258090 -> C25744
- R81: LCSC C25744 -> C4142
- R82: LCSC C25744 -> C258090
- U2: LCSC (none) -> C460326
Connections:
- net +1V1: now also C48.1
- net +2V5: now also C49.1
- net CTL0/FLAGA: now also U6.B12 (PT56A/+); no longer U6.A15 (PT67B/-)
- net CTL1/FLAGB: now also U6.B13 (PT60A/+); no longer U6.D12 (PT58A/+)
- net GND: now also C48.2, C49.2, D66.1 (K)
- net IO00: now also U6.T4 (PL44B/-/HS/LDQSN44); no longer U6.L1 (PL26A/+/PCLKT6_1/HS/LDQ32)
- net IO01: now also U6.R4 (PL41C/+/LDQ44); no longer U6.L2 (PL26B/-/PCLKC6_1/HS/LDQ32)
- net IO02: now also U6.T3 (PL41D/-/LDQ44); no longer U6.M1 (PL26C/+/PCLKT6_0/LDQ32)
- net IO03: now also U6.R3 (PL41B/-/HS/LDQ44); no longer U6.M2 (PL26D/-/PCLKC6_0/LDQ32)
- net IO04: now also U6.T2 (PL38D/-/LDQ44); no longer U6.N1 (PL32A/+/HS/LDQS32)
- net IO05: now also U6.P3 (PL38B/-/HS/LDQ44); no longer U6.P2 (PL32B/-/HS/LDQSN32)
- net IO06: now also U6.R2 (PL38C/+/LDQ44); no longer U6.P1 (PL35A/+/HS/LDQ32)
- net IO08: now also U6.N3 (PL35D/-/LDQ32); no longer U6.R2 (PL38C/+/LDQ44)
- net IO09: now also U6.P1 (PL35A/+/HS/LDQ32); no longer U6.T2 (PL38D/-/LDQ44)
- net IO10: now also U6.P2 (PL32B/-/HS/LDQSN32); no longer U6.R3 (PL41B/-/HS/LDQ44)
- net IO11: now also U6.N1 (PL32A/+/HS/LDQS32); no longer U6.R4 (PL41C/+/LDQ44)
- net IO12: now also U6.M2 (PL26D/-/PCLKC6_0/LDQ32); no longer U6.T3 (PL41D/-/LDQ44)
- net IO13: now also U6.M1 (PL26C/+/PCLKT6_0/LDQ32); no longer U6.N3 (PL35D/-/LDQ32)
- net IO14: now also U6.L2 (PL26B/-/PCLKC6_1/HS/LDQ32); no longer U6.T4 (PL44B/-/HS/LDQSN44)
- net IO15: now also U6.L1 (PL26A/+/PCLKT6_1/HS/LDQ32); no longer U6.P3 (PL38B/-/HS/LDQ44)
- net IO16: now also U6.F2 (PL11C/+/LDQ8); no longer U6.B1 (PL2A/+/HS/LDQ8)
- net IO17: now also U6.E1 (PL11D/-/LDQ8); no longer U6.B2 (PL2B/-/HS/LDQ8)
- net IO18: now also U6.E2 (PL8B/-/HS/LDQSN8); no longer U6.C1 (PL5A/+/HS/LDQ8)
- net IO19: now also U6.D1 (PL8A/+/HS/LDQS8); no longer U6.C2 (PL5B/-/HS/LDQ8)
- net IO20: now also U6.C1 (PL5A/+/HS/LDQ8); no longer U6.D1 (PL8A/+/HS/LDQS8)
- net IO21: now also U6.C2 (PL5B/-/HS/LDQ8); no longer U6.E2 (PL8B/-/HS/LDQSN8)
- net IO22: now also U6.B1 (PL2A/+/HS/LDQ8); no longer U6.F2 (PL11C/+/LDQ8)
- net IO23: now also U6.B2 (PL2B/-/HS/LDQ8); no longer U6.E1 (PL11D/-/LDQ8)
- net IO24: now also U6.K2 (PL23D/-/PCLKC7_0/LDQ20); no longer U6.F1 (PL14A/+/HS/LDQ20)
- net IO25: now also U6.K1 (PL23C/+/PCLKT7_0/LDQ20); no longer U6.G2 (PL14B/-/HS/LDQ20)
- net IO26: now also U6.J2 (PL23B/-/PCLKC7_1/HS/LDQ20); no longer U6.G1 (PL20A/+/GR_PCLK7_1/HS/LDQS20)
- net IO27: now also U6.J1 (PL23A/+/PCLKT7_1/HS/LDQ20); no longer U6.H2 (PL20B/-/HS/LDQSN20)
- net IO28: now also U6.H2 (PL20B/-/HS/LDQSN20); no longer U6.J1 (PL23A/+/PCLKT7_1/HS/LDQ20)
- net IO29: now also U6.G1 (PL20A/+/GR_PCLK7_1/HS/LDQS20); no longer U6.J2 (PL23B/-/PCLKC7_1/HS/LDQ20)
- net IO30: now also U6.G2 (PL14B/-/HS/LDQ20); no longer U6.K1 (PL23C/+/PCLKT7_0/LDQ20)
- net IO31: now also U6.F1 (PL14A/+/HS/LDQ20); no longer U6.K2 (PL23D/-/PCLKC7_0/LDQ20)
- net IO32: now also U6.K15 (PR23D/-/PCLKC2_0/RDQ20); no longer U6.B16 (PR2A/+/HS/RDQ8)
- net IO33: now also U6.K16 (PR23C/+/PCLKT2_0/RDQ20); no longer U6.B15 (PR2B/-/S0_IN/HS/RDQ8)
- net IO34: now also U6.J15 (PR23B/-/PCLKC2_1/HS/RDQ20); no longer U6.C16 (PR5A/+/HS/RDQ8)
- net IO35: now also U6.J16 (PR23A/+/PCLKT2_1/HS/RDQ20); no longer U6.C15 (PR5B/-/HS/RDQ8)
- net IO36: now also U6.H15 (PR20B/-/HS/RDQSN20); no longer U6.D16 (PR8A/+/HS/RDQS8)
- net IO37: now also U6.G15 (PR14B/-/HS/RDQ20); no longer U6.E15 (PR8B/-/HS/RDQSN8)
- net IO38: now also U6.G16 (PR20A/+/GR_PCLK2_1/HS/RDQS20); no longer U6.F15 (PR11C/+/RDQ8)
- net IO39: now also U6.F15 (PR11C/+/RDQ8); no longer U6.E16 (PR11D/-/RDQ8)
- net IO41: now also U6.E15 (PR8B/-/HS/RDQSN8); no longer U6.G15 (PR14B/-/HS/RDQ20)
- net IO42: now also U6.D16 (PR8A/+/HS/RDQS8); no longer U6.K15 (PR23D/-/PCLKC2_0/RDQ20)
- net IO43: now also U6.E16 (PR11D/-/RDQ8); no longer U6.G16 (PR20A/+/GR_PCLK2_1/HS/RDQS20)
- net IO44: now also U6.C15 (PR5B/-/HS/RDQ8); no longer U6.H15 (PR20B/-/HS/RDQSN20)
- net IO45: now also U6.C16 (PR5A/+/HS/RDQ8); no longer U6.J16 (PR23A/+/PCLKT2_1/HS/RDQ20)
- net IO46: now also U6.B15 (PR2B/-/S0_IN/HS/RDQ8); no longer U6.J15 (PR23B/-/PCLKC2_1/HS/RDQ20)
- net IO47: now also U6.B16 (PR2A/+/HS/RDQ8); no longer U6.K16 (PR23C/+/PCLKT2_0/RDQ20)
- net IO48: now also U6.R16 (PR35B/-/VREF1_3/HS/RDQ32); no longer U6.L16 (PR26A/+/PCLKT3_1/HS/RDQ32)
- net IO49: now also U6.P15 (PR32B/-/HS/RDQSN32); no longer U6.L15 (PR26B/-/PCLKC3_1/HS/RDQ32)
- net IO50: now also U6.P16 (PR35A/+/HS/RDQ32); no longer U6.M16 (PR26C/+/PCLKT3_0/RDQ32)
- net IO51: now also U6.N16 (PR32A/+/HS/RDQS32); no longer U6.M15 (PR26D/-/PCLKC3_0/RDQ32)
- net IO52: now also U6.M15 (PR26D/-/PCLKC3_0/RDQ32); no longer U6.N16 (PR32A/+/HS/RDQS32)
- net IO53: now also U6.M16 (PR26C/+/PCLKT3_0/RDQ32); no longer U6.P15 (PR32B/-/HS/RDQSN32)
- net IO54: now also U6.L15 (PR26B/-/PCLKC3_1/HS/RDQ32); no longer U6.P16 (PR35A/+/HS/RDQ32)
- net IO55: now also U6.L16 (PR26A/+/PCLKT3_1/HS/RDQ32); no longer U6.R16 (PR35B/-/VREF1_3/HS/RDQ32)
- net IO56: now also U6.R12 (PR44A/+/HS/RDQS44); no longer U6.P14 (PR38B/-/HS/RDQ44)
- net IO57: now also U6.T13 (PR44B/-/HS/RDQSN44); no longer U6.R15 (PR38C/+/RDQ44)
- net IO58: now also U6.R13 (PR41C/+/RDQ44); no longer U6.T15 (PR38D/-/RDQ44)
- net IO59: now also U6.T14 (PR41D/-/RDQ44); no longer U6.R14 (PR41B/-/HS/RDQ44)
- net IO60: now also U6.R14 (PR41B/-/HS/RDQ44); no longer U6.R13 (PR41C/+/RDQ44)
- net IO61: now also U6.T15 (PR38D/-/RDQ44); no longer U6.T14 (PR41D/-/RDQ44)
- net IO62: now also U6.R15 (PR38C/+/RDQ44); no longer U6.R12 (PR44A/+/HS/RDQS44)
- net IO63: now also U6.P14 (PR38B/-/HS/RDQ44); no longer U6.T13 (PR44B/-/HS/RDQSN44)
- net PA0/~{INT0}: now also U6.B14 (PT67A/+); no longer U6.A14 (PT65B/-)
- net PA2/SLOE: now also U6.C13 (PT60B/-); no longer U6.A12 (PT53B/-)
- net PA4/FIOADDR0: now also U6.D12 (PT58A/+); no longer U6.B11 (PT49A/+)
- net PA5/FIOADDR1: now also U6.C12 (PT56B/-); no longer U6.C13 (PT60B/-)
- net PA6/PKTEND: now also U6.D13 (PT62A/+); no longer U6.B10 (PT44A/+)
- net PB0/FD0: now also U6.A9 (PT42A/+); no longer U6.C12 (PT56B/-)
- net PB1/FD1: now also U6.B10 (PT44A/+); no longer U6.A11 (PT53A/+)
- net PB2/FD2: now also U6.A10 (PT42B/-); no longer U6.B12 (PT56A/+)
- net PB3/FD3: now also U6.A11 (PT53A/+); no longer U6.A13 (PT65A/+)
- net PB4/FD4: now also U6.A12 (PT53B/-); no longer U6.B14 (PT67A/+)
- net PB5/FD5: now also U6.A13 (PT65A/+); no longer U6.B13 (PT60A/+)
- net PB6/FD6: now also U6.A14 (PT65B/-); no longer U6.C10 (PT44B/-)
- net PB7/FD7: now also U6.A15 (PT67B/-); no longer U6.A10 (PT42B/-)
- net RDY0/SLRD: now also U6.B11 (PT49A/+); no longer U6.A9 (PT42A/+)
- net RDY1/SLWR: now also U6.C10 (PT44B/-); no longer U6.D13 (PT62A/+)
- net LED: now reaches U6.A2 (PT4A/+)
- net LED: now also R83.1
- new net: D66.2 (A), R83.2
- no-connect marks 128 -> 127
