File: ssla.kicad_sch (KiCad schematic)
At the start: 221 parts, among them J1 USB_C_Receptacle_USB2.0_14P, J2 Conn_02x10_Odd_Even, J3 Conn_02x10_Odd_Even, J4 Conn_02x10_Odd_Even, J5 Conn_02x10_Odd_Even, J6 TC2050, U1 TLV75533PDRV, U2 AP2127K-2.5, U3 BL24C256A, U4 USBLC6-2P6, U5 CY7C68013A-56LTX, U6 ECP5U_25_CABGA256, U7 W25Q16JVUXIQ, U8 TPS62A01ADRLR, Y1 24 MHz

Commit message: wip
Parts:
- removed C11, C12, C15, C18, C21, C22, C25, C26, C27, C29, C30: 0.1u, Capacitor_SMD:C_0402_1005Metric, symbol Device:C_Small
- removed C19, C20: 12p, Capacitor_SMD:C_0402_1005Metric, symbol Device:C_Small
- removed TP11, TP12: TestPoint_Small, TestPoint:TestPoint_Pad_D1.0mm, symbol Connector:TestPoint_Small
- removed U3: BL24C256A, Package_SO:TSSOP-8_4.4x3mm_P0.65mm, symbol Memory_EEPROM:CAT24C256
- removed U4: USBLC6-2P6, Package_TO_SOT_SMD:SOT-666, symbol Power_Protection:USBLC6-2P6
- removed U5: CY7C68013A-56LTX, Package_DFN_QFN:QFN-56-1EP_8x8mm_P0.5mm_EP4.5x5.2mm, symbol MCU_Cypress:CY7C68013A-56LTX
- removed Y1: 24 MHz, Crystal:Crystal_SMD_2016-4Pin_2.0x1.6mm, symbol Device:Crystal_GND24_Small
- added C50, C54: 22u, Capacitor_SMD:C_0603_1608Metric, symbol Device:C_Small
- added C51: 2.2u, Capacitor_SMD:C_0402_1005Metric, symbol Device:C_Small
- added C52, C53, C55, C56, C57: 0.1u, Capacitor_SMD:C_0402_1005Metric, symbol Device:C_Small
- added C58: 10u, Capacitor_SMD:C_0603_1608Metric, symbol Device:C_Small
- added FB2: 120 ohm, Inductor_SMD:L_0402_1005Metric, symbol Device:FerriteBead_Small
- added J7: RJ45_Hanrun_HR911105A_Horizontal, Connector_RJ:RJ45_Hanrun_HR911105A_Horizontal, symbol Connector:RJ45_Hanrun_HR911105A_Horizontal
- added R84: 6.49k, Resistor_SMD:R_0402_1005Metric, symbol Device:R_Small
- added R85: 1k, Resistor_SMD:R_0402_1005Metric, symbol Device:R_Small
- added R86: 10k, Resistor_SMD:R_0402_1005Metric, symbol Device:R_Small
- added U9: KSZ8081RNA, Package_DFN_QFN:QFN-24-1EP_4x4mm_P0.5mm_EP2.6x2.6mm, symbol Interface_Ethernet:KSZ8081RNA
- added Y1: 25 MHz, Oscillator:Oscillator_SMD_SiT_PQFN-4Pin_2.0x1.6mm, symbol Oscillator:ASCO
- C8: value 4.7u -> 0.1u; LCSC C23733 -> C307331
- R4: value 0 -> 22; footprint Resistor_SMD:R_0805_2012Metric -> Resistor_SMD:R_0402_1005Metric; now fitted
- R5: value 2.2k -> 22; LCSC C25933 -> (none)
- R6: value 100k -> 5.1k; LCSC C258090 -> C25905
- R7: value 2.2k -> 5.1k; LCSC C25933 -> C25905
- R8: value 100k -> 10k; LCSC C258090 -> C25744
Connections:
- net CLKOUT is gone; now on net FPGA_XI: U6.B9 (PT38A/+/GR_PCLK1_0)
- net SDA is gone; now on net ETH.MDC: R7.2
- net ~{RESET} is gone; now on net ETH.MDIO: R6.2
- net +3V3: now also C8.2, C54.1, C55.2, FB2.2, R85.2, U9.14 (VDDIO), Y1.1 (Tri-State), Y1.4 (VDD); no longer C8.1, R4.1, R5.1, R8.2
- net GND: now also C8.1, R8.2, C50.2, C51.2, C52.1, C53.1, C54.2, C55.1, C56.1, C57.1, J7.8, J7.SH, R84.1, U9.22 (GND), U9.25 (GND), Y1.2 (GND); no longer C8.2
- net FPGA_XI: now reaches R4.2
- net CTL0/FLAGA renamed ETH.MDIO
- net ETH.MDIO: now also U9.10 (MDIO)
- net CTL1/FLAGB renamed ETH.MDC
- net ETH.MDC: now also U9.11 (MDC)
- net D_N: no longer names the net of J1.A7 (D-)
- net D_N: no longer J1.B7 (D-)
- net D_P: no longer names the net of J1.A6 (D+)
- net D_P: no longer J1.B6 (D+)
- net IFCLK renamed ETH.REF_CLK
- net ETH.REF_CLK: now also U9.16 (REF_CLK)
- net PA0/~{INT0} renamed ~{ETH.RST}
- net ~{ETH.RST}: now also U9.24 (~{RST})
- net PA2/SLOE: no longer names the net of U6.C13 (PT60B/-)
- net PA4/FIOADDR0: no longer names the net of U6.D12 (PT58A/+)
- net PA5/FIOADDR1: no longer names the net of U6.C12 (PT56B/-)
- net PA6/PKTEND: no longer names the net of U6.D13 (PT62A/+)
- net PB0/FD0 renamed ETH.TXEN
- net ETH.TXEN: now also U9.19 (TXEN)
- net PB1/FD1: no longer names the net of U6.B10 (PT44A/+)
- net PB2/FD2 renamed ETH.TXD0
- net ETH.TXD0: now also U9.20 (TXD0)
- net PB3/FD3 renamed ETH.TXD1
- net ETH.TXD1: now also U9.21 (TXD1)
- net PB4/FD4 renamed ETH.RXD0
- net ETH.RXD0: now also U9.13 (RXD0)
- net PB5/FD5 renamed ETH.RXD1
- net ETH.RXD1: now also U9.12 (RXD1)
- net PB6/FD6 renamed ETH.CRS_DV
- net ETH.CRS_DV: now also U9.15 (CRS_DV/PHYAD[1:0])
- net PB7/FD7 renamed ETH.RXER
- net ETH.RXER: now also U9.17 (RXER)
- net RDY0/SLRD: no longer names the net of U6.B11 (PT49A/+)
- net RDY1/SLWR: no longer names the net of U6.C10 (PT44B/-)
- net SCL renamed PHY_XI
- net PHY_XI: now also U9.8 (XI)
- new net: J7.11, U9.23 (LED0/ANEN_SPEED)
- new net: R84.2, U9.9 (REXT)
- new net: C56.2, J7.4 (TCT)
- new net: R4.1, R5.1, Y1.3 (OUT)
- new net: J7.12, R85.1
- new net: C57.2, J7.5 (RCT)
- new net RX+: J7.2 (TD-), U9.4 (RXP)
- new net RX-: J7.1 (TD+), U9.3 (RXM)
- new net TX+: J7.6 (RD-), U9.6 (TXP)
- new net TX-: J7.3 (RD+), U9.5 (TXM)
- new net VDDA_3.3: C50.1, C53.2, FB2.1, U9.2 (VDDA_3.3)
- new net VDD_1.2: C51.1, C52.2, U9.1 (VDD_1.2)
- no-connect marks 127 -> 110
Other:
- moved on the sheet: FB1, H1, H2, H3, H4, J1, R1, R2

Commit message: Save
Parts:
- removed C3: 4.7u, Capacitor_SMD:C_0402_1005Metric, symbol Device:C_Small
- removed C31, C33, C34, C58: 10u, Capacitor_SMD:C_0603_1608Metric, symbol Device:C_Small
- removed D1, D10, D11, D12, D13, D14, D15, D16, D17, D18, D19, D2, D20, D21, D22, D23, D24, D25, D26, D27, D28, D29, D3, D30, D31, D32, D33, D34, D35, D36, D37, D38, D39, D4, D40, D41, D42, D43, D44, D45, D46, D47, D48, D49, D5, D50, D51, D52, D53, D54, D55, D56, D57, D58, D59, D6, D60, D61, D62, D63, D64, D7, D8, D9: D_TVS_Small, Diode_SMD:D_SOD-923, symbol Device:D_TVS_Small
- removed J3, J4, J5: Conn_02x10_Odd_Even, Connector_IDC:IDC-Header_2x10_P2.54mm_Vertical, symbol Connector_Generic:Conn_02x10_Odd_Even
- removed J6: TC2050, Connector:Tag-Connect_TC2050-IDC-NL_2x05_P1.27mm_Vertical, symbol Connector_Generic:Conn_01x10
- removed R11, R12, R13, R14, R15, R16, R17, R18, R19, R20, R21, R22, R23, R24, R25, R26, R27, R28, R29, R30, R31, R32, R33, R34, R35, R36, R37, R38, R39, R40, R41, R42, R46, R47, R48, R49, R50, R51, R52, R53, R54, R55, R56, R57, R58, R59, R60, R61, R62, R63, R64, R65, R66, R67, R68, R69, R70, R71, R72, R73, R74, R75, R76, R77: 100, Resistor_SMD:R_0402_1005Metric, symbol Device:R_Small
- removed R3: 1k, Resistor_SMD:R_0402_1005Metric, symbol Device:R_Small
- removed R86: 10k, Resistor_SMD:R_0402_1005Metric, symbol Device:R_Small
- removed U1: TLV75533PDRV, Package_SON:WSON-6-1EP_2x2mm_P0.65mm_EP1x1.6mm, symbol Regulator_Linear:TLV75533PDRV
- added C101: 4.7u, Capacitor_SMD:C_0402_1005Metric, symbol Device:C_Small
- added C102: 27p, Capacitor_SMD:C_0402_1005Metric, symbol Device:C_Small
- added C103, C105, C106: 22u, Capacitor_SMD:C_0603_1608Metric, symbol Device:C_Small
- added C104, C107, C108, C109: 0.1u, Capacitor_SMD:C_0402_1005Metric, symbol Device:C_Small
- added J101: Sync In, symbol Connector_Generic:Conn_01x02
- added J102: Sync Out, symbol Connector_Generic:Conn_01x02
- added J6: TC2050, Connector:Tag-Connect_TC2050-IDC-NL_2x05_P1.27mm_Vertical, symbol Connector:TC2050
- added L101: 1.5u, Inductor_SMD:L_1008_2520Metric, symbol Device:L
- added R101: 450k, Resistor_SMD:R_0402_1005Metric, symbol Device:R_Small
- added R102, R125, R126, R127, R128, R129, R130, R131, R132, R133, R134, R135, R136, R137, R138, R139, R140: 100k, Resistor_SMD:R_0402_1005Metric, symbol Device:R_Small
- added R103, R104, R105, R106, R107, R108, R109, R110, R111, R112, R113, R114, R115, R116, R117, R118, R124: 47, Resistor_SMD:R_0402_1005Metric, symbol Device:R_Small
- added R119, R120, R121, R122, R123: 10k, Resistor_SMD:R_0402_1005Metric, symbol Device:R_Small
- added R141: 150, Resistor_SMD:R_0402_1005Metric, symbol Device:R_Small
- added R142: 1k, Resistor_SMD:R_0402_1005Metric, symbol Device:R_Small
- added U101: TPS62A01ADRLR, Package_TO_SOT_SMD:SOT-563, symbol dc_dc_regulators:TPS62A01
- added U102, U103, U104: SN74LV6T17, Package_DFN_QFN:DHVQFN-14-1EP_2.5x3mm_P0.5mm_EP1x1.5mm, symbol 74xx:74HC7014
- added U105, U106, U107: NUF6401MNT1, dfn:DFN-12-1EP_1.35x3mm_P0.5mm, symbol interface_esd:NUF6401MNT1
- added U108: TLP2362, Package_SO:SO-5-6_4.55x3.7mm_P1.27mm, symbol Isolator:TLP2310
- FB1: value FerriteBead_Small -> 120 ohm; LCSC C491490 -> C88970
- FB2: LCSC (none) -> C88970
- R4, R5: value 22 -> 47
Connections:
- net +1V1: now also C105.1, C106.1
- net +3V3: now also C23.1, U2.1 (VIN), U2.3 (EN), C102.2, C103.1, C104.2, C107.2, C108.2, C109.2, L101.2, R101.2, R120.2, R121.2, R122.2, R124.2, R142.2, U102.14 (VCC), U103.14 (VCC), U104.14 (VCC), U108.6 (VDD)
- net +5V: now also C101.1, U101.3 (VIN), U101.4 (EN); no longer C23.1, U2.1 (VIN), U2.3 (EN)
- net ETH.CRS_DV: now also R119.1
- net GND: now also C101.2, C103.2, C104.1, C105.2, C106.2, C107.1, C108.1, C109.1, J102.2 (Pin_2), J6.3, J6.5, J6.9, R102.1, R119.2, R123.2, R125.1, R126.1, R127.1, R128.1, R129.1, R130.1, R131.1, R132.1, R133.1, R134.1, R135.1, R136.1, R137.1, R138.1, R139.1, R140.1, U101.1 (GND), U102.7 (GND), U103.11, U103.13, U103.7 (GND), U104.7 (GND), U105.13 (GND), U106.13 (GND), U106.5 (5A), U106.6 (6A), U107.13 (GND), U108.4 (GND)
- net IO00: now also R103.1
- net IO01: now also R104.1
- net IO02: now also R105.1
- net IO03: now also R106.1
- net IO04: now also R107.1
- net IO05: now also R108.1
- net IO06: now also R109.1
- net IO07: now also R110.1
- net IO08: now also R111.1
- net IO09: now also R112.1
- net IO10: now also R113.1
- net IO11: now also R114.1
- net IO12: now also R115.1
- net IO13: now also R116.1
- net IO14: now also R117.1
- net IO15: now also R118.1
- net RX+: now also J7.3 (RD+); no longer J7.2 (TD-)
- net RX-: now also J7.6 (RD-); no longer J7.1 (TD+)
- net TCK: now also J6.4, R121.1
- net TDI: now also J6.8
- net TDO: now also J6.6, R123.1
- net TMS: now also J6.2, R122.1
- net TX+: now also J7.1 (TD+); no longer J7.6 (RD-)
- net TX-: now also J7.2 (TD-); no longer J7.3 (RD+)
- net LED0/ANEN_SPEED: now reaches J7.11, U9.23 (LED0/ANEN_SPEED)
- net LED0/ANEN_SPEED: now also R120.1
- net REXT: now reaches R84.2, U9.9 (REXT)
- net IN6: now reaches J2.17 (Pin_17)
- net IN6: now also R130.2, U107.1 (1A)
- net IN12: now reaches J2.10 (Pin_10)
- net IN12: now also R140.2, U106.1 (1A)
- net IN2: now reaches J2.7 (Pin_7)
- net IN2: now also R126.2, U105.3 (3A)
- net IN14: now reaches J2.4 (Pin_4)
- net IN14: now also R136.2, U106.3 (3A)
- net IN3: now reaches J2.9 (Pin_9)
- net IN3: now also R125.2, U105.4 (4A)
- net at C56.2: now also J7.5 (RCT); no longer J7.4 (TCT)
- net IN15: now reaches J2.2 (Pin_2)
- net IN15: now also R134.2, U106.4 (4A)
- net SYNC_IN: now reaches U6.A3 (PT6A/+)
- net SYNC_IN: now also R142.1, U108.5 (VO)
- net SYNC_OUT: now reaches U6.E4 (PT9A/+)
- net SYNC_OUT: now also R141.1
- net IN8: now reaches J2.20 (Pin_20)
- net IN8: now also R139.2, U107.3 (3A)
- net at C57.2: now also J7.4 (TCT); no longer J7.5 (RCT)
- net IN4: now reaches J2.11 (Pin_11)
- net IN4: now also R132.2, U105.5 (5A)
- net IN9: now reaches J2.18 (Pin_18)
- net IN9: now also R137.2, U107.4 (4A)
- net IN0: now reaches J2.1 (Pin_1)
- net IN0: now also R128.2, U105.1 (1A)
- net IN1: now reaches J2.3 (Pin_3)
- net IN1: now also R127.2, U105.2 (2A)
- net IN10: now reaches J2.14 (Pin_14)
- net IN10: now also R135.2, U107.5 (5A)
- net IN11: now reaches J2.12 (Pin_12)
- net IN11: now also R133.2, U107.6 (6A)
- net IN7: now reaches J2.19 (Pin_19)
- net IN7: now also R129.2, U107.2 (2A)
- net IN5: now reaches J2.13 (Pin_13)
- net IN5: now also R131.2, U105.6 (6A)
- net IN13: now reaches J2.8 (Pin_8)
- net IN13: now also R138.2, U106.2 (2A)
- net FB renamed FB1V1
- net IO16: no longer names the net of U6.F2 (PL11C/+/LDQ8)
- net IO17: no longer names the net of U6.E1 (PL11D/-/LDQ8)
- net IO18: no longer names the net of U6.E2 (PL8B/-/HS/LDQSN8)
- net IO19: no longer names the net of U6.D1 (PL8A/+/HS/LDQS8)
- net IO20: no longer names the net of U6.C1 (PL5A/+/HS/LDQ8)
- net IO21: no longer names the net of U6.C2 (PL5B/-/HS/LDQ8)
- net IO22: no longer names the net of U6.B1 (PL2A/+/HS/LDQ8)
- net IO23: no longer names the net of U6.B2 (PL2B/-/HS/LDQ8)
- net IO24: no longer names the net of U6.K2 (PL23D/-/PCLKC7_0/LDQ20)
- net IO25: no longer names the net of U6.K1 (PL23C/+/PCLKT7_0/LDQ20)
- net IO26: no longer names the net of U6.J2 (PL23B/-/PCLKC7_1/HS/LDQ20)
- net IO27: no longer names the net of U6.J1 (PL23A/+/PCLKT7_1/HS/LDQ20)
- net IO28: no longer names the net of U6.H2 (PL20B/-/HS/LDQSN20)
- net IO29: no longer names the net of U6.G1 (PL20A/+/GR_PCLK7_1/HS/LDQS20)
- net IO30: no longer names the net of U6.G2 (PL14B/-/HS/LDQ20)
- net IO31: no longer names the net of U6.F1 (PL14A/+/HS/LDQ20)
- net IO32: no longer names the net of U6.K15 (PR23D/-/PCLKC2_0/RDQ20)
- net IO33: no longer names the net of U6.K16 (PR23C/+/PCLKT2_0/RDQ20)
- net IO34: no longer names the net of U6.J15 (PR23B/-/PCLKC2_1/HS/RDQ20)
- net IO35: no longer names the net of U6.J16 (PR23A/+/PCLKT2_1/HS/RDQ20)
- net IO36: no longer names the net of U6.H15 (PR20B/-/HS/RDQSN20)
- net IO37: no longer names the net of U6.G15 (PR14B/-/HS/RDQ20)
- net IO38: no longer names the net of U6.G16 (PR20A/+/GR_PCLK2_1/HS/RDQS20)
- net IO39: no longer names the net of U6.F15 (PR11C/+/RDQ8)
- net IO40: no longer names the net of U6.F16 (PR14A/+/HS/RDQ20)
- net IO41: no longer names the net of U6.E15 (PR8B/-/HS/RDQSN8)
- net IO42: no longer names the net of U6.D16 (PR8A/+/HS/RDQS8)
- net IO43: no longer names the net of U6.E16 (PR11D/-/RDQ8)
- net IO44: no longer names the net of U6.C15 (PR5B/-/HS/RDQ8)
- net IO45: no longer names the net of U6.C16 (PR5A/+/HS/RDQ8)
- net IO46: no longer names the net of U6.B15 (PR2B/-/S0_IN/HS/RDQ8)
- net IO47: no longer names the net of U6.B16 (PR2A/+/HS/RDQ8)
- net IO48: no longer names the net of U6.R16 (PR35B/-/VREF1_3/HS/RDQ32)
- net IO49: no longer names the net of U6.P15 (PR32B/-/HS/RDQSN32)
- net IO50: no longer names the net of U6.P16 (PR35A/+/HS/RDQ32)
- net IO51: no longer names the net of U6.N16 (PR32A/+/HS/RDQS32)
- net IO52: no longer names the net of U6.M15 (PR26D/-/PCLKC3_0/RDQ32)
- net IO53: no longer names the net of U6.M16 (PR26C/+/PCLKT3_0/RDQ32)
- net IO54: no longer names the net of U6.L15 (PR26B/-/PCLKC3_1/HS/RDQ32)
- net IO55: no longer names the net of U6.L16 (PR26A/+/PCLKT3_1/HS/RDQ32)
- net IO56: no longer names the net of U6.R12 (PR44A/+/HS/RDQS44)
- net IO57: no longer names the net of U6.T13 (PR44B/-/HS/RDQSN44)
- net IO58: no longer names the net of U6.R13 (PR41C/+/RDQ44)
- net IO59: no longer names the net of U6.T14 (PR41D/-/RDQ44)
- net IO60: no longer names the net of U6.R14 (PR41B/-/HS/RDQ44)
- net IO61: no longer names the net of U6.T15 (PR38D/-/RDQ44)
- net IO62: no longer names the net of U6.R15 (PR38C/+/RDQ44)
- net IO63: no longer names the net of U6.P14 (PR38B/-/HS/RDQ44)
- net SW renamed SW1V1
- new net: R103.2, U104.2
- new net: R109.2, U102.2
- new net: R105.2, U104.6
- new net: R107.2, U104.10
- new net: R114.2, U102.12
- new net: U102.13, U107.7 (6B)
- new net: U104.1, U105.12 (1B)
- new net: R112.2, U102.8
- new net: J6.1, R124.1
- new net: R118.2, U103.8
- new net: U103.9, U106.9 (4B)
- new net: J102.1 (Pin_1), R141.2
- new net: U103.5, U106.10 (3B)
- new net: R117.2, U103.6
- new net: U103.3, U106.11 (2B)
- new net: U103.1, U106.12 (1B)
- new net: R106.2, U104.8
- new net: U104.9, U105.9 (4B)
- new net: U104.11, U105.8 (5B)
- new net: R113.2, U102.10
- new net: U102.11, U107.8 (5B)
- new net: U102.3, U107.11 (2B)
- new net: R110.2, U102.4
- new net: U104.3, U105.11 (2B)
- new net: R104.2, U104.4
- new net: U104.5, U105.10 (3B)
- new net: U104.13, U105.7 (6B)
- new net: R108.2, U104.12
- new net: U102.1, U107.12 (1B)
- new net: R115.2, U103.2
- new net: R111.2, U102.6
- new net: R116.2, U103.4
- new net: U102.5, U107.10 (3B)
- new net: U102.9, U107.9 (4B)
- new net FB3V3: C102.1, R101.1, R102.2, U101.5 (FB)
- new net SW3V3: L101.1, U101.2 (SW)
- new net SYNC+: J101.1 (Pin_1), U108.1 (A)
- new net SYNC-: J101.2 (Pin_2), U108.3 (K)
- no-connect marks 110 -> 179
Other:
- note removed: "DESIGN NOTE: Master SPI config."
- moved on the sheet: C1, C10, C13, C14, C16, C17, C2, C23, C24, C28, C32, C35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

Commit message: save
Parts:
- removed C101, C23, C24: 4.7u, Capacitor_SMD:C_0402_1005Metric, symbol Device:C_Small
- removed C102, C32: 27p, Capacitor_SMD:C_0402_1005Metric, symbol Device:C_Small
- removed C103, C105, C106, C50, C54: 22u, Capacitor_SMD:C_0603_1608Metric, symbol Device:C_Small
- removed C107, C108, C109, C52, C53, C55, C56, C57: 0.1u, Capacitor_SMD:C_0402_1005Metric, symbol Device:C_Small
- removed C28: 10u, Capacitor_SMD:C_0603_1608Metric, symbol Device:C_Small
- removed C51: 2.2u, Capacitor_SMD:C_0402_1005Metric, symbol Device:C_Small
- removed FB1: 120 ohm, Resistor_SMD:R_0402_1005Metric, symbol Device:FerriteBead_Small
- removed FB2: 120 ohm, Inductor_SMD:L_0402_1005Metric, symbol Device:FerriteBead_Small
- removed J1: USB_C_Receptacle_USB2.0_14P, Connector_USB:USB_C_Receptacle_GCT_USB4105-xx-A_16P_TopMnt_Horizontal, symbol Connector:USB_C_Receptacle_USB2.0_16P
- removed J2: Conn_02x10_Odd_Even, Connector_IDC:IDC-Header_2x10_P2.54mm_Vertical, symbol Connector_Generic:Conn_02x10_Odd_Even
- removed J7: RJ45_Hanrun_HR911105A_Horizontal, Connector_RJ:RJ45_Hanrun_HR911105A_Horizontal, symbol Connector:RJ45_Hanrun_HR911105A_Horizontal
- removed L1, L101: 1.5u, Inductor_SMD:L_1008_2520Metric, symbol Device:L
- removed R1, R2, R6, R7: 5.1k, Resistor_SMD:R_0402_1005Metric, symbol Device:R_Small
- removed R101: 450k, Resistor_SMD:R_0402_1005Metric, symbol Device:R_Small
- removed R102, R125, R126, R127, R128, R129, R130, R131, R132, R133, R134, R135, R136, R137, R138, R139, R140, R82: 100k, Resistor_SMD:R_0402_1005Metric, symbol Device:R_Small
- removed R103, R104, R105, R106, R107, R108, R109, R110, R111, R112, R113, R114, R115, R116, R117, R118: 47, Resistor_SMD:R_0402_1005Metric, symbol Device:R_Small
- removed R119, R120, R8: 10k, Resistor_SMD:R_0402_1005Metric, symbol Device:R_Small
- removed R141: 150, Resistor_SMD:R_0402_1005Metric, symbol Device:R_Small
- removed R81: 82k, Resistor_SMD:R_0402_1005Metric, symbol Device:R_Small
- removed R84: 6.49k, Resistor_SMD:R_0402_1005Metric, symbol Device:R_Small
- removed R85: 1k, Resistor_SMD:R_0402_1005Metric, symbol Device:R_Small
- removed U101, U8: TPS62A01ADRLR, Package_TO_SOT_SMD:SOT-563, symbol dc_dc_regulators:TPS62A01
- removed U102, U103, U104: SN74LV6T17, Package_DFN_QFN:DHVQFN-14-1EP_2.5x3mm_P0.5mm_EP1x1.5mm, symbol 74xx:74HC7014
- removed U105, U106, U107: NUF6401MNT1, dfn:DFN-12-1EP_1.35x3mm_P0.5mm, symbol interface_esd:NUF6401MNT1
- removed U2: AP2127K-2.5, Package_TO_SOT_SMD:SOT-23-5, symbol Regulator_Linear:AP2127K-2.5
- removed U9: KSZ8081RNA, Package_DFN_QFN:QFN-24-1EP_4x4mm_P0.5mm_EP2.6x2.6mm, symbol Interface_Ethernet:KSZ8081RNA
- added D102: CDSOD323-T03SC, Diode_SMD:D_SOD-323, symbol Device:D_TVS
- added J10, J11, J12, J13, J14, J15, J16, J4, J5, J8, J9: Sync Out, symbol Connector_Generic:Conn_01x02
- added R47, R48, R49, R50, R51, R52, R53, R54, R55, R56, R57, R58: 47, Resistor_SMD:R_0402_1005Metric, symbol Device:R_Small
- added U13, U14: NUF6401MNT1, dfn:DFN-12-1EP_1.35x3mm_P0.5mm, symbol interface_esd:NUF6401MNT1
Connections:
- net PHY_XI is gone; now on an unnamed net: R5.2
- net +3V3: no longer C38.2, C39.2, C40.2, C41.2, C47.1, U6.J6 (VCCIO6[2]), U6.J7 (VCCIO6[2]), U6.K11 (VCCIO3[2]), U6.L11 (VCCIO3[2])
- net GND: now also J10.2 (Pin_2), J11.2 (Pin_2), J12.2 (Pin_2), J13.2 (Pin_2), J14.2 (Pin_2), J15.2 (Pin_2), J16.2 (Pin_2), J4.2 (Pin_2), J5.2 (Pin_2), J8.2 (Pin_2), J9.2 (Pin_2), U13.13 (GND), U14.13 (GND)
- net SYNC+: now also D102.1 (A1)
- net SYNC-: now also D102.2 (A2)
- net at R4.1, Y1.3 (OUT): no longer R5.1
- net SYNC_OUT4: now reaches U6.B4 (PT11B/-)
- net SYNC_OUT4: now also U13.9 (4B)
- net SYNC_OUT8: now reaches U6.B6 (PT22B/-)
- net SYNC_OUT8: now also U14.11 (2B)
- net SYNC_OUT12: now reaches U6.B7 (PT27B/-/PCLKC0_1)
- net SYNC_OUT12: now also U14.7 (6B)
- net SYNC_OUT3: now reaches U6.C4 (PT11A/+)
- net SYNC_OUT3: now also U13.10 (3B)
- net SYNC_OUT7: now reaches U6.C6 (PT22A/+)
- net SYNC_OUT7: now also U14.12 (1B)
- net SYNC_OUT11: now reaches U6.C7 (PT27A/+/PCLKT0_1)
- net SYNC_OUT11: now also U14.8 (5B)
- net SYNC_OUT2: now reaches U6.D4 (PT9B/-)
- net SYNC_OUT2: now also U13.11 (2B)
- net SYNC_OUT6: now reaches U6.D5 (PT13B/-)
- net SYNC_OUT6: now also U13.7 (6B)
- net SYNC_OUT10: now reaches U6.D7 (PT24B/-/GR_PCLK0_0)
- net SYNC_OUT10: now also U14.9 (4B)
- net SYNC_OUT5: now reaches U6.E5 (PT13A/+)
- net SYNC_OUT5: now also U13.8 (5B)
- net SYNC_OUT9: now reaches U6.E7 (PT24A/+/GR_PCLK0_1)
- net SYNC_OUT9: now also U14.10 (3B)
- net at J102.1 (Pin_1): now also R47.1
- net PORT2_I1: now reaches U6.L15 (PR26B/-/PCLKC3_1/HS/RDQ32)
- net PORT2_I0: now reaches U6.L16 (PR26A/+/PCLKT3_1/HS/RDQ32)
- net PORT2_I3: now reaches U6.M15 (PR26D/-/PCLKC3_0/RDQ32)
- net PORT2_I2: now reaches U6.M16 (PR26C/+/PCLKT3_0/RDQ32)
- net PORT2_I4: now reaches U6.N16 (PR32A/+/HS/RDQS32)
- net PORT2_I8: now reaches U6.P14 (PR38B/-/HS/RDQ44)
- net PORT2_I5: now reaches U6.P15 (PR32B/-/HS/RDQSN32)
- net PORT2_I6: now reaches U6.P16 (PR35A/+/HS/RDQ32)
- net PORT2_I14: now reaches U6.R12 (PR44A/+/HS/RDQS44)
- net PORT2_I12: now reaches U6.R13 (PR41C/+/RDQ44)
- net PORT2_I11: now reaches U6.R14 (PR41B/-/HS/RDQ44)
- net PORT2_I9: now reaches U6.R15 (PR38C/+/RDQ44)
- net PORT2_I7: now reaches U6.R16 (PR35B/-/VREF1_3/HS/RDQ32)
- net PORT2_I15: now reaches U6.T13 (PR44B/-/HS/RDQSN44)
- net PORT2_I13: now reaches U6.T14 (PR41D/-/RDQ44)
- net PORT2_I10: now reaches U6.T15 (PR38D/-/RDQ44)
- net FPGA_XI renamed FPGA_25MHz
- net IO00 renamed PORT1_I15
- net IO01 renamed PORT1_I13
- net IO02 renamed PORT1_I14
- net IO03 renamed PORT1_I12
- net IO04 renamed PORT1_I11
- net IO05 renamed PORT1_I9
- net IO06 renamed PORT1_I10
- net IO07 renamed PORT1_I7
- net IO08 renamed PORT1_I8
- net IO09 renamed PORT1_I6
- net IO10 renamed PORT1_I5
- net IO11 renamed PORT1_I4
- net IO12 renamed PORT1_I3
- net IO13 renamed PORT1_I2
- net IO14 renamed PORT1_I1
- net IO15 renamed PORT1_I0
- net SYNC_OUT renamed SYNC_OUT1
- net SYNC_OUT1: now also U13.12 (1B)
- net ~{ETH.RST} renamed ETH.~{RST}
- new net: J8.1 (Pin_1), R50.1
- new net: J11.1 (Pin_1), R53.1
- new net: R53.2, U14.1 (1A)
- new net: J4.1 (Pin_1), R48.1
- new net: J9.1 (Pin_1), R51.1
- new net: R51.2, U13.5 (5A)
- new net: J5.1 (Pin_1), R49.1
- new net: R49.2, U13.3 (3A)
- new net: J16.1 (Pin_1), R58.1
- new net: R58.2, U14.6 (6A)
- new net: J13.1 (Pin_1), R55.1
- new net: J15.1 (Pin_1), R57.1
- new net: R57.2, U14.5 (5A)
- new net: J14.1 (Pin_1), R56.1
- new net: R56.2, U14.4 (4A)
- new net: J10.1 (Pin_1), R52.1
- new net: R52.2, U13.6 (6A)
- new net: R47.2, U13.1 (1A)
- new net: J12.1 (Pin_1), R54.1
- new net: R50.2, U13.4 (4A)
- new net: R48.2, U13.2 (2A)
- new net: R54.2, U14.2 (2A)
- new net: R55.2, U14.3 (3A)
- new net +1V8: C38.2, C39.2, C40.2, C41.2, C47.1, U6.J6 (VCCIO6[2]), U6.J7 (VCCIO6[2]), U6.K11 (VCCIO3[2]), U6.L11 (VCCIO3[2])
- new net Ethernet/ETH.25MHz_CLOCK_IN: R5.1
- no-connect marks 179 -> 136
Other:
- added sheet Ethernet (ethernet.kicad_sch)
- added sheet IO Port 1 (ioport.kicad_sch)
- added sheet IO Port 2 (ioport.kicad_sch)
- added sheet Power (power.kicad_sch)
- moved on the sheet: C1, C10, C104, C13, C14, C16, C17, C2, C35, C36, C37, C38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

Commit message: save
Parts:
- removed C1, C10, C14, C17, C37, C39, C41, C43, C45, C9: 10n, Capacitor_SMD:C_0402_1005Metric, symbol Device:C_Small
- removed C13, C16, C2, C35, C36, C38, C40, C42, C44, C6, C7: 0.1u, Capacitor_SMD:C_0402_1005Metric, symbol Device:C_Small
- removed C46, C47, C48, C49: 4.7u, Capacitor_SMD:C_0402_1005Metric, symbol Device:C_Small
- removed D102: CDSOD323-T03SC, Diode_SMD:D_SOD-323, symbol Device:D_TVS
- removed D65: LED_Small, LED_SMD:LED_0603_1608Metric, symbol Device:LED_Small
- removed J6: TC2050, Connector:Tag-Connect_TC2050-IDC-NL_2x05_P1.27mm_Vertical, symbol Connector:TC2050
- removed R10, R142, R43, R44, R9: 1k, Resistor_SMD:R_0402_1005Metric, symbol Device:R_Small
- removed R121, R122, R123, R45, R78, R79, R80: 10k, Resistor_SMD:R_0402_1005Metric, symbol Device:R_Small
- removed R124, R47, R48, R49, R50, R51, R52, R53, R54, R55, R56, R57, R58: 47, Resistor_SMD:R_0402_1005Metric, symbol Device:R_Small
- removed U108: TLP2362, Package_SO:SO-5-6_4.55x3.7mm_P1.27mm, symbol Isolator:TLP2310
- removed unit 9 of U6
- removed unit 4 of U6
- removed unit 3 of U6
- removed unit 5 of U6
- removed unit 6 of U6
- removed unit 1 of U6
- removed unit 8 of U6
- removed unit 7 of U6
- removed U7: W25Q16JVUXIQ, Package_SON:Winbond_USON-8-1EP_3x2mm_P0.5mm_EP0.2x1.6mm, symbol Memory_Flash:W25Q32JVZP
- added FB101: 120 ohm, Inductor_SMD:L_0402_1005Metric, symbol Device:FerriteBead_Small
- added J102: USB_C_Receptacle_USB2.0_14P, Connector_USB:USB_C_Receptacle_GCT_USB4105-xx-A_16P_TopMnt_Horizontal, symbol Connector:USB_C_Receptacle_USB2.0_16P
- added J103, J104: Conn_02x10_Odd_Even, Connector_IDC:IDC-Header_2x10_P2.54mm_Vertical, symbol Connector_Generic:Conn_02x10_Odd_Even
- added R101, R104: 5.1k, Resistor_SMD:R_0402_1005Metric, symbol Device:R_Small
- C104: value 0.1u -> 4.7u; LCSC C307331 -> C23733
- D101: renamed from D66; value LED_Small -> RED
- J101: footprint (none) -> Connector_JST:JST_XH_B2B-XH-A_1x02_P2.50mm_Vertical; LCSC (none) -> C158012; MFPN (none) -> B2B-XH-A(LF)(SN)
- J105: renamed from J102; footprint (none) -> Connector_JST:JST_XH_B2B-XH-A_1x02_P2.50mm_Vertical; LCSC (none) -> C158012
- J106: renamed from J4; footprint (none) -> Connector_JST:JST_XH_B2B-XH-A_1x02_P2.50mm_Vertical; LCSC (none) -> C158012
- J107: renamed from J5; footprint (none) -> Connector_JST:JST_XH_B2B-XH-A_1x02_P2.50mm_Vertical; LCSC (none) -> C158012
- J108: renamed from J8; footprint (none) -> Connector_JST:JST_XH_B2B-XH-A_1x02_P2.50mm_Vertical; LCSC (none) -> C158012
- J109: renamed from J9; footprint (none) -> Connector_JST:JST_XH_B2B-XH-A_1x02_P2.50mm_Vertical; LCSC (none) -> C158012
- J110: renamed from J10; footprint (none) -> Connector_JST:JST_XH_B2B-XH-A_1x02_P2.50mm_Vertical; LCSC (none) -> C158012
- J111: renamed from J11; footprint (none) -> Connector_JST:JST_XH_B2B-XH-A_1x02_P2.50mm_Vertical; LCSC (none) -> C158012
- J112: renamed from J12; footprint (none) -> Connector_JST:JST_XH_B2B-XH-A_1x02_P2.50mm_Vertical; LCSC (none) -> C158012
- J113: renamed from J13; footprint (none) -> Connector_JST:JST_XH_B2B-XH-A_1x02_P2.50mm_Vertical; LCSC (none) -> C158012
- J114: renamed from J14; footprint (none) -> Connector_JST:JST_XH_B2B-XH-A_1x02_P2.50mm_Vertical; LCSC (none) -> C158012
- J115: renamed from J15; footprint (none) -> Connector_JST:JST_XH_B2B-XH-A_1x02_P2.50mm_Vertical; LCSC (none) -> C158012
- J116: renamed from J16; footprint (none) -> Connector_JST:JST_XH_B2B-XH-A_1x02_P2.50mm_Vertical; LCSC (none) -> C158012
- R102: renamed from R5; LCSC (none) -> C25118
- R103: renamed from R4; LCSC (none) -> C25118
- U101: renamed from U13; LCSC (none) -> C233491
- U102: renamed from U14; LCSC (none) -> C233491
- renumbered C8 to C101, C5 to C102, C4 to C103, H1 to H101, H2 to H102, H3 to H103, H4 to H104, R83 to R105, U6 to U100, Y1 to Y101
Connections:
- net FPGA_25MHz is gone; now on net Ethernet port/ETH.25MHz_CLOCK_IN: R103.2
- net +3V3: now also C104.1; no longer C104.2
- net Ethernet port/ETH.25MHz_CLOCK_IN: no longer R102.1
- net GND: now also C104.2, J102.A1 (GND), J102.A12 (GND), J102.B1 (GND), J102.B12 (GND), J102.S1 (SHIELD), J103.15 (Pin_15), J103.16 (Pin_16), J103.5 (Pin_5), J103.6 (Pin_6), J104.15 (Pin_15), J104.16 (Pin_16), J104.5 (Pin_5), J104.6 (Pin_6), R101.2, R104.2; no longer C104.1
- net at J108.1 (Pin_1): now also U101.4 (4A)
- net at J111.1 (Pin_1): now also U102.1 (1A)
- net at J106.1 (Pin_1): now also U101.2 (2A)
- net at J109.1 (Pin_1): now also U101.5 (5A)
- net at J107.1 (Pin_1): now also U101.3 (3A)
- net at J116.1 (Pin_1): now also U102.6 (6A)
- net CLOCK_OUT: now reaches R102.2, R103.1, Y101.3 (OUT)
- net at J113.1 (Pin_1): now also U102.3 (3A)
- net at J115.1 (Pin_1): now also U102.5 (5A)
- net at J114.1 (Pin_1): now also U102.4 (4A)
- net at J105.1 (Pin_1): now also U101.1 (1A)
- net at J110.1 (Pin_1): now also U101.6 (6A)
- net at J112.1 (Pin_1): now also U102.2 (2A)
- net SYNC+ renamed Time synchronization/SYNC+
- net SYNC- renamed Time synchronization/SYNC-
- new net CC1: J102.A5 (CC1), R104.1
- new net CC2: J102.B5 (CC2), R101.1
- new net Ethernet port/FPGA.25MHz_CLOCK_IN: R102.1
- new net P1.0: J103.1 (Pin_1)
- new net P1.1: J103.3 (Pin_3)
- new net P1.10: J103.14 (Pin_14)
- new net P1.11: J103.12 (Pin_12)
- new net P1.12: J103.10 (Pin_10)
- new net P1.13: J103.8 (Pin_8)
- new net P1.14: J103.4 (Pin_4)
- new net P1.15: J103.2 (Pin_2)
- new net P1.2: J103.7 (Pin_7)
- new net P1.3: J103.9 (Pin_9)
- new net P1.4: J103.11 (Pin_11)
- new net P1.5: J103.13 (Pin_13)
- new net P1.6: J103.17 (Pin_17)
- new net P1.7: J103.19 (Pin_19)
- new net P1.8: J103.20 (Pin_20)
- new net P1.9: J103.18 (Pin_18)
- new net P2.0: J104.1 (Pin_1)
- new net P2.1: J104.3 (Pin_3)
- new net P2.10: J104.14 (Pin_14)
- new net P2.11: J104.12 (Pin_12)
- new net P2.12: J104.10 (Pin_10)
- new net P2.13: J104.8 (Pin_8)
- new net P2.14: J104.4 (Pin_4)
- new net P2.15: J104.2 (Pin_2)
- new net P2.2: J104.7 (Pin_7)
- new net P2.3: J104.9 (Pin_9)
- new net P2.4: J104.11 (Pin_11)
- new net P2.5: J104.13 (Pin_13)
- new net P2.6: J104.17 (Pin_17)
- new net P2.7: J104.19 (Pin_19)
- new net P2.8: J104.20 (Pin_20)
- new net P2.9: J104.18 (Pin_18)
- new net Power/5V: FB101.2
- new net VBUS: FB101.1, J102.A4 (VBUS), J102.A9 (VBUS), J102.B4 (VBUS), J102.B9 (VBUS)
- no-connect marks 136 -> 16
Other:
- sheet Ethernet renamed Ethernet port
- removed sheet IO Port 1
- removed sheet IO Port 2
- added sheet FPGA settings & programming (fpga_settings.kicad_sch)
- added sheet Logic Channels (logic_channels.kicad_sch)
- added sheet Time synchronization (timesync.kicad_sch)
- added sheet Unused FPGA banks (fpga_unused.kicad_sch)
- sheet Ethernet port ports: added FPGA.25MHz_CLOCK_IN; removed ETH{ETH}
- sheet Power ports: added 5V; removed none
- moved on the sheet: C101, C102, C103, D101, H101, H102, H103, H104, J101, J105, J106, J107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
