File: ssla.kicad_sch (KiCad schematic)
At the start: 35 parts, among them J101 Sync In, J102 USB_C_Receptacle_USB2.0_14P, J103 Conn_02x10_Odd_Even, J104 Conn_02x10_Odd_Even, J105 Sync Out, J106 Sync Out, J107 Sync Out, J108 Sync Out, J109 Sync Out, J110 Sync Out, J111 Sync Out, J112 Sync Out, J113 Sync Out, J114 Sync Out, J115 Sync Out, J116 Sync Out, U100 ECP5U_25_CABGA256, U101 NUF6401MNT1, U102 NUF6401MNT1, Y101 25 MHz

Commit message: save
Parts:
- J101, J105, J106, J107, J108, J109, J110, J111, J112, J113, J114, J115, J116: footprint Connector_JST:JST_XH_B2B-XH-A_1x02_P2.50mm_Vertical -> Connector_JST:JST_PH_B2B-PH-K_1x02_P2.00mm_Vertical
- J103: value Conn_02x10_Odd_Even -> Channel 1
- J104: value Conn_02x10_Odd_Even -> Channel 2
- R102, R103: value 47 -> 33; LCSC C25118 -> C25105
- U100: value ECP5U_25_CABGA256 -> ECP5U_25
- U101, U102: footprint dfn:DFN-12-1EP_1.35x3mm_P0.5mm -> footprints:DFN-12-1EP_1.35x3mm_P0.5mm
Other:
- sheet Ethernet port renamed Ethernet
- moved on the sheet: C101, C102, C103, C104, D101, FB101, H101, H102, H103, H104, J101, J102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

Commit message: Save
Parts:
- removed U100: ECP5U_25, Package_BGA:BGA-256_14.0x14.0mm_Layout16x16_P0.8mm_Ball0.45mm_Pad0.32mm_NSMD, symbol Lattice_ECP5_FPGA:ECP5U_25_CABGA256
- added U100: ECP5U_25, Package_BGA:BGA-256_14.0x14.0mm_Layout16x16_P0.8mm_Ball0.45mm_Pad0.32mm_NSMD, symbol Lattice_ECP5_FPGA:ECP5U_25_CABGA256
Connections:
- net +3V3: now also U100.H6 (VCCIO7[2]), U100.H7 (VCCIO7[2])
- net SYNC_OUT1: now also U100.B1 (PL2A/+/HS/LDQ8)
- net SYNC_OUT10: now also U100.G2 (PL14B/-/HS/LDQ20)
- net SYNC_OUT11: now also U100.G1 (PL20A/+/GR_PCLK7_1/HS/LDQS20)
- net SYNC_OUT12: now also U100.H2 (PL20B/-/HS/LDQSN20)
- net SYNC_OUT2: now also U100.B2 (PL2B/-/HS/LDQ8)
- net SYNC_OUT3: now also U100.C3 (PL2C/+/LDQ8)
- net SYNC_OUT4: now also U100.D3 (PL2D/-/LDQ8)
- net SYNC_OUT5: now also U100.C1 (PL5A/+/HS/LDQ8)
- net SYNC_OUT6: now also U100.C2 (PL5B/-/HS/LDQ8)
- net SYNC_OUT7: now also U100.F2 (PL11C/+/LDQ8)
- net SYNC_OUT8: now also U100.E1 (PL11D/-/LDQ8)
- net SYNC_OUT9: now also U100.F1 (PL14A/+/HS/LDQ20)
- net LED renamed Logic Channels/ACQ_LED
- no-connect marks 16 -> 6
Other:
- sheet Logic Channels ports: added ACQ_LED, SYNC_IN; removed none
- moved on the sheet: C102, C103, C104, D101, J105, J106, J107, J108, J109, J110, J111, J112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
