File: fpga_settings.kicad_sch (KiCad schematic)
At the start: 29 parts, among them J601 TC2050, U100 ECP5U_25_CABGA256, U601 W25Q16JVUXIQ

Commit message: save
Parts:
- R604: value 47 -> 33; LCSC C25118 -> C25105
- U100: value ECP5U_25_CABGA256 -> ECP5U_25
Other:
- moved on the sheet: U601
Changed lines of the file:
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@@
 			)
 		)
-		(property "Value" "ECP5U_25_CABGA256"
+		(property "Value" "ECP5U_25"
 			(at 74.93 138.43 0)
 			(effects
@@
 			)
 		)
-		(property "LCSC" "C5272996"
+		(property "LCSC" ""
 			(at 83.82 143.51 0)
 			(effects
@@
 			)
 		)
-		(property "Value" "ECP5U_25_CABGA256"
+		(property "Value" "ECP5U_25"
 			(at 72.39 72.3899 0)
 			(effects
@@
 			)
 		)
-		(property "LCSC" "C5272996"
+		(property "LCSC" ""
 			(at 127 52.07 0)
 			(effects
@@
 			)
 		)
-		(property "Value" "ECP5U_25_CABGA256"
+		(property "Value" "ECP5U_25"
 			(at 210.82 86.36 0)
 			(effects
@@
 			)
 		)
-		(property "LCSC" "C5272996"
+		(property "LCSC" ""
 			(at 196.85 88.9 0)
 			(effects
@@
 			)
 		)
-		(property "Value" "47"
+		(property "Value" "33"
 			(at 124.46 157.4799 0)
 			(effects
@@
 			)
 		)
-		(property "LCSC" "C25118"
+		(property "LCSC" "C25105"
 			(at 127 156.21 0)
 			(effects
@@
 	)
 	(symbol
+		(lib_name "W25Q32JVZP_1")
 		(lib_id "Memory_Flash:W25Q32JVZP")
 		(at 208.28 146.05 0)
@@
 			)
 		)
-		(property "Description" "32Mb Serial Flash Memory, Standard/Dual/Quad SPI, DFN-8"
+		(property "Description" "32Mbit / 4MiB Serial Flash Memory, Standard/Dual/Quad SPI, 2.7-3.6V, WSON-8"
 			(at 208.28 146.05 0)
 			(effects
