File: ioport.kicad_sch (KiCad schematic)
At the start: 42 parts, among them J2 Conn_02x10_Odd_Even, U102 SN74LV6T17, U103 SN74LV6T17, U104 SN74LV6T17, U105 NUF6401MNT1, U106 NUF6401MNT1, U107 NUF6401MNT1

Commit message: save
Parts:
- removed J2: Conn_02x10_Odd_Even, Connector_IDC:IDC-Header_2x10_P2.54mm_Vertical, symbol Connector_Generic:Conn_02x10_Odd_Even
- R201: renamed from R129; LCSC C258090 -> C25741
- R202: renamed from R131; LCSC C258090 -> C25741
- R203: renamed from R130; LCSC C258090 -> C25741
- R204: renamed from R132; LCSC C258090 -> C25741
- R205: renamed from R125; LCSC C258090 -> C25741
- R206: renamed from R133; LCSC C258090 -> C25741
- R207: renamed from R134; LCSC C258090 -> C25741
- R208: renamed from R126; LCSC C258090 -> C25741
- R209: renamed from R135; LCSC C258090 -> C25741
- R210: renamed from R136; LCSC C258090 -> C25741
- R211: renamed from R127; LCSC C258090 -> C25741
- R212: renamed from R137; LCSC C258090 -> C25741
- R213: renamed from R138; LCSC C258090 -> C25741
- R214: renamed from R128; LCSC C258090 -> C25741
- R215: renamed from R139; LCSC C258090 -> C25741
- R216: renamed from R140; LCSC C258090 -> C25741
- R217: renamed from R103; LCSC (none) -> C25118
- R218: renamed from R104; LCSC (none) -> C25118
- R219: renamed from R105; LCSC (none) -> C25118
- R220: renamed from R106; LCSC (none) -> C25118
- R221: renamed from R107; LCSC (none) -> C25118
- R222: renamed from R108; LCSC (none) -> C25118
- R223: renamed from R109; LCSC (none) -> C25118
- R224: renamed from R110; LCSC (none) -> C25118
- R225: renamed from R111; LCSC (none) -> C25118
- R226: renamed from R112; LCSC (none) -> C25118
- R227: renamed from R113; LCSC (none) -> C25118
- R228: renamed from R114; LCSC (none) -> C25118
- R229: renamed from R115; LCSC (none) -> C25118
- R230: renamed from R116; LCSC (none) -> C25118
- R231: renamed from R117; LCSC (none) -> C25118
- R232: renamed from R118; LCSC (none) -> C25118
- U201: renamed from U104; LCSC (none) -> C22428345
- U202, U203: renamed from U102; LCSC (none) -> C22428345
- U202, U203: renamed from U103; LCSC (none) -> C22428345
- U204: renamed from U105; LCSC (none) -> C233491
- U205: renamed from U107; LCSC (none) -> C233491
- U206: renamed from U106; LCSC (none) -> C233491
- renumbered C109 to C201, C108 to C202, C107 to C203
Connections:
- net IN0 renamed P0
- net IN1 renamed P1
- net IN10 renamed P10
- net P10: now also R204.2; no longer R209.2
- net IN11 renamed P11
- net P11: now also R202.2; no longer R206.2
- net IN12 renamed P12
- net IN13 renamed P13
- net IN14 renamed P14
- net IN15 renamed P15
- net IN2 renamed P2
- net IN3 renamed P3
- net IN4 renamed P4
- net P4: now also R203.2; no longer R204.2
- net IN5 renamed P5
- net P5: now also R201.2; no longer R202.2
- net IN6 renamed P6
- net P6: now also R215.2; no longer R203.2
- net IN7 renamed P7
- net P7: now also R212.2; no longer R201.2
- net IN8 renamed P8
- net P8: now also R209.2; no longer R215.2
- net IN9 renamed P9
- net P9: now also R206.2; no longer R212.2
Other:
- moved on the sheet: R201, R202, R203, R204, R205, R206, R207, R208, R209, R210, R211, R212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

Commit message: save
Parts:
- R217, R218, R219, R220, R221, R222, R223, R224, R225, R226, R227, R228, R229, R230, R231, R232: value 47 -> 33; LCSC C25118 -> C25105
- U201, U202, U203: symbol 74xx:74HC7014 -> buffer:SN74LV6T17
- U204, U205, U206: footprint dfn:DFN-12-1EP_1.35x3mm_P0.5mm -> footprints:DFN-12-1EP_1.35x3mm_P0.5mm
Connections:
- net GND: now also U201.15 (PAD), U202.15 (PAD), U203.15 (PAD)
Other:
- moved on the sheet: C201, C202
