File: power.kicad_sch (KiCad schematic)
At the start: 30 parts, among them J1 USB_C_Receptacle_USB2.0_14P, U1 TPS62A01ADRLR, U101 TPS62A01ADRLR, U2 AP2127K-2.5, U8 TPS62A01ADRLR

Commit message: save
Parts:
- removed C28: 10u, Capacitor_SMD:C_0603_1608Metric, symbol Device:C_Small
- removed FB1: 120 ohm, Resistor_SMD:R_0402_1005Metric, symbol Device:FerriteBead_Small
- removed J1: USB_C_Receptacle_USB2.0_14P, Connector_USB:USB_C_Receptacle_GCT_USB4105-xx-A_16P_TopMnt_Horizontal, symbol Connector:USB_C_Receptacle_USB2.0_16P
- removed R1, R2: 5.1k, Resistor_SMD:R_0402_1005Metric, symbol Device:R_Small
- added C405, C414: 4.7u, Capacitor_SMD:C_0402_1005Metric, symbol Device:C_Small
- R402: renamed from R82; LCSC C258090 -> C25741
- R403: renamed from R3; LCSC C4142 -> C25764
- R404: renamed from R11; LCSC C258090 -> C25741
- R405: renamed from R101; LCSC (none) -> C5159688
- R406: renamed from R102; LCSC C258090 -> C25741
- renumbered C24 to C401, C3 to C402, C101 to C403, C23 to C404, C32 to C406, C11 to C407, C102 to C408, C105 to C409, C12 to C410, C103 to C411, C106 to C412, C15 to C413, L1 to L401, L2 to L402, L101 to L403, R81 to R401, U8 to U401, U1 to U402, U101 to U403, U2 to U404
Connections:
- net +2V5: now also C405.1, C414.1
- net GND: now also C405.2, C414.2
- net +5V renamed 5V
- no-connect marks 9 -> 3
Other:
- moved on the sheet: C401, C402, C403, C404, C406, C407, C408, C409, C410, C411, C412, C413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

Commit message: save
Parts:
- L401, L402, L403: value 1.5u -> 1u; footprint Inductor_SMD:L_1008_2520Metric -> Inductor_SMD:L_0805_2012Metric; LCSC C2047523 -> C20770353; MFPN SRP2512A-1R5M -> SRN2012T-1R0K
- U401, U402, U403: symbol dc_dc_regulators:TPS62A01 -> Regulator_Switching:TPS62A01ADRL
Connections:
- net FB1V1: no longer C407.1, R403.1, R404.2, U402.5 (FB)
- net SW1V1: no longer L402.1, U402.2 (SW)
- new net FB1V8: C407.1, R403.1, R404.2, U402.5 (FB)
- new net SW1V8: L402.1, U402.2 (SW)
Other:
- moved on the sheet: U401, U402, U403
