File: timesync.kicad_sch (KiCad schematic)
At the start: 6 parts, among them U901 TLP2362

Commit message: save
Parts:
- R901, R902: value 47 -> 33; LCSC C25118 -> C25105
Connections:
- net SYNC+: now also D901.1 (A1)
- net SYNC-: now also D901.2 (A2)
- net at R901.1, U901.1 (A): no longer D901.1 (A1)
- net at R902.1, U901.3 (K): no longer D901.2 (A2)
Other:
- moved on the sheet: D901, R901, R902
Changed lines of the file:
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@@
 	)
 	(junction
-		(at 134.62 110.49)
+		(at 125.73 110.49)
 		(diameter 0)
 		(color 0 0 0 0)
 	)
 	(junction
-		(at 134.62 100.33)
+		(at 125.73 100.33)
 		(diameter 0)
 		(color 0 0 0 0)
@@
 	(wire
 		(pts
-			(xy 123.19 110.49) (xy 134.62 110.49)
+			(xy 133.35 110.49) (xy 137.16 110.49)
 		)
 		(stroke
@@
 	(wire
 		(pts
-			(xy 134.62 100.33) (xy 134.62 101.6)
+			(xy 125.73 100.33) (xy 125.73 101.6)
 		)
 		(stroke
@@
 	(wire
 		(pts
-			(xy 106.68 110.49) (xy 118.11 110.49)
+			(xy 106.68 110.49) (xy 125.73 110.49)
 		)
 		(stroke
@@
 	(wire
 		(pts
+			(xy 125.73 100.33) (xy 128.27 100.33)
+		)
+		(stroke
+			(width 0)
+			(type default)
+		)
+	)
+	(wire
+		(pts
 			(xy 162.56 86.36) (xy 147.32 86.36)
 		)
@@
 	(wire
 		(pts
-			(xy 106.68 100.33) (xy 118.11 100.33)
+			(xy 106.68 100.33) (xy 125.73 100.33)
+		)
+		(stroke
+			(width 0)
+			(type default)
+		)
+	)
+	(wire
+		(pts
+			(xy 125.73 110.49) (xy 128.27 110.49)
 		)
 		(stroke
@@
 	(wire
 		(pts
-			(xy 123.19 100.33) (xy 134.62 100.33)
-		)
-		(stroke
-			(width 0)
-			(type default)
-		)
-	)
-	(wire
-		(pts
-			(xy 134.62 100.33) (xy 137.16 100.33)
-		)
-		(stroke
-			(width 0)
-			(type default)
-		)
-	)
-	(wire
-		(pts
-			(xy 134.62 109.22) (xy 134.62 110.49)
+			(xy 133.35 100.33) (xy 137.16 100.33)
+		)
+		(stroke
+			(width 0)
+			(type default)
+		)
+	)
+	(wire
+		(pts
+			(xy 125.73 109.22) (xy 125.73 110.49)
 		)
 		(stroke
@@
 		(pts
 			(xy 162.56 105.41) (xy 170.18 105.41)
-		)
-		(stroke
-			(width 0)
-			(type default)
-		)
-	)
-	(wire
-		(pts
-			(xy 134.62 110.49) (xy 137.16 110.49)
 		)
 		(stroke
@@
 	(symbol
 		(lib_id "Device:R_Small")
-		(at 120.65 100.33 270)
+		(at 130.81 100.33 270)
 		(unit 1)
 		(exclude_from_sim no)
@@
 		(fields_autoplaced yes)
 		(property "Reference" "R901"
-			(at 120.65 95.25 90)
-			(effects
-				(font
-					(size 1.27 1.27)
-				)
-			)
-		)
-		(property "Value" "47"
-			(at 120.65 97.79 90)
+			(at 130.81 95.25 90)
+			(effects
+				(font
+					(size 1.27 1.27)
+				)
+			)
+		)
+		(property "Value" "33"
+			(at 130.81 97.79 90)
 			(effects
 				(font
@@
 		)
 		(property "Footprint" "Resistor_SMD:R_0402_1005Metric"
-			(at 120.65 100.33 0)
+			(at 130.81 100.33 0)
 			(effects
 				(font
@@
 		)
 		(property "Datasheet" "~"
-			(at 120.65 100.33 0)
+			(at 130.81 100.33 0)
 			(effects
 				(font
@@
 		)
 		(property "Description" "Resistor, small symbol"
-			(at 120.65 100.33 0)
+			(at 130.81 100.33 0)
 			(effects
 				(font
@@
 		)
 		(property "MFPN" ""
-			(at 120.65 100.33 0)
+			(at 130.81 100.33 0)
 			(effects
 				(font
@@
 		)
 		(property "Specification" ""
-			(at 120.65 100.33 0)
-			(effects
-				(font
-					(size 1.27 1.27)
-				)
-				(hide yes)
-			)
-		)
-		(property "LCSC" "C25118"
-			(at 120.65 100.33 0)
+			(at 130.81 100.33 0)
+			(effects
+				(font
+					(size 1.27 1.27)
+				)
+				(hide yes)
+			)
+		)
+		(property "LCSC" "C25105"
+			(at 130.81 100.33 0)
 			(effects
 				(font
@@
 	(symbol
 		(lib_id "Device:D_TVS")
-		(at 134.62 105.41 90)
+		(at 125.73 105.41 90)
 		(mirror x)
 		(unit 1)
@@
 		(dnp no)
 		(property "Reference" "D901"
-			(at 132.08 104.1399 90)
+			(at 123.19 104.1399 90)
 			(effects
 				(font
@@
 		)
 		(property "Value" "CDSOD323-T03SC"
-			(at 132.08 106.6799 90)
+			(at 123.19 106.6799 90)
 			(effects
 				(font
@@
 		)
 		(property "Footprint" "Diode_SMD:D_SOD-323"
-			(at 134.62 105.41 0)
+			(at 125.73 105.41 0)
 			(effects
 				(font
@@
 		)
 		(property "Datasheet" "https://www.bourns.com/docs/Product-Datasheets/CDSOD323-TxxSC.pdf"
-			(at 134.62 105.41 0)
+			(at 125.73 105.41 0)
 			(effects
 				(font
@@
 		)
 		(property "Description" "Bidirectional transient-voltage-suppression diode"
-			(at 134.62 105.41 0)
+			(at 125.73 105.41 0)
 			(effects
 				(font
@@
 		)
 		(property "MFPN" "CDSOD323-T03SC"
-			(at 134.62 105.41 0)
+			(at 125.73 105.41 0)
 			(effects
 				(font
@@
 		)
 		(property "LCSC" "C840638"
-			(at 134.62 105.41 0)
+			(at 125.73 105.41 0)
 			(effects
 				(font
@@
 	(symbol
 		(lib_id "Device:R_Small")
-		(at 120.65 110.49 270)
+		(at 130.81 110.49 270)
 		(unit 1)
 		(exclude_from_sim no)
@@
 		(fields_autoplaced yes)
 		(property "Reference" "R902"
-			(at 120.65 113.03 90)
-			(effects
-				(font
-					(size 1.27 1.27)
-				)
-			)
-		)
-		(property "Value" "47"
-			(at 120.65 115.57 90)
+			(at 130.81 113.03 90)
+			(effects
+				(font
+					(size 1.27 1.27)
+				)
+			)
+		)
+		(property "Value" "33"
+			(at 130.81 115.57 90)
 			(effects
 				(font
@@
 		)
 		(property "Footprint" "Resistor_SMD:R_0402_1005Metric"
-			(at 120.65 110.49 0)
+			(at 130.81 110.49 0)
 			(effects
 				(font
@@
 		)
 		(property "Datasheet" "~"
-			(at 120.65 110.49 0)
+			(at 130.81 110.49 0)
 			(effects
 				(font
@@
 		)
 		(property "Description" "Resistor, small symbol"
-			(at 120.65 110.49 0)
+			(at 130.81 110.49 0)
 			(effects
 				(font
@@
 		)
 		(property "MFPN" ""
-			(at 120.65 110.49 0)
+			(at 130.81 110.49 0)
 			(effects
 				(font
@@
 		)
 		(property "Specification" ""
-			(at 120.65 110.49 0)
-			(effects
-				(font
-					(size 1.27 1.27)
-				)
-				(hide yes)
-			)
-		)
-		(property "LCSC" "C25118"
-			(at 120.65 110.49 0)
-			(effects
-				(font
+			(at 130.81 110.49 0)
+			(effects
+				(font
+					(size 1.27 1.27)
+				)
+				(hide yes)
+			)
+		)
+		(property "LCSC" "C25105"
+			(at 130.81 110.49 0)
+			(effects
+				(font
