File: ethernet.kicad_sch (KiCad schematic)
At the start: 18 parts, among them J7 RJ45_Hanrun_HR911105A_Horizon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, U9 KSZ8081RNA

Commit message: save
Parts:
- added C509: 0.1u, Capacitor_SMD:C_0402_1005Metric, symbol Device:C_Small
- added C510: 10n, Capacitor_SMD:C_0402_1005Metric, symbol Device:C_Small
- added U100: ECP5U_25_CABGA256, Package_BGA:BGA-256_14.0x14.0mm_Layout16x16_P0.8mm_Ball0.45mm_Pad0.32mm_NSMD, symbol Lattice_ECP5_FPGA:ECP5U_25_CABGA256
- R507: renamed from R84; LCSC (none) -> C25916
- U501: renamed from U9; LCSC (none) -> C100017
- renumbered C55 to C501, C56 to C502, C57 to C503, C54 to C504, C53 to C505, C50 to C506, C52 to C507, C51 to C508, FB2 to FB501, J7 to J501, R85 to R501, R119 to R502, R120 to R503, R8 to R504, R6 to R505, R7 to R506
Connections:
- net +3V3: now also C509.2, C510.2, U100.F10 (VCCIO1[2]), U100.F11 (VCCIO1[2])
- net ETH.CRS_DV: now also U100.A14 (PT65B/-)
- net ETH.MDC: now also U100.B13 (PT60A/+)
- net ETH.MDIO: now also U100.B12 (PT56A/+)
- net ETH.REF_CLK: now also U100.C8 (PT35A/+/PCLKT1_0)
- net ETH.RXD0: now also U100.A12 (PT53B/-)
- net ETH.RXD1: now also U100.A13 (PT65A/+)
- net ETH.RXER: now also U100.A15 (PT67B/-)
- net ETH.TXD0: now also U100.A10 (PT42B/-)
- net ETH.TXD1: now also U100.A11 (PT53A/+)
- net ETH.TXEN: now also U100.A9 (PT42A/+)
- net ETH.~{RST}: now also U100.B14 (PT67A/+)
- net GND: now also C509.1, C510.1
- new net FPGA.25MHz_CLOCK_IN: U100.B9 (PT38A/+/GR_PCLK1_0)
- no-connect marks 4 -> 24
Other:
- moved on the sheet: C501, C502, C503, C504, C505, C506, C507, C508, FB501, J501, R501, R502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

Commit message: save
Parts:
- added R508, R509, R510, R511, R512, R513, R514, R515: 33, Resistor_SMD:R_0402_1005Metric, symbol Device:R_Small
- U100: value ECP5U_25_CABGA256 -> ECP5U_25
Connections:
- net ~{ETH.RST} is gone; now on net ETH.~{RST}: R504.1
- net ETH.CRS_DV: now also R513.1; no longer U100.A14 (PT65B/-)
- net ETH.REF_CLK: now also R514.1; no longer U100.C8 (PT35A/+/PCLKT1_0)
- net ETH.RXD0: now also R511.1; no longer U100.A12 (PT53B/-)
- net ETH.RXD1: now also R512.1; no longer U100.A13 (PT65A/+)
- net ETH.RXER: now also R515.1; no longer U100.A15 (PT67B/-)
- net ETH.TXD0: now also R509.1; no longer U100.A10 (PT42B/-)
- net ETH.TXD1: now also R510.1; no longer U100.A11 (PT53A/+)
- net ETH.TXEN: now also R508.1; no longer U100.A9 (PT42A/+)
- new net ETH.CRS_DV_{F}: R513.2, U100.A14 (PT65B/-)
- new net ETH.REF_CLK_{F}: R514.2, U100.C8 (PT35A/+/PCLKT1_0)
- new net ETH.RXD0_{F}: R511.2, U100.A12 (PT53B/-)
- new net ETH.RXD1_{F}: R512.2, U100.A13 (PT65A/+)
- new net ETH.RXER_{F}: R515.2, U100.A15 (PT67B/-)
- new net ETH.TXD0_{F}: R509.2, U100.A10 (PT42B/-)
- new net ETH.TXD1_{F}: R510.2, U100.A11 (PT53A/+)
- new net ETH.TXEN_{F}: R508.2, U100.A9 (PT42A/+)

Commit message: Save
Connections:
- net ETH.MDC: now also U100.B10 (PT44A/+); no longer U100.B13 (PT60A/+)
- net ETH.MDIO: now also U100.B8 (PT35B/-/PCLKC1_0); no longer U100.B12 (PT56A/+)
- no-connect marks 24 -> 22
Changed lines of the file:
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@@
-	)
-	(no_connect
-		(at 222.25 80.01)
 	)
 	(no_connect
@@
 	(no_connect
 		(at 222.25 54.61)
-	)
-	(no_connect
-		(at 222.25 62.23)
 	)
 	(wire
@@
 	)
 	(label "ETH.MDC"
-		(at 222.25 115.57 180)
+		(at 222.25 80.01 180)
 		(effects
 			(font
@@
 	)
 	(label "ETH.MDIO"
-		(at 222.25 105.41 180)
-		(effects
-			(font
+		(at 222.25 62.23 180)
+		(effects
+			(font
