File: fpga_unused.kicad_sch (KiCad schematic)
At the start: 5 parts, among them U100 ECP5U_25_CABGA256

Commit message: save
Parts:
- U100: value ECP5U_25_CABGA256 -> ECP5U_25
Changed lines of the file:
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@@
 			)
 		)
-		(property "Value" "ECP5U_25_CABGA256"
+		(property "Value" "ECP5U_25"
 			(at 123.19 102.8699 0)
 			(effects
@@
 			)
 		)
-		(property "LCSC" "C5272996"
+		(property "LCSC" ""
 			(at 73.66 69.85 0)
 			(effects
@@
 			)
 		)
-		(property "Value" "ECP5U_25_CABGA256"
+		(property "Value" "ECP5U_25"
 			(at 204.47 102.8699 0)
 			(effects
@@
 			)
 		)
-		(property "LCSC" "C5272996"
+		(property "LCSC" ""
 			(at 154.94 69.85 0)
 			(effects

Commit message: Save
Parts:
- removed unit 7 of U100
- added unit 2 of U100
Connections:
- net +3V3: now also U100.F6 (VCCIO0[2]), U100.F7 (VCCIO0[2])
- no-connect marks 64 -> 56
