File: logic_channels.kicad_sch (KiCad schematic)
At the start: 7 parts, among them U100 ECP5U_25_CABGA256

Commit message: save
Parts:
- U100: value ECP5U_25_CABGA256 -> ECP5U_25
Other:
- sheet IO Port 1 renamed Buffer 1
- sheet IO Port 2 renamed Buffer 2
Changed lines of the file:
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@@
 	)
 	(label "PORT1_I[0..15]"
-		(at 102.8108 29.1718 0)
+		(at 102.87 27.94 0)
 		(effects
 			(font
@@
 			)
 		)
-		(property "Value" "ECP5U_25_CABGA256"
+		(property "Value" "ECP5U_25"
 			(at 166.37 96.5199 0)
 			(effects
@@
 			)
 		)
-		(property "LCSC" "C5272996"
+		(property "LCSC" ""
 			(at 116.84 63.5 0)
 			(effects
@@
 			)
 		)
-		(property "Value" "ECP5U_25_CABGA256"
+		(property "Value" "ECP5U_25"
 			(at 261.62 96.5199 0)
 			(effects
@@
 			)
 		)
-		(property "LCSC" "C5272996"
+		(property "LCSC" ""
 			(at 212.09 63.5 0)
 			(effects
@@
 			(color 0 0 0 0.0000)
 		)
-		(property "Sheetname" "IO Port 2"
+		(property "Sheetname" "Buffer 2"
 			(at 80.01 45.0084 0)
 			(effects
@@
 			)
 		)
-		(pin "I[0..15]" input
+		(pin "I[0..15]" output
 			(at 100.33 50.8 0)
 			(effects
@@
 			(color 0 0 0 0.0000)
 		)
-		(property "Sheetname" "IO Port 1"
+		(property "Sheetname" "Buffer 1"
 			(at 80.01 22.1484 0)
 			(effects
@@
 			)
 		)
-		(pin "I[0..15]" input
+		(pin "I[0..15]" output
 			(at 100.33 27.94 0)
 			(effects

Commit message: Save
Connections:
- net ACQ_LED: now reaches U100.L13 (PR29C/+/GR_PCLK3_1/RDQ32)
- net SYNC_IN: now reaches U100.L14 (PR32C/+/RDQ32)
- no-connect marks 32 -> 30
Changed lines of the file:
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@@
-	)
-	(no_connect
-		(at 116.84 78.74)
 	)
 	(no_connect
@@
 	)
 	(no_connect
-		(at 116.84 88.9)
-	)
-	(no_connect
 		(at 212.09 76.2)
 	)
@@
 		)
 	)
+	(wire
+		(pts
+			(xy 68.58 88.9) (xy 116.84 88.9)
+		)
+		(stroke
+			(width 0)
+			(type default)
+		)
+	)
 	(bus
 		(pts
@@
 		(pts
 			(xy 226.06 34.29) (xy 228.6 34.29)
+		)
+		(stroke
+			(width 0)
+			(type default)
+		)
+	)
+	(wire
+		(pts
+			(xy 68.58 78.74) (xy 116.84 78.74)
 		)
 		(stroke
@@
 			)
 			(justify right bottom)
+		)
+	)
+	(hierarchical_label "ACQ_LED"
+		(shape input)
+		(at 68.58 78.74 180)
+		(effects
+			(font
+				(size 1.27 1.27)
+			)
+			(justify right)
 		)
 	)
@@
 		(effects
 			(font
+				(size 1.27 1.27)
+			)
+			(justify right)
+		)
+	)
+	(hierarchical_label "SYNC_IN"
+		(shape input)
+		(at 68.58 88.9 180)
+		(effects
+			(font
